Commit message: fix left ft sensor

File: thormang3_description/urdf/thormang3.structure.leg.xacro (robot description, xacro)
@@ -200,7 +200,18 @@
         </link>
 	<!-- left ft joint -->
-        <joint name="l_leg_ft" type="fixed">
+	<!--use "fixed" revolute joint for FT sensor simulation-->
+	<joint name="l_leg_ft" type="revolute">
           <origin xyz="-0.057 0.0 -0.087" rpy="0 0 0"/>
           <parent link="l_leg_an_r_link"/>
+          <child link="l_foot_ft_link"/>
+	  <limit velocity="6.5" effort="1000" lower="0" upper="0" />
+        </joint>
+	<!-- left foot ft link -->
+        <link name="l_foot_ft_link">
+        </link>
+	<!-- left ft fixed joint -->
+        <joint name="l_leg_ft_fixed" type="fixed">
+	  <origin xyz="0 0.0 -0.0275" rpy="0 0 0"/>
+          <parent link="l_foot_ft_link"/>
           <child link="l_leg_foot_link"/>
         </joint>
@@ -208,5 +219,5 @@
         <link name="l_leg_foot_link">
     	  <collision>
-      	    <origin xyz="0 0.014 -0.02" rpy="0 0 0"/>
+      	    <origin xyz="0.0 0.014 0.0075" rpy="0 0 0"/>
       	    <geometry>
               <box size="0.22 0.15 0.015" />
@@ -214,5 +225,5 @@
     	  </collision>
    	  <visual>
-      	    <origin xyz="0 0 0" rpy="0 0 0"/>
+	  <origin xyz="0 0.0 0.0275" rpy="0 0 0"/>
       	    <geometry>
               <mesh filename="package://thormang3_description/meshes/robotis_l_leg_foot.stl" scale="0.001 0.001 0.001"/>
@@ -226,13 +237,4 @@
             <!-- <inertia ixx="0.00219" ixy="0.0" ixz="0.0" iyy="0.00433" iyz="0.00011" izz="0.00609" /> -->
     	  </inertial>
-        </link>
-	<!-- left ft fixed joint -->
-        <joint name="l_leg_ft_fixed" type="fixed">
-          <origin xyz="0.0 0.0 0.0" rpy="${pi} 0 0"/>
-          <parent link="l_leg_foot_link"/>
-          <child link="l_foot_ft_link"/>
-        </joint>
-	<!-- left foot ft link -->
-        <link name="l_foot_ft_link">
         </link>
     </xacro:macro>

Commit message: add mirrored urdf for legs andf fix tf sensor

File: thormang3_description/urdf/thormang3.structure.leg.xacro (robot description, xacro)
@@ -2,17 +2,17 @@
 <robot xmlns:xacro="http://ros.org/wiki/xacro">
     <xacro:property name="pi" value="3.141592654" />
-    <xacro:macro name="thormang3_l_leg" params="parent">
+    <xacro:macro name="thormang3_leg" params="parent prefix reflect">
 	<!-- left hip yaw joint -->
-        <joint name="l_leg_hip_y" type="revolute">
-          <axis xyz="0 0 -1" />
-          <origin xyz="0.0 0.093 -0.018" rpy="0 0 0"/>
+        <joint name="${prefix}_leg_hip_y" type="revolute">
+          <axis xyz="0 0 ${-reflect}" />
+          <origin xyz="0.0 ${reflect * 0.093} -0.018" rpy="0 0 0"/>
           <parent link="${parent}"/>
-          <child link="l_leg_hip_y_link"/>
+          <child link="${prefix}_leg_hip_y_link"/>
           <limit velocity="6.5" effort="1000" lower="${-pi*0.45}" upper="${pi*0.45}" />
           <dynamics damping="0.1" friction="0.0" />
         </joint>
-        <xacro:insert_transmission name="l_leg_hip_y" />
+        <xacro:insert_transmission name="${prefix}_leg_hip_y" />
 	<!-- left hip yaw link -->
-        <link name="l_leg_hip_y_link">
+        <link name="${prefix}_leg_hip_y_link">
     	  <collision>
       	    <origin xyz="-0.01 0 -0.05" rpy="0 0 0"/>
@@ -24,5 +24,5 @@
       	    <origin xyz="0 0 0" rpy="0 0 0"/>
       	    <geometry>
-              <mesh filename="package://thormang3_description/meshes/robotis_l_leg_hip_y_link.stl" scale="0.001 0.001 0.001"/>
+              <mesh filename="package://thormang3_description/meshes/robotis_${prefix}_leg_hip_y_link.stl" scale="0.001 0.001 0.001"/>
       	    </geometry>
       	    <material name="grey"/>
@@ -36,15 +36,15 @@
         </link>
 	<!-- left hip roll joint -->
-        <joint name="l_leg_hip_r" type="revolute">
+        <joint name="${prefix}_leg_hip_r" type="revolute">
           <axis xyz="-1 0 0" />
           <origin xyz="0.057 0.0 -0.075" rpy="0 0 0"/>
-          <parent link="l_leg_hip_y_link"/>
-          <child link="l_leg_hip_r_link"/>
+          <parent link="${prefix}_leg_hip_y_link"/>
+          <child link="${prefix}_leg_hip_r_link"/>
           <limit velocity="6.5" effort="1000" lower="${-pi*0.2}" upper="${pi*0.3}" />
           <dynamics damping="0.1" friction="0.0" />
         </joint>
-        <xacro:insert_transmission name="l_leg_hip_r" />
+        <xacro:insert_transmission name="${prefix}_leg_hip_r" />
 	<!-- left hip roll link -->
-        <link name="l_leg_hip_r_link">
+        <link name="${prefix}_leg_hip_r_link">
 <!--
     	  <collision>
@@ -58,5 +58,5 @@
       	    <origin xyz="0 0 0" rpy="0 0 0"/>
       	    <geometry>
-              <mesh filename="package://thormang3_description/meshes/robotis_l_leg_hip_r_link.stl" scale="0.001 0.001 0.001"/>
+              <mesh filename="package://thormang3_description/meshes/robotis_${prefix}_leg_hip_r_link.stl" scale="0.001 0.001 0.001"/>
       	    </geometry>
       	    <material name="grey"/>
@@ -70,15 +70,15 @@
         </link>
 	<!-- left hip pitch joint -->
-        <joint name="l_leg_hip_p" type="revolute">
-          <axis xyz="0 1 0" />
-          <origin xyz="-0.057 0.033 0.0" rpy="0 0 0"/>
-          <parent link="l_leg_hip_r_link"/>
-          <child link="l_leg_hip_p_link"/>
+        <joint name="${prefix}_leg_hip_p" type="revolute">
+          <axis xyz="0 ${reflect} 0" />
+          <origin xyz="-0.057 ${reflect * 0.033} 0.0" rpy="0 0 0"/>
+          <parent link="${prefix}_leg_hip_r_link"/>
+          <child link="${prefix}_leg_hip_p_link"/>
           <limit velocity="6.5" effort="1000" lower="${-pi*0.4}" upper="${pi*0.4}" />
           <dynamics damping="0.1" friction="0.0" />
         </joint>
-        <xacro:insert_transmission name="l_leg_hip_p" />
+        <xacro:insert_transmission name="${prefix}_leg_hip_p" />
 	<!-- left hip pitch link -->
-        <link name="l_leg_hip_p_link">
+        <link name="${prefix}_leg_hip_p_link">
     	  <collision>
       	    <origin xyz="0 -0.005 -0.145" rpy="0 0 0"/>
@@ -90,5 +90,5 @@
       	    <origin xyz="0 0 0" rpy="0 0 0"/>
       	    <geometry>
-              <mesh filename="package://thormang3_description/meshes/robotis_l_leg_hip_p_link.stl" scale="0.001 0.001 0.001"/>
+              <mesh filename="package://thormang3_description/meshes/robotis_${prefix}_leg_hip_p_link.stl" scale="0.001 0.001 0.001"/>
       	    </geometry>
       	    <material name="grey"/>
@@ -102,17 +102,17 @@
         </link>
 	<!-- left knee pitch joint -->
-        <joint name="l_leg_kn_p" type="revolute">
+        <joint name="${prefix}_leg_kn_p" type="revolute">
           <axis xyz="0 1 0" />
-          <origin xyz="0.0 0.06 -0.3" rpy="0 0 0"/>
-          <parent link="l_leg_hip_p_link"/>
-          <child link="l_leg_kn_p_link"/>
+          <origin xyz="0.0 ${reflect * 0.06} -0.3" rpy="0 0 0"/>
+          <parent link="${prefix}_leg_hip_p_link"/>
+          <child link="${prefix}_leg_kn_p_link"/>
           <limit velocity="6.5" effort="1000" lower="${-pi*0.1}" upper="${pi*0.7}" />
           <dynamics damping="0.1" friction="0.0" />
         </joint>
-        <xacro:insert_transmission name="l_leg_kn_p" />
+        <xacro:insert_transmission name="${prefix}_leg_kn_p" />
 	<!-- left knee pitch link -->
-        <link name="l_leg_kn_p_link">
-    	  <collision>
-      	    <origin xyz="0.01 -0.065 -0.145" rpy="0 0 0"/>
+        <link name="${prefix}_leg_kn_p_link">
+    	  <collision>
+      	    <origin xyz="0.01 ${reflect * -0.065} -0.145" rpy="0 0 0"/>
       	    <geometry>
               <box size="0.11 0.16 0.33" />
@@ -122,5 +122,5 @@
       	    <origin xyz="0 0 0" rpy="0 0 0"/>
       	    <geometry>
-              <mesh filename="package://thormang3_description/meshes/robotis_l_leg_kn_p_link.stl" scale="0.001 0.001 0.001"/>
+              <mesh filename="package://thormang3_description/meshes/robotis_${prefix}_leg_kn_p_link.stl" scale="0.001 0.001 0.001"/>
       	    </geometry>
       	    <material name="grey"/>
@@ -134,15 +134,15 @@
         </link>
 	<!-- left ankle pitch joint -->
-        <joint name="l_leg_an_p" type="revolute">
+        <joint name="${prefix}_leg_an_p" type="revolute">
           <axis xyz="0 -1 0" />
-          <origin xyz="-0.0 -0.06 -0.3" rpy="0 0 0"/>
-          <parent link="l_leg_kn_p_link"/>
-          <child link="l_leg_an_p_link"/>
+          <origin xyz="0.0 ${reflect * -0.06} -0.3" rpy="0 0 0"/>
+          <parent link="${prefix}_leg_kn_p_link"/>
+          <child link="${prefix}_leg_an_p_link"/>
           <limit velocity="6.5" effort="1000" lower="${-pi*0.45}" upper="${pi*0.45}" />
           <dynamics damping="0.1" friction="0.0" />
         </joint>
-        <xacro:insert_transmission name="l_leg_an_p" />
+        <xacro:insert_transmission name="${prefix}_leg_an_p" />
 	<!-- left ankle pitch link -->
-        <link name="l_leg_an_p_link">
+        <link name="${prefix}_leg_an_p_link">
 <!--
     	  <collision>
@@ -156,5 +156,5 @@
       	    <origin xyz="0 0 0" rpy="0 0 0"/>
       	    <geometry>
-              <mesh filename="package://thormang3_description/meshes/robotis_l_leg_an_p_link.stl" scale="0.001 0.001 0.001"/>
+              <mesh filename="package://thormang3_description/meshes/robotis_${prefix}_leg_an_p_link.stl" scale="0.001 0.001 0.001"/>
       	    </geometry>
       	    <material name="grey"/>
@@ -168,15 +168,15 @@
         </link>
 	<!-- left ankle roll joint -->
-        <joint name="l_leg_an_r" type="revolute">
+        <joint name="${prefix}_leg_an_r" type="revolute">
           <axis xyz="1 0 0" />
-          <origin xyz="0.057 -0.033 0.0" rpy="0 0 0"/>
-          <parent link="l_leg_an_p_link"/>
-          <child link="l_leg_an_r_link"/>
+          <origin xyz="0.057 ${reflect * -0.033} 0.0" rpy="0 0 0"/>
+          <parent link="${prefix}_leg_an_p_link"/>
+          <child link="${prefix}_leg_an_r_link"/>
           <limit velocity="6.5" effort="1000" lower="${-pi*0.5}" upper="${pi*0.4}" />
           <dynamics damping="0.1" friction="0.0" />
         </joint>
-        <xacro:insert_transmission name="l_leg_an_r" />
+        <xacro:insert_transmission name="${prefix}_leg_an_r" />
 	<!-- left ankle roll link -->
-        <link name="l_leg_an_r_link">
+        <link name="${prefix}_leg_an_r_link">
     	  <collision>
       	    <origin xyz="-0.067 0 -0.02" rpy="0 0 0"/>
@@ -188,5 +188,5 @@
       	    <origin xyz="0 0 0" rpy="0 0 0"/>
       	    <geometry>
-              <mesh filename="package://thormang3_description/meshes/robotis_l_leg_an_r_link.stl" scale="0.001 0.001 0.001"/>
+              <mesh filename="package://thormang3_description/meshes/robotis_${prefix}_leg_an_r_link.stl" scale="0.001 0.001 0.001"/>
       	    </geometry>
       	    <material name="grey"/>
@@ -201,23 +201,23 @@
 	<!-- left ft joint -->
 	<!--use "fixed" revolute joint for FT sensor simulation-->
-	<joint name="l_leg_ft" type="revolute">
+	<joint name="${prefix}_leg_ft" type="revolute">
           <origin xyz="-0.057 0.0 -0.087" rpy="0 0 0"/>
-          <parent link="l_leg_an_r_link"/>
-          <child link="l_foot_ft_link"/>
+          <parent link="${prefix}_leg_an_r_link"/>
+          <child link="${prefix}_foot_ft_link"/>
 	  <limit velocity="6.5" effort="1000" lower="0" upper="0" />
         </joint>
 	<!-- left foot ft link -->
-        <link name="l_foot_ft_link">
+        <link name="${prefix}_foot_ft_link">
         </link>
 	<!-- left ft fixed joint -->
-        <joint name="l_leg_ft_fixed" type="fixed">
+        <joint name="${prefix}_leg_ft_fixed" type="fixed">
 	  <origin xyz="0 0.0 -0.0275" rpy="0 0 0"/>
-          <parent link="l_foot_ft_link"/>
-          <child link="l_leg_foot_link"/>
+          <parent link="${prefix}_foot_ft_link"/>
+          <child link="${prefix}_leg_foot_link"/>
         </joint>
 	<!-- left foot link -->
-        <link name="l_leg_foot_link">
-    	  <collision>
-      	    <origin xyz="0.0 0.014 0.0075" rpy="0 0 0"/>
+        <link name="${prefix}_leg_foot_link">
+    	  <collision>
+      	    <origin xyz="0.0 ${reflect * 0.014} 0.0075" rpy="0 0 0"/>
       	    <geometry>
               <box size="0.22 0.15 0.015" />
@@ -227,5 +227,5 @@
 	  <origin xyz="0 0.0 0.0275" rpy="0 0 0"/>
       	    <geometry>
-              <mesh filename="package://thormang3_description/meshes/robotis_l_leg_foot.stl" scale="0.001 0.001 0.001"/>
+              <mesh filename="package://thormang3_description/meshes/robotis_${prefix}_leg_foot.stl" scale="0.001 0.001 0.001"/>
       	    </geometry>
       	    <material name="grey"/>
@@ -239,238 +239,3 @@
         </link>
     </xacro:macro>
-    <xacro:macro name="thormang3_r_leg" params="parent">
-	<!-- right hip yaw joint -->
-        <joint name="r_leg_hip_y" type="revolute">
-          <axis xyz="0 0 -1" />
-          <origin xyz="0.0 -0.093 -0.018" rpy="0 0 0"/>
-          <parent link="${parent}"/>
-          <child link="r_leg_hip_y_link"/>
-          <limit velocity="6.5" effort="1000" lower="${-pi*0.45}" upper="${pi*0.45}" />
-          <dynamics damping="0.1" friction="0.0" />
-        </joint>
-        <xacro:insert_transmission name="r_leg_hip_y" />
-	<!-- right hip yaw link -->
-        <link name="r_leg_hip_y_link">
-    	  <collision>
-      	    <origin xyz="-0.01 0 -0.05" rpy="0 0 0"/>
-      	    <geometry>
-              <box size="0.17 0.07 0.1" />
-      	    </geometry>
-    	  </collision>
-   	  <visual>
-      	    <origin xyz="0 0 0" rpy="0 0 0"/>
-      	    <geometry>
-              <mesh filename="package://thormang3_description/meshes/robotis_r_leg_hip_y_link.stl" scale="0.001 0.001 0.001"/>
-      	    </geometry>
-      	    <material name="grey"/>
-    	  </visual>
-          <inertial>
-      	    <origin xyz="-0.012 0.000 -0.025" rpy="0 0 0"/>
-      	    <mass value="0.243"/>
-      	    <inertia ixx="1.0" ixy="0.0" ixz="0.0" iyy="1.0" iyz="0.0" izz="1.0" />
-            <!-- <inertia ixx="0.00024" ixy="0.0" ixz="0.0" iyy="0.00101" iyz="0.0" izz="0.00092" /> -->
-    	  </inertial>
-        </link>
-	<!-- right hip roll joint -->
-        <joint name="r_leg_hip_r" type="revolute">
-          <axis xyz="-1 0 0" />
-          <origin xyz="0.057 0.0 -0.075" rpy="0 0 0"/>
-          <parent link="r_leg_hip_y_link"/>
-          <child link="r_leg_hip_r_link"/>
-          <limit velocity="6.5" effort="1000" lower="${-pi*0.3}" upper="${pi*0.2}" />
-          <dynamics damping="0.1" friction="0.0" />
-        </joint>
-        <xacro:insert_transmission name="r_leg_hip_r" />
-	<!-- right hip roll link -->
-        <link name="r_leg_hip_r_link">
-<!--
-    	  <collision>
-      	    <origin xyz="0 0 0" rpy="0 0 0"/>
-      	    <geometry>
-              <box size="0.01 0.01 0.01" />
-      	    </geometry>
-    	  </collision>
--->
-   	  <visual>
-      	    <origin xyz="0 0 0" rpy="0 0 0"/>
-      	    <geometry>
-              <mesh filename="package://thormang3_description/meshes/robotis_r_leg_hip_r_link.stl" scale="0.001 0.001 0.001"/>
-      	    </geometry>
-      	    <material name="grey"/>
-    	  </visual>
-          <inertial>
-      	    <origin xyz="-0.068 0.000 0.000" rpy="0 0 0"/>
-      	    <mass value="1.045"/>
-      	    <inertia ixx="1.0" ixy="0.0" ixz="0.0" iyy="1.0" iyz="0.0" izz="1.0" />
-            <!-- <inertia ixx="0.00056" ixy="0.0" ixz="0.0" iyy="0.00168" iyz="0.0" izz="0.00171" /> -->
-    	  </inertial>
-        </link>
-	<!-- right hip pitch joint -->
-        <joint name="r_leg_hip_p" type="revolute">
-          <axis xyz="0 -1 0" />
-          <origin xyz="-0.057 -0.033 0.0" rpy="0 0 0"/>
-          <parent link="r_leg_hip_r_link"/>
-          <child link="r_leg_hip_p_link"/>
-          <limit velocity="6.5" effort="1000" lower="${-pi*0.4}" upper="${pi*0.4}" />
-          <dynamics damping="0.1" friction="0.0" />
-        </joint>
-        <xacro:insert_transmission name="r_leg_hip_p" />
-	<!-- right hip pitch link -->
-        <link name="r_leg_hip_p_link">
-    	  <collision>
-      	    <origin xyz="0 0.005 -0.145" rpy="0 0 0"/>
-      	    <geometry>
-              <box size="0.11 0.16 0.33" />
-      	    </geometry>
-    	  </collision>
-   	  <visual>
-      	    <origin xyz="0 0 0" rpy="0 0 0"/>
-      	    <geometry>
-              <mesh filename="package://thormang3_description/meshes/robotis_r_leg_hip_p_link.stl" scale="0.001 0.001 0.001"/>
-      	    </geometry>
-      	    <material name="grey"/>
-    	  </visual>
-          <inertial>
-      	    <origin xyz="0.022 0.007 -0.168" rpy="0 0 0"/>
-      	    <mass value="3.095"/>
-      	    <inertia ixx="1.0" ixy="0.0" ixz="0.0" iyy="1.0" iyz="0.0" izz="1.0" />
-            <!-- <inertia ixx="0.04328" ixy="-0.00027" ixz="0.00286" iyy="0.04042" iyz="-0.00202" izz="0.00560" /> -->
-    	  </inertial>
-        </link>
-	<!-- right knee pitch joint -->
-        <joint name="r_leg_kn_p" type="revolute">
-          <axis xyz="0 -1 0" />
-          <origin xyz="0.0 -0.06 -0.3" rpy="0 0 0"/>
-          <parent link="r_leg_hip_p_link"/>
-          <child link="r_leg_kn_p_link"/>
-          <limit velocity="6.5" effort="1000" lower="${-pi*0.7}" upper="${pi*0.1}" />
-          <dynamics damping="0.1" friction="0.0" />
-        </joint>
-        <xacro:insert_transmission name="r_leg_kn_p" />
-	<!-- right knee pitch link -->
-        <link name="r_leg_kn_p_link">
-    	  <collision>
-      	    <origin xyz="0.01 0.065 -0.145" rpy="0 0 0"/>
-      	    <geometry>
-              <box size="0.11 0.16 0.33" />
-      	    </geometry>
-    	  </collision>
-   	  <visual>
-      	    <origin xyz="0 0 0" rpy="0 0 0"/>
-      	    <geometry>
-              <mesh filename="package://thormang3_description/meshes/robotis_r_leg_kn_p_link.stl" scale="0.001 0.001 0.001"/>
-      	    </geometry>
-      	    <material name="grey"/>
-    	  </visual>
-          <inertial>
-      	    <origin xyz="-0.002 0.066 -0.183" rpy="0 0 0"/>
-      	    <mass value="2.401"/>
-      	    <inertia ixx="1.0" ixy="0.0" ixz="0.0" iyy="1.0" iyz="0.0" izz="1.0" />
-            <!-- <inertia ixx="0.01971" ixy="-0.00031" ixz="-0.00294" iyy="0.01687" iyz="-0.00140" izz="0.00574" /> -->
-    	  </inertial>
-        </link>
-	<!-- right ankle pitch joint -->
-        <joint name="r_leg_an_p" type="revolute">
-          <axis xyz="0 1 0" />
-          <origin xyz="-0.0 0.06 -0.3" rpy="0 0 0"/>
-          <parent link="r_leg_kn_p_link"/>
-          <child link="r_leg_an_p_link"/>
-          <limit velocity="6.5" effort="1000" lower="${-pi*0.45}" upper="${pi*0.45}" />
-          <dynamics damping="0.1" friction="0.0" />
-        </joint>
-        <xacro:insert_transmission name="r_leg_an_p" />
-	<!-- right ankle pitch link -->
-        <link name="r_leg_an_p_link">
-<!--
-    	  <collision>
-      	    <origin xyz="0 0 0" rpy="0 0 0"/>
-      	    <geometry>
-              <box size="0.01 0.01 0.01" />
-      	    </geometry>
-    	  </collision>
--->
-   	  <visual>
-      	    <origin xyz="0 0 0" rpy="0 0 0"/>
-      	    <geometry>
-              <mesh filename="package://thormang3_description/meshes/robotis_r_leg_an_p_link.stl" scale="0.001 0.001 0.001"/>
-      	    </geometry>
-      	    <material name="grey"/>
-    	  </visual>
-          <inertial>
-      	    <origin xyz="-0.011 0.033 0.000" rpy="0 0 0"/>
-      	    <mass value="1.045"/>
-      	    <inertia ixx="1.0" ixy="0.0" ixz="0.0" iyy="1.0" iyz="0.0" izz="1.0" />
-            <!-- <inertia ixx="0.00056" ixy="0.0" ixz="0.0" iyy="0.00168" iyz="0.0" izz="0.00171" /> -->
-    	  </inertial>
-        </link>
-	<!-- right ankle roll joint -->
-        <joint name="r_leg_an_r" type="revolute">
-          <axis xyz="1 0 0" />
-          <origin xyz="0.057 0.033 0.0" rpy="0 0 0"/>
-          <parent link="r_leg_an_p_link"/>
-          <child link="r_leg_an_r_link"/>
-          <limit velocity="6.5" effort="1000" lower="${-pi*0.45}" upper="${pi*0.45}" />
-          <dynamics damping="0.1" friction="0.0" />
-        </joint>
-        <xacro:insert_transmission name="r_leg_an_r" />
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
File: thormang3_description/urdf/thormang3.structure.torso.xacro (robot description, xacro)
@@ -118,6 +118,6 @@
   <xacro:thormang3_l_arm parent="chest_link" />
   <xacro:thormang3_r_arm parent="chest_link" />
-  <xacro:thormang3_l_leg parent="pelvis_link" />
-  <xacro:thormang3_r_leg parent="pelvis_link" />
+  <xacro:thormang3_leg parent="pelvis_link" prefix="l" reflect="1" />
+  <xacro:thormang3_leg parent="pelvis_link" prefix="r" reflect="-1" />
   <xacro:thormang3_head parent="chest_link" />
 </robot>

Commit message: fix axes

File: thormang3_description/urdf/thormang3.structure.leg.xacro (robot description, xacro)
@@ -37,5 +37,5 @@
 	<!-- left hip roll joint -->
         <joint name="${prefix}_leg_hip_r" type="revolute">
-          <axis xyz="-1 0 0" />
+          <axis xyz="${-reflect} 0 0" />
           <origin xyz="0.057 0.0 -0.075" rpy="0 0 0"/>
           <parent link="${prefix}_leg_hip_y_link"/>
@@ -103,9 +103,9 @@
 	<!-- left knee pitch joint -->
         <joint name="${prefix}_leg_kn_p" type="revolute">
-          <axis xyz="0 1 0" />
+          <axis xyz="0 ${reflect} 0" />
           <origin xyz="0.0 ${reflect * 0.06} -0.3" rpy="0 0 0"/>
           <parent link="${prefix}_leg_hip_p_link"/>
           <child link="${prefix}_leg_kn_p_link"/>
-          <limit velocity="6.5" effort="1000" lower="${-pi*0.1}" upper="${pi*0.7}" />
+          <limit velocity="6.5" effort="1000" lower="${-pi*0.5}" upper="${pi*0.5}" />
           <dynamics damping="0.1" friction="0.0" />
         </joint>
@@ -135,5 +135,5 @@
 	<!-- left ankle pitch joint -->
         <joint name="${prefix}_leg_an_p" type="revolute">
-          <axis xyz="0 -1 0" />
+          <axis xyz="0 ${-reflect} 0" />
           <origin xyz="0.0 ${reflect * -0.06} -0.3" rpy="0 0 0"/>
           <parent link="${prefix}_leg_kn_p_link"/>
@@ -169,5 +169,5 @@
 	<!-- left ankle roll joint -->
         <joint name="${prefix}_leg_an_r" type="revolute">
-          <axis xyz="1 0 0" />
+          <axis xyz="${reflect} 0 0" />
           <origin xyz="0.057 ${reflect * -0.033} 0.0" rpy="0 0 0"/>
           <parent link="${prefix}_leg_an_p_link"/>
