Commit message: fix wrong axes

File: thormang3_description/urdf/thormang3.structure.leg.xacro (robot description, xacro)
@@ -5,5 +5,5 @@
 	<!-- left hip yaw joint -->
         <joint name="${prefix}_leg_hip_y" type="revolute">
-          <axis xyz="0 0 ${-reflect}" />
+          <axis xyz="0 0 -1" />
           <origin xyz="0.0 ${reflect * 0.093} -0.018" rpy="0 0 0"/>
           <parent link="${parent}"/>
@@ -37,5 +37,5 @@
 	<!-- left hip roll joint -->
         <joint name="${prefix}_leg_hip_r" type="revolute">
-          <axis xyz="${-reflect} 0 0" />
+          <axis xyz="-1 0 0" />
           <origin xyz="0.057 0.0 -0.075" rpy="0 0 0"/>
           <parent link="${prefix}_leg_hip_y_link"/>
@@ -169,5 +169,5 @@
 	<!-- left ankle roll joint -->
         <joint name="${prefix}_leg_an_r" type="revolute">
-          <axis xyz="${reflect} 0 0" />
+          <axis xyz="1 0 0" />
           <origin xyz="0.057 ${reflect * -0.033} 0.0" rpy="0 0 0"/>
           <parent link="${prefix}_leg_an_p_link"/>

Commit message: adjusted joint limits for legs

File: thormang3_description/urdf/thormang3.structure.leg.xacro (robot description, xacro)
@@ -41,5 +41,5 @@
           <parent link="${prefix}_leg_hip_y_link"/>
           <child link="${prefix}_leg_hip_r_link"/>
-          <limit velocity="6.5" effort="1000" lower="${-pi*0.2}" upper="${pi*0.3}" />
+          <limit velocity="6.5" effort="1000" lower="${-pi*0.2}" upper="${pi*0.2}" />
           <dynamics damping="0.1" friction="0.0" />
         </joint>
@@ -75,5 +75,10 @@
           <parent link="${prefix}_leg_hip_r_link"/>
           <child link="${prefix}_leg_hip_p_link"/>
-          <limit velocity="6.5" effort="1000" lower="${-pi*0.4}" upper="${pi*0.4}" />
+	  <xacro:if value="${reflect - 1}">
+           <limit velocity="6.5" effort="1000" lower="${-pi*0.25}" upper="${pi*0.4}" />
+	  </xacro:if>
+	  <xacro:unless value="${reflect - 1}">
+	    <limit velocity="6.5" effort="1000" lower="${-pi*0.4}" upper="${pi*0.25}" />
+	  </xacro:unless>
           <dynamics damping="0.1" friction="0.0" />
         </joint>
@@ -107,5 +112,10 @@
           <parent link="${prefix}_leg_hip_p_link"/>
           <child link="${prefix}_leg_kn_p_link"/>
-          <limit velocity="6.5" effort="1000" lower="${-pi*0.5}" upper="${pi*0.5}" />
+	  <xacro:if value="${reflect - 1}">
+           <limit velocity="6.5" effort="1000" lower="${-pi*0.6}" upper="${pi*0.45}" />
+	  </xacro:if>
+	  <xacro:unless value="${reflect - 1}">
+	    <limit velocity="6.5" effort="1000" lower="${-pi*0.45}" upper="${pi*0.6}" />
+	  </xacro:unless>
           <dynamics damping="0.1" friction="0.0" />
         </joint>
@@ -173,5 +183,5 @@
           <parent link="${prefix}_leg_an_p_link"/>
           <child link="${prefix}_leg_an_r_link"/>
-          <limit velocity="6.5" effort="1000" lower="${-pi*0.5}" upper="${pi*0.4}" />
+          <limit velocity="6.5" effort="1000" lower="${-pi*0.25}" upper="${pi*0.25}" />
           <dynamics damping="0.1" friction="0.0" />
         </joint>

Commit message: Removed double definition of pi

File: thormang3_description/urdf/thormang3.structure.leg.xacro (robot description, xacro)
@@ -1,5 +1,4 @@
 <?xml version="1.0"?>
 <robot xmlns:xacro="http://ros.org/wiki/xacro">
-    <xacro:property name="pi" value="3.141592654" />
     <xacro:macro name="thormang3_leg" params="parent prefix reflect">
 	<!-- left hip yaw joint -->

Commit message: cleaned up xacro

File: thormang3_description/urdf/thormang3.structure.leg.xacro (robot description, xacro)
@@ -2,248 +2,248 @@
 <robot xmlns:xacro="http://ros.org/wiki/xacro">
     <xacro:macro name="thormang3_leg" params="parent prefix reflect">
-	<!-- left hip yaw joint -->
+        <!-- hip yaw joint -->
         <joint name="${prefix}_leg_hip_y" type="revolute">
-          <axis xyz="0 0 -1" />
-          <origin xyz="0.0 ${reflect * 0.093} -0.018" rpy="0 0 0"/>
-          <parent link="${parent}"/>
-          <child link="${prefix}_leg_hip_y_link"/>
-          <limit velocity="6.5" effort="1000" lower="${-pi*0.45}" upper="${pi*0.45}" />
-          <dynamics damping="0.1" friction="0.0" />
+            <axis xyz="0 0 -1" />
+            <origin xyz="0.0 ${reflect * 0.093} -0.018" rpy="0 0 0"/>
+            <parent link="${parent}"/>
+            <child link="${prefix}_leg_hip_y_link"/>
+            <limit velocity="6.5" effort="1000" lower="${-pi*0.45}" upper="${pi*0.45}" />
+            <dynamics damping="0.1" friction="0.0" />
         </joint>
         <xacro:insert_transmission name="${prefix}_leg_hip_y" />
-	<!-- left hip yaw link -->
+        <!-- hip yaw link -->
         <link name="${prefix}_leg_hip_y_link">
-    	  <collision>
-      	    <origin xyz="-0.01 0 -0.05" rpy="0 0 0"/>
-      	    <geometry>
-              <box size="0.17 0.07 0.1" />
-      	    </geometry>
-    	  </collision>
-   	  <visual>
-      	    <origin xyz="0 0 0" rpy="0 0 0"/>
-      	    <geometry>
-              <mesh filename="package://thormang3_description/meshes/robotis_${prefix}_leg_hip_y_link.stl" scale="0.001 0.001 0.001"/>
-      	    </geometry>
-      	    <material name="grey"/>
-    	  </visual>
-          <inertial>
-      	    <origin xyz="0.012 0.000 -0.025" rpy="0 0 0"/>
-      	    <mass value="0.243"/>
-      	    <inertia ixx="1.0" ixy="0.0" ixz="0.0" iyy="1.0" iyz="0.0" izz="1.0" />
-    	    <!-- <inertia ixx="0.00024" ixy="0.0" ixz="0.0" iyy="0.00101" iyz="0.0" izz="0.00092" /> -->
-	  </inertial>
-        </link>
-	<!-- left hip roll joint -->
+            <collision>
+                <origin xyz="-0.01 0 -0.05" rpy="0 0 0"/>
+                <geometry>
+                    <box size="0.17 0.07 0.1" />
+                </geometry>
+            </collision>
+            <visual>
+                <origin xyz="0 0 0" rpy="0 0 0"/>
+                <geometry>
+                    <mesh filename="package://thormang3_description/meshes/robotis_${prefix}_leg_hip_y_link.stl" scale="0.001 0.001 0.001"/>
+                </geometry>
+                <material name="grey"/>
+            </visual>
+            <inertial>
+                <origin xyz="0.012 0.000 -0.025" rpy="0 0 0"/>
+                <mass value="0.243"/>
+                <inertia ixx="1.0" ixy="0.0" ixz="0.0" iyy="1.0" iyz="0.0" izz="1.0" />
+              <!-- <inertia ixx="0.00024" ixy="0.0" ixz="0.0" iyy="0.00101" iyz="0.0" izz="0.00092" /> -->
+            </inertial>
+        </link>
+        <!-- hip roll joint -->
         <joint name="${prefix}_leg_hip_r" type="revolute">
-          <axis xyz="-1 0 0" />
-          <origin xyz="0.057 0.0 -0.075" rpy="0 0 0"/>
-          <parent link="${prefix}_leg_hip_y_link"/>
-          <child link="${prefix}_leg_hip_r_link"/>
-          <limit velocity="6.5" effort="1000" lower="${-pi*0.2}" upper="${pi*0.2}" />
-          <dynamics damping="0.1" friction="0.0" />
+            <axis xyz="-1 0 0" />
+            <origin xyz="0.057 0.0 -0.075" rpy="0 0 0"/>
+            <parent link="${prefix}_leg_hip_y_link"/>
+            <child link="${prefix}_leg_hip_r_link"/>
+            <limit velocity="6.5" effort="1000" lower="${-pi*0.2}" upper="${pi*0.2}" />
+            <dynamics damping="0.1" friction="0.0" />
         </joint>
         <xacro:insert_transmission name="${prefix}_leg_hip_r" />
-	<!-- left hip roll link -->
+        <!-- hip roll link -->
         <link name="${prefix}_leg_hip_r_link">
-<!--
-    	  <collision>
-      	    <origin xyz="-0.057 0 0" rpy="0 0 0"/>
-      	    <geometry>
-              <box size="0.01 0.01 0.01" />
-      	    </geometry>
-    	  </collision>
--->
-   	  <visual>
-      	    <origin xyz="0 0 0" rpy="0 0 0"/>
-      	    <geometry>
-              <mesh filename="package://thormang3_description/meshes/robotis_${prefix}_leg_hip_r_link.stl" scale="0.001 0.001 0.001"/>
-      	    </geometry>
-      	    <material name="grey"/>
-    	  </visual>
-          <inertial>
-      	    <origin xyz="-0.068 0.000 0.000" rpy="0 0 0"/>
-      	    <mass value="1.045"/>
-      	    <inertia ixx="1.0" ixy="0.0" ixz="0.0" iyy="1.0" iyz="0.0" izz="1.0" />
-            <!-- <inertia ixx="0.00056" ixy="0.0" ixz="0.0" iyy="0.00168" iyz="0.0" izz="0.00171" /> -->
-    	  </inertial>
-        </link>
-	<!-- left hip pitch joint -->
+  <!--
+          <collision>
+              <origin xyz="-0.057 0 0" rpy="0 0 0"/>
+              <geometry>
+                <box size="0.01 0.01 0.01" />
+              </geometry>
+          </collision>
+  -->
+            <visual>
+                <origin xyz="0 0 0" rpy="0 0 0"/>
+                <geometry>
+                    <mesh filename="package://thormang3_description/meshes/robotis_${prefix}_leg_hip_r_link.stl" scale="0.001 0.001 0.001"/>
+                </geometry>
+                <material name="grey"/>
+            </visual>
+            <inertial>
+                <origin xyz="-0.068 0.000 0.000" rpy="0 0 0"/>
+                <mass value="1.045"/>
+                <inertia ixx="1.0" ixy="0.0" ixz="0.0" iyy="1.0" iyz="0.0" izz="1.0" />
+                <!-- <inertia ixx="0.00056" ixy="0.0" ixz="0.0" iyy="0.00168" iyz="0.0" izz="0.00171" /> -->
+            </inertial>
+        </link>
+  <!-- hip pitch joint -->
         <joint name="${prefix}_leg_hip_p" type="revolute">
-          <axis xyz="0 ${reflect} 0" />
-          <origin xyz="-0.057 ${reflect * 0.033} 0.0" rpy="0 0 0"/>
-          <parent link="${prefix}_leg_hip_r_link"/>
-          <child link="${prefix}_leg_hip_p_link"/>
-	  <xacro:if value="${reflect - 1}">
-           <limit velocity="6.5" effort="1000" lower="${-pi*0.25}" upper="${pi*0.4}" />
-	  </xacro:if>
-	  <xacro:unless value="${reflect - 1}">
-	    <limit velocity="6.5" effort="1000" lower="${-pi*0.4}" upper="${pi*0.25}" />
-	  </xacro:unless>
-          <dynamics damping="0.1" friction="0.0" />
+            <axis xyz="0 ${reflect} 0" />
+            <origin xyz="-0.057 ${reflect * 0.033} 0.0" rpy="0 0 0"/>
+            <parent link="${prefix}_leg_hip_r_link"/>
+            <child link="${prefix}_leg_hip_p_link"/>
+            <xacro:if value="${reflect - 1}">
+                <limit velocity="6.5" effort="1000" lower="${-pi*0.25}" upper="${pi*0.4}" />
+            </xacro:if>
+            <xacro:unless value="${reflect - 1}">
+                <limit velocity="6.5" effort="1000" lower="${-pi*0.4}" upper="${pi*0.25}" />
+            </xacro:unless>
+            <dynamics damping="0.1" friction="0.0" />
         </joint>
         <xacro:insert_transmission name="${prefix}_leg_hip_p" />
-	<!-- left hip pitch link -->
+        <!-- hip pitch link -->
         <link name="${prefix}_leg_hip_p_link">
-    	  <collision>
-      	    <origin xyz="0 -0.005 -0.145" rpy="0 0 0"/>
-      	    <geometry>
-              <box size="0.11 0.16 0.33" />
-      	    </geometry>
-    	  </collision>
-   	  <visual>
-      	    <origin xyz="0 0 0" rpy="0 0 0"/>
-      	    <geometry>
-              <mesh filename="package://thormang3_description/meshes/robotis_${prefix}_leg_hip_p_link.stl" scale="0.001 0.001 0.001"/>
-      	    </geometry>
-      	    <material name="grey"/>
-    	  </visual>
-          <inertial>
-      	    <origin xyz="0.022 -0.007 -0.168" rpy="0 0 0"/>
-      	    <mass value="3.095"/>
-      	    <inertia ixx="1.0" ixy="0.0" ixz="0.0" iyy="1.0" iyz="0.0" izz="1.0" />
-            <!-- <inertia ixx="0.04328" ixy="0.00028" ixz="0.00288" iyy="0.04042" iyz="-0.00202" izz="0.00560" /> -->
-    	  </inertial>
-        </link>
-	<!-- left knee pitch joint -->
+            <collision>
+                <origin xyz="0 -0.005 -0.145" rpy="0 0 0"/>
+                <geometry>
+                    <box size="0.11 0.16 0.33" />
+                </geometry>
+            </collision>
+            <visual>
+                <origin xyz="0 0 0" rpy="0 0 0"/>
+                <geometry>
+                    <mesh filename="package://thormang3_description/meshes/robotis_${prefix}_leg_hip_p_link.stl" scale="0.001 0.001 0.001"/>
+                </geometry>
+                <material name="grey"/>
+            </visual>
+            <inertial>
+                <origin xyz="0.022 -0.007 -0.168" rpy="0 0 0"/>
+                <mass value="3.095"/>
+                <inertia ixx="1.0" ixy="0.0" ixz="0.0" iyy="1.0" iyz="0.0" izz="1.0" />
+                <!-- <inertia ixx="0.04328" ixy="0.00028" ixz="0.00288" iyy="0.04042" iyz="-0.00202" izz="0.00560" /> -->
+            </inertial>
+        </link>
+        <!-- knee pitch joint -->
         <joint name="${prefix}_leg_kn_p" type="revolute">
-          <axis xyz="0 ${reflect} 0" />
-          <origin xyz="0.0 ${reflect * 0.06} -0.3" rpy="0 0 0"/>
-          <parent link="${prefix}_leg_hip_p_link"/>
-          <child link="${prefix}_leg_kn_p_link"/>
-	  <xacro:if value="${reflect - 1}">
-           <limit velocity="6.5" effort="1000" lower="${-pi*0.6}" upper="${pi*0.45}" />
-	  </xacro:if>
-	  <xacro:unless value="${reflect - 1}">
-	    <limit velocity="6.5" effort="1000" lower="${-pi*0.45}" upper="${pi*0.6}" />
-	  </xacro:unless>
-          <dynamics damping="0.1" friction="0.0" />
+            <axis xyz="0 ${reflect} 0" />
+            <origin xyz="0.0 ${reflect * 0.06} -0.3" rpy="0 0 0"/>
+            <parent link="${prefix}_leg_hip_p_link"/>
+            <child link="${prefix}_leg_kn_p_link"/>
+            <xacro:if value="${reflect - 1}">
+                <limit velocity="6.5" effort="1000" lower="${-pi*0.6}" upper="${pi*0.45}" />
+            </xacro:if>
+            <xacro:unless value="${reflect - 1}">
+                <limit velocity="6.5" effort="1000" lower="${-pi*0.45}" upper="${pi*0.6}" />
+            </xacro:unless>
+            <dynamics damping="0.1" friction="0.0" />
         </joint>
         <xacro:insert_transmission name="${prefix}_leg_kn_p" />
-	<!-- left knee pitch link -->
+        <!-- knee pitch link -->
         <link name="${prefix}_leg_kn_p_link">
-    	  <collision>
-      	    <origin xyz="0.01 ${reflect * -0.065} -0.145" rpy="0 0 0"/>
-      	    <geometry>
-              <box size="0.11 0.16 0.33" />
-      	    </geometry>
-    	  </collision>
-   	  <visual>
-      	    <origin xyz="0 0 0" rpy="0 0 0"/>
-      	    <geometry>
-              <mesh filename="package://thormang3_description/meshes/robotis_${prefix}_leg_kn_p_link.stl" scale="0.001 0.001 0.001"/>
-      	    </geometry>
-      	    <material name="grey"/>
-    	  </visual>
-          <inertial>
-      	    <origin xyz="-0.002 -0.066 -0.183" rpy="0 0 0"/>
-      	    <mass value="2.401"/>
-      	    <inertia ixx="1.0" ixy="0.0" ixz="0.0" iyy="1.0" iyz="0.0" izz="1.0" />
-            <!-- <inertia ixx="0.01971" ixy="0.00031" ixz="-0.00294" iyy="0.01687" iyz="0.00140" izz="0.00574" /> -->
-    	  </inertial>
-        </link>
-	<!-- left ankle pitch joint -->
+            <collision>
+                <origin xyz="0.01 ${reflect * -0.065} -0.145" rpy="0 0 0"/>
+                <geometry>
+                    <box size="0.11 0.16 0.33" />
+                </geometry>
+            </collision>
+            <visual>
+                <origin xyz="0 0 0" rpy="0 0 0"/>
+                <geometry>
+                    <mesh filename="package://thormang3_description/meshes/robotis_${prefix}_leg_kn_p_link.stl" scale="0.001 0.001 0.001"/>
+                </geometry>
+                <material name="grey"/>
+            </visual>
+              <inertial>
+                <origin xyz="-0.002 -0.066 -0.183" rpy="0 0 0"/>
+                <mass value="2.401"/>
+                <inertia ixx="1.0" ixy="0.0" ixz="0.0" iyy="1.0" iyz="0.0" izz="1.0" />
+                <!-- <inertia ixx="0.01971" ixy="0.00031" ixz="-0.00294" iyy="0.01687" iyz="0.00140" izz="0.00574" /> -->
+            </inertial>
+        </link>
+        <!-- ankle pitch joint -->
         <joint name="${prefix}_leg_an_p" type="revolute">
-          <axis xyz="0 ${-reflect} 0" />
-          <origin xyz="0.0 ${reflect * -0.06} -0.3" rpy="0 0 0"/>
-          <parent link="${prefix}_leg_kn_p_link"/>
-          <child link="${prefix}_leg_an_p_link"/>
-          <limit velocity="6.5" effort="1000" lower="${-pi*0.45}" upper="${pi*0.45}" />
-          <dynamics damping="0.1" friction="0.0" />
+            <axis xyz="0 ${-reflect} 0" />
+            <origin xyz="0.0 ${reflect * -0.06} -0.3" rpy="0 0 0"/>
+            <parent link="${prefix}_leg_kn_p_link"/>
+            <child link="${prefix}_leg_an_p_link"/>
+            <limit velocity="6.5" effort="1000" lower="${-pi*0.45}" upper="${pi*0.45}" />
+            <dynamics damping="0.1" friction="0.0" />
         </joint>
         <xacro:insert_transmission name="${prefix}_leg_an_p" />
-	<!-- left ankle pitch link -->
+        <!-- ankle pitch link -->
         <link name="${prefix}_leg_an_p_link">
 <!--
-    	  <collision>
-      	    <origin xyz="0 0 0" rpy="0 0 0"/>
-      	    <geometry>
+        <collision>
+            <origin xyz="0 0 0" rpy="0 0 0"/>
+            <geometry>
               <box size="0.01 0.01 0.01" />
-      	    </geometry>
-    	  </collision>
+            </geometry>
+        </collision>
 -->
-   	  <visual>
-      	    <origin xyz="0 0 0" rpy="0 0 0"/>
-      	    <geometry>
-              <mesh filename="package://thormang3_description/meshes/robotis_${prefix}_leg_an_p_link.stl" scale="0.001 0.001 0.001"/>
-      	    </geometry>
-      	    <material name="grey"/>
-    	  </visual>
-          <inertial>
-      	    <origin xyz="-0.011 -0.033 0.000" rpy="0 0 0"/>
-      	    <mass value="1.045"/>
-      	    <inertia ixx="1.0" ixy="0.0" ixz="0.0" iyy="1.0" iyz="0.0" izz="1.0" />
-            <!-- <inertia ixx="0.00056" ixy="0.0" ixz="0.0" iyy="0.00168" iyz="0.0" izz="0.00171" /> -->
-    	  </inertial>
-        </link>
-	<!-- left ankle roll joint -->
+            <visual>
+            <origin xyz="0 0 0" rpy="0 0 0"/>
+                <geometry>
+                    <mesh filename="package://thormang3_description/meshes/robotis_${prefix}_leg_an_p_link.stl" scale="0.001 0.001 0.001"/>
+                </geometry>
+                <material name="grey"/>
+            </visual>
+            <inertial>
+                <origin xyz="-0.011 -0.033 0.000" rpy="0 0 0"/>
+                <mass value="1.045"/>
+                <inertia ixx="1.0" ixy="0.0" ixz="0.0" iyy="1.0" iyz="0.0" izz="1.0" />
+                <!-- <inertia ixx="0.00056" ixy="0.0" ixz="0.0" iyy="0.00168" iyz="0.0" izz="0.00171" /> -->
+            </inertial>
+        </link>
+        <!-- ankle roll joint -->
         <joint name="${prefix}_leg_an_r" type="revolute">
-          <axis xyz="1 0 0" />
-          <origin xyz="0.057 ${reflect * -0.033} 0.0" rpy="0 0 0"/>
-          <parent link="${prefix}_leg_an_p_link"/>
-          <child link="${prefix}_leg_an_r_link"/>
-          <limit velocity="6.5" effort="1000" lower="${-pi*0.25}" upper="${pi*0.25}" />
-          <dynamics damping="0.1" friction="0.0" />
+            <axis xyz="1 0 0" />
+            <origin xyz="0.057 ${reflect * -0.033} 0.0" rpy="0 0 0"/>
+            <parent link="${prefix}_leg_an_p_link"/>
+            <child link="${prefix}_leg_an_r_link"/>
+            <limit velocity="6.5" effort="1000" lower="${-pi*0.25}" upper="${pi*0.25}" />
+            <dynamics damping="0.1" friction="0.0" />
         </joint>
         <xacro:insert_transmission name="${prefix}_leg_an_r" />
-	<!-- left ankle roll link -->
+        <!-- ankle roll link -->
         <link name="${prefix}_leg_an_r_link">
-    	  <collision>
-      	    <origin xyz="-0.067 0 -0.02" rpy="0 0 0"/>
-      	    <geometry>
-              <box size="0.17 0.06 0.12" />
-      	    </geometry>
-    	  </collision>
-   	  <visual>
-      	    <origin xyz="0 0 0" rpy="0 0 0"/>
-      	    <geometry>
-              <mesh filename="package://thormang3_description/meshes/robotis_${prefix}_leg_an_r_link.stl" scale="0.001 0.001 0.001"/>
-      	    </geometry>
-      	    <material name="grey"/>
-    	  </visual>
-          <inertial>
-      	    <origin xyz="-0.070 0.000 -0.048" rpy="0 0 0"/>
-      	    <mass value="0.223"/>
-      	    <inertia ixx="1.0" ixy="0.0" ixz="0.0" iyy="1.0" iyz="0.0" izz="1.0" />
-            <!-- <inertia ixx="0.00022" ixy="0.0" ixz="-0.00001" iyy="0.00099" iyz="0.0" izz="0.00091" /> -->
-    	  </inertial>
-        </link>
-	<!-- left ft joint -->
-	<!--use "fixed" revolute joint for FT sensor simulation-->
-	<joint name="${prefix}_leg_ft" type="revolute">
-          <origin xyz="-0.057 0.0 -0.087" rpy="0 0 0"/>
-          <parent link="${prefix}_leg_an_r_link"/>
-          <child link="${prefix}_foot_ft_link"/>
-	  <limit velocity="6.5" effort="1000" lower="0" upper="0" />
-        </joint>
-	<!-- left foot ft link -->
+            <collision>
+                <origin xyz="-0.067 0 -0.02" rpy="0 0 0"/>
+                <geometry>
+                    <box size="0.17 0.06 0.12" />
+                </geometry>
+            </collision>
+           <visual>
+                <origin xyz="0 0 0" rpy="0 0 0"/>
+                <geometry>
+                    <mesh filename="package://thormang3_description/meshes/robotis_${prefix}_leg_an_r_link.stl" scale="0.001 0.001 0.001"/>
+                </geometry>
+                <material name="grey"/>
+            </visual>
+            <inertial>
+                <origin xyz="-0.070 0.000 -0.048" rpy="0 0 0"/>
+                <mass value="0.223"/>
+                <inertia ixx="1.0" ixy="0.0" ixz="0.0" iyy="1.0" iyz="0.0" izz="1.0" />
+                <!-- <inertia ixx="0.00022" ixy="0.0" ixz="-0.00001" iyy="0.00099" iyz="0.0" izz="0.00091" /> -->
+            </inertial>
+        </link>
+        <!-- ft joint -->
+        <!--use "fixed" revolute joint for FT sensor simulation-->
+        <joint name="${prefix}_leg_ft" type="revolute">
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