Commit message: fixed center of mass in legs

File: thormang3_description/urdf/thormang3.structure.leg.xacro (robot description, xacro)
@@ -28,5 +28,5 @@
             </visual>
             <inertial>
-                <origin xyz="0.012 0.000 -0.025" rpy="0 0 0"/>
+                <origin xyz="0.012 ${reflect * 0.000} -0.025" rpy="0 0 0"/>
                 <mass value="0.243"/>
                 <inertia ixx="1.0" ixy="0.0" ixz="0.0" iyy="1.0" iyz="0.0" izz="1.0" />
@@ -62,5 +62,5 @@
             </visual>
             <inertial>
-                <origin xyz="-0.068 0.000 0.000" rpy="0 0 0"/>
+                <origin xyz="-0.068 ${reflect * 0.000} 0.000" rpy="0 0 0"/>
                 <mass value="1.045"/>
                 <inertia ixx="1.0" ixy="0.0" ixz="0.0" iyy="1.0" iyz="0.0" izz="1.0" />
@@ -99,5 +99,5 @@
             </visual>
             <inertial>
-                <origin xyz="0.022 -0.007 -0.168" rpy="0 0 0"/>
+                <origin xyz="0.022 ${reflect * -0.007} -0.168" rpy="0 0 0"/>
                 <mass value="3.095"/>
                 <inertia ixx="1.0" ixy="0.0" ixz="0.0" iyy="1.0" iyz="0.0" izz="1.0" />
@@ -136,5 +136,5 @@
             </visual>
               <inertial>
-                <origin xyz="-0.002 -0.066 -0.183" rpy="0 0 0"/>
+                <origin xyz="-0.002 ${reflect * -0.066} -0.183" rpy="0 0 0"/>
                 <mass value="2.401"/>
                 <inertia ixx="1.0" ixy="0.0" ixz="0.0" iyy="1.0" iyz="0.0" izz="1.0" />
@@ -170,5 +170,5 @@
             </visual>
             <inertial>
-                <origin xyz="-0.011 -0.033 0.000" rpy="0 0 0"/>
+                <origin xyz="-0.011 ${reflect * -0.033} 0.000" rpy="0 0 0"/>
                 <mass value="1.045"/>
                 <inertia ixx="1.0" ixy="0.0" ixz="0.0" iyy="1.0" iyz="0.0" izz="1.0" />
@@ -202,5 +202,5 @@
             </visual>
             <inertial>
-                <origin xyz="-0.070 0.000 -0.048" rpy="0 0 0"/>
+                <origin xyz="-0.070 ${reflect * 0.000} -0.048" rpy="0 0 0"/>
                 <mass value="0.223"/>
                 <inertia ixx="1.0" ixy="0.0" ixz="0.0" iyy="1.0" iyz="0.0" izz="1.0" />
@@ -241,5 +241,5 @@
             </visual>
             <inertial>
-                <origin xyz="0.000 0.009 -0.013" rpy="0 0 0"/>
+                <origin xyz="0.000 ${reflect * 0.009} -0.013" rpy="0 0 0"/>
                 <mass value="1.689"/>
                 <inertia ixx="1.0" ixy="0.0" ixz="0.0" iyy="1.0" iyz="0.0" izz="1.0" />
