Commit message: fixed leg collision

File: thormang3_description/urdf/johnny5.urdf (robot description, URDF)
Before this commit: robot johnny5, 47 links, 46 joints
Links:
- link head_p_link: mass 1.0 -> 0.724
- link head_y_link: mass 1.0 -> 0.087
- link l_leg_hip_p_link: geometry collision box size=0.11 0.16 0.34; visual mesh filename=package://thormang3_description/meshes/robotis_l_leg_hip_p_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 scale=0.001 0.001 0.001
- link r_leg_hip_p_link: geometry collision box size=0.11 0.16 0.34; visual mesh filename=package://thormang3_description/meshes/robotis_r_leg_hip_p_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 scale=0.001 0.001 0.001
Joints:
- joint imu_fixed: origin xyz=0.03 0.0 0.0 rpy=3.14159265359 0.0 3.14159265359 -> xyz=0.03 0.0 0.0 rpy=0.0 0.0 3.14159265359

File: thormang3_description/urdf/thormang3.structure.leg.xacro (robot description, xacro)
@@ -86,7 +86,7 @@
         <link name="${prefix}_leg_hip_p_link">
             <collision>
-                <origin xyz="0 -0.005 -0.145" rpy="0 0 0"/>
-                <geometry>
-                    <box size="0.11 0.16 0.33" />
+                <origin xyz="0 ${reflect * -0.005} -0.135" rpy="0 0 0"/>
+                <geometry>
+                    <box size="0.11 0.16 0.34" />
                 </geometry>
             </collision>
