Commit message: use team hectors multisensor head

File: thormang3_description/urdf/thormang3.structure.head.xacro (robot description, xacro)
@@ -2,4 +2,5 @@
 <robot xmlns:xacro="http://ros.org/wiki/xacro">
     <xacro:property name="pi" value="3.141592654" />
+    <xacro:include filename="$(find hector_components_description)/urdf/hector_multisensor_head.urdf.xacro" />
     <xacro:macro name="thormang3_head" params="parent">
 	<!-- head yaw joint -->
@@ -53,5 +54,5 @@
     	  </collision>
    	  <visual>
-      	    <origin xyz="0 0 0" rpy="0 0 0"/>
+      	    <origin xyz="0 0 0" rpy="${pi*0.5} 0 0"/>
       	    <geometry>
               <mesh filename="package://thormang3_description/meshes/robotis_head_p_link.stl" scale="0.001 0.001 0.001"/>
@@ -65,32 +66,15 @@
     	  </inertial>
         </link>
-	<!-- camera joint -->
-        <joint name="cam" type="fixed">
-          <origin xyz="0.0682 0.045 0.056" rpy="${-pi*0.5} 0 ${-pi*0.5}"/>
+	<!-- multisensor head joint -->
+        <joint name="multisensor_head_link" type="fixed">
+          <origin xyz="0.0 0.042 0.021" rpy="0 0 0"/>
           <parent link="head_p_link"/>
-          <child link="cam_link"/>
+          <child link="head_link"/>
         </joint>
-	<!-- camera link -->
-        <link name="cam_link">
-        </link>
-	<!-- lidar joint -->
-        <joint name="lidar_fixed" type="fixed">
-          <origin xyz="0.0 0.045 0.10675" rpy="0 0 0"/>
-          <parent link="head_p_link"/>
-          <child link="lidar_link"/>
-        </joint>
-	<!-- lidar link -->
-        <link name="lidar_link">
-        </link>
-	<!-- realsense joint -->
-        <joint name="realsense_fixed" type="fixed">
-	  <!--<origin xyz="0.0749 0.02 0.0292" rpy="0 0 0"/>-->
-          <origin xyz="0.0529 -0.009 0.0292" rpy="0 0 0"/>
-          <parent link="head_p_link"/>
-          <child link="realsense_link"/>
-        </joint>
-	<!-- realsense link -->
-        <link name="realsense_link">
-        </link>
+	<hector_multisensor_head_macro parent="head_y_link"  name="head" scaling="0.001">
+	  <origin xyz="0.0 0.0 0.0" rpy="${M_PI*0.5} 0.0 ${M_PI*0.5}"/>
+	  <!-- Calibrated origin of the laser scanner-->
+	  <origin xyz="0.0 0.000323461 0.0127965" rpy="0.0 0.021197 -0.00357142"/>
+	</hector_multisensor_head_macro>
     </xacro:macro>
 </robot>

Commit message: Updated collision model for the head

File: thormang3_description/urdf/thormang3.structure.head.xacro (robot description, xacro)
@@ -17,7 +17,7 @@
         <link name="head_y_link">
     	  <collision>
-      	    <origin xyz="0 0 0" rpy="0 0 0"/>
+      	    <origin xyz="0 0 0.005" rpy="0 0 0"/>
       	    <geometry>
-              <box size="0.07 0.1 0.1" />
+              <box size="0.05 0.1 0.01" />
       	    </geometry>
     	  </collision>
@@ -48,7 +48,7 @@
         <link name="head_p_link">
     	  <collision>
-      	    <origin xyz="0.01 0.045 0.06" rpy="0 0 0"/>
+      	    <origin xyz="0.0 0.045 0.0" rpy="0 0 0"/>
       	    <geometry>
-              <box size="0.13 0.15 0.15" />
+              <box size="0.04 0.1 0.04" />
       	    </geometry>
     	  </collision>

File: thormang3_description/urdf/thormang3.structure.torso.xacro (robot description, xacro)
@@ -59,7 +59,7 @@
   <link name="chest_link">
     <collision>
-      <origin xyz="-0.01 0 0.11" rpy="0 0 0"/>
+      <origin xyz="-0.045 0 0.1" rpy="0 0 0"/>
       <geometry>
-        <box size="0.2 0.25 0.23" />
+        <box size="0.2 0.25 0.20" />
       </geometry>
     </collision>

Commit message: joint limit for hear pitch

File: thormang3_description/urdf/thormang3.structure.head.xacro (robot description, xacro)
@@ -41,5 +41,5 @@
           <parent link="head_y_link"/>
           <child link="head_p_link"/>
-          <limit velocity="6.5" effort="1000" lower="${-pi*0.5}" upper="${pi*0.5}" />
+	  <limit velocity="6.5" effort="1000" lower="-0.745" upper="1.301" />
           <dynamics damping="0.1" friction="0.0" />
         </joint>

Commit message: calibration now included from separat file

File: thormang3_description/urdf/thormang3.structure.head.xacro (robot description, xacro)
@@ -75,5 +75,5 @@
 	  <origin xyz="0.0 0.0 0.0" rpy="${M_PI*0.5} 0.0 ${M_PI*0.5}"/>
 	  <!-- Calibrated origin of the laser scanner-->
-	  <origin xyz="0.0 0.000323461 0.0127965" rpy="0.0 0.021197 -0.00357142"/>
+	   <xacro:include filename="$(find thormang3_description)/calibration/multisensor_head_calibration.urdf.xacro" />
 	</hector_multisensor_head_macro>
     </xacro:macro>

Commit message: added inertial values of head (urdf)

File: thormang3_description/urdf/thormang3.structure.head.xacro (robot description, xacro)
@@ -29,7 +29,7 @@
     	  </visual>
           <inertial>
-      	    <origin xyz="0.0 0.0 0.0" rpy="0 0 0"/>
-      	    <mass value="1.0"/>
-      	    <inertia ixx="1.0" ixy="0.0" ixz="0.0" iyy="1.0" iyz="0.0" izz="1.0" />
+      	    <origin xyz="0.0 -0.002 0.010" rpy="0 0 0"/>
+      	    <mass value="0.087"/>
+      	    <inertia ixx="0.00011" ixy="0.0" ixz="0.0" iyy="0.00003" iyz="0.0" izz="0.00012" />
     	  </inertial>
         </link>
@@ -60,7 +60,7 @@
     	  </visual>
           <inertial>
-      	    <origin xyz="0.0 0.0 0.0" rpy="0 0 0"/>
-      	    <mass value="1.0"/>
-      	    <inertia ixx="1.0" ixy="0.0" ixz="0.0" iyy="1.0" iyz="0.0" izz="1.0" />
+      	    <origin xyz="0.009 0.046 0.022" rpy="0 0 0"/>
+      	    <mass value="0.724"/>
+      	    <inertia ixx="0.00113" ixy="0.00001" ixz="0.0" iyy="0.00114" iyz="0.00002" izz="0.00084" />
     	  </inertial>
         </link>

Commit message: reset inertia to identity matrix in head urdf

File: thormang3_description/urdf/thormang3.structure.head.xacro (robot description, xacro)
@@ -31,5 +31,5 @@
       	    <origin xyz="0.0 -0.002 0.010" rpy="0 0 0"/>
       	    <mass value="0.087"/>
-      	    <inertia ixx="0.00011" ixy="0.0" ixz="0.0" iyy="0.00003" iyz="0.0" izz="0.00012" />
+      	    <inertia ixx="1.0" ixy="0.0" ixz="0.0" iyy="1.0" iyz="0.0" izz="1.0" />
     	  </inertial>
         </link>
@@ -62,5 +62,5 @@
       	    <origin xyz="0.009 0.046 0.022" rpy="0 0 0"/>
       	    <mass value="0.724"/>
-      	    <inertia ixx="0.00113" ixy="0.00001" ixz="0.0" iyy="0.00114" iyz="0.00002" izz="0.00084" />
+      	    <inertia ixx="1.0" ixy="0.0" ixz="0.0" iyy="1.0" iyz="0.0" izz="1.0" />
     	  </inertial>
         </link>

Commit message: clean up

File: thormang3_description/urdf/thormang3.structure.head.xacro (robot description, xacro)
@@ -60,8 +60,6 @@
     	  </visual>
           <inertial>
-      	    <!--<origin xyz="0.009 0.046 0.022" rpy="0 0 0"/>-->
       	    <origin xyz="-0.012 0.044 0.072" rpy="0 0 0"/>
-+      	    <!--<mass value="0.724"/>-->
-+	    <mass value="1.048"/>
+	    <mass value="1.048"/>
       	    <inertia ixx="1.0" ixy="0.0" ixz="0.0" iyy="1.0" iyz="0.0" izz="1.0" />
     	  </inertial>

File: thormang3_description/urdf/thormang3.structure.torso.xacro (robot description, xacro)
@@ -26,8 +26,6 @@
   <link name="pelvis_link">
     <collision>
-      <!--<origin xyz="-0.01 0 0.07" rpy="0 0 0"/>-->
       <origin xyz="0.01 0 0.072" rpy="0 0 0"/>
       <geometry>
-        <!--<box size="0.2 0.25 0.17" />-->
 	<box size="0.2 0.25 0.174" />
       </geometry>
@@ -41,5 +39,4 @@
     </visual>
     <inertial>
-      <!--<origin xyz="-0.011 0.000 0.058" rpy="0 0 0"/>-->
       <origin xyz="0.011 0.000 0.060" rpy="0 0 0"/>
       <mass value="6.869"/>
@@ -52,6 +49,5 @@
     <parent link="pelvis_link"/>
     <child link="chest_link"/>
-    <!--<origin xyz="0 0 0.1705" rpy="0 0 0"/>-->
-    <origin xyz="0 0 0.1795" rpy="0 0 0"/><!--torso 9mm higher because of pelvis upgrade (cf. new .stl)-->
+    <origin xyz="0 0 0.1795" rpy="0 0 0"/>
     <axis xyz="0 0 1"/>
     <limit velocity="6.5" effort="1000" lower="${-pi*0.25}" upper="${pi*0.25}" />
@@ -214,5 +210,4 @@
     </inertial>
   </link>
-  <!--Comment/uncomment the following lines to check center of mass of bacpack housing-->
   <joint name="backpack_fixed" type="fixed">
     <parent link="chest_link"/>
@@ -220,12 +215,4 @@
     <origin xyz="-0.030 -0.123 0.130" rpy="0.0 0.0 0.0"/>
   </joint>
-  <!--<joint name="backpack_test_joint" type="revolute">
-    <parent link="chest_link"/>
-    <child link="backpack_link"/>
-    <origin xyz="-0.030 -0.123 0.130" rpy="0 0 0"/>
-    <axis xyz="1 0 0"/>
-    <limit velocity="6.5" effort="1000" lower="0.0" upper="0.0" />
-    <dynamics damping="0.1" friction="0.0" />
-  </joint>-->
   <!-- power module housing -->
   <link name="power_module_link">
@@ -249,5 +236,4 @@
     </inertial>
   </link>
-  <!--Comment/uncomment the following lines to check center of mass of power module housing-->
   <joint name="power_module_fixed" type="fixed">
     <parent link="pelvis_link"/>
@@ -255,12 +241,4 @@
     <origin xyz="-0.060 -0.068 0.116" rpy="0.0 0.0 0.0"/>
   </joint>
-  <!--<joint name="power_module_test_joint" type="revolute">
-    <parent link="pelvis_link"/>
-    <child link="power_module_link"/>
-    <origin xyz="-0.060 -0.068 0.116" rpy="0 0 0"/>
-    <axis xyz="1 0 0"/>
-    <limit velocity="6.5" effort="1000" lower="0.0" upper="0.0" />
-    <dynamics damping="0.1" friction="0.0" />
-  </joint>-->
   <xacro:thormang3_arm parent="chest_link" prefix="l" reflect="1" />
   <xacro:thormang3_arm parent="chest_link" prefix="r" reflect="-1" />

Commit message: updated head pitch limits

File: thormang3_description/urdf/thormang3.structure.head.xacro (robot description, xacro)
@@ -40,5 +40,5 @@
           <parent link="head_y_link"/>
           <child link="head_p_link"/>
-	  <limit velocity="6.5" effort="1000" lower="-0.745" upper="1.301" />
+	  <limit velocity="6.5" effort="1000" lower="-0.745" upper="0.745" />
           <dynamics damping="0.1" friction="0.0" />
         </joint>
