Commit message: add servos to collision model of the torso

File: thormang3_description/urdf/thormang3.structure.torso.xacro (robot description, xacro)
@@ -61,5 +61,35 @@
       <origin xyz="-0.045 0 0.1" rpy="0 0 0"/>
       <geometry>
-        <box size="0.2 0.25 0.20" />
+        <box size="0.15 0.25 0.20" />
+      </geometry>
+    </collision>
+    <collision>
+      <origin xyz="0 0 0.077" rpy="0 0 0"/>
+      <geometry>
+        <box size="0.2 0.2 0.15" />
+      </geometry>
+    </collision>
+    <collision>
+      <origin xyz="0 0 0.077" rpy="0 0 0"/>
+      <geometry>
+        <box size="0.2 0.2 0.15" />
+      </geometry>
+    </collision>
+    <collision>
+      <origin xyz="0 -0.115 0.16" rpy="0 0 0"/>
+      <geometry>
+        <box size="0.064 0.126 0.064" />
+      </geometry>
+    </collision>
+    <collision>
+      <origin xyz="0 0.115 0.16" rpy="0 0 0"/>
+      <geometry>
+        <box size="0.064 0.126 0.064" />
+      </geometry>
+    </collision>
+    <collision>
+      <origin xyz="0 0.0 0.2125" rpy="0 0 0"/>
+      <geometry>
+        <box size="0.064 0.064 0.03" />
       </geometry>
     </collision>

Commit message: add handles to urdf

File: thormang3_description/urdf/thormang3.structure.torso.xacro (robot description, xacro)
@@ -121,3 +121,50 @@
   <xacro:thormang3_leg parent="pelvis_link" prefix="r" reflect="-1" />
   <xacro:thormang3_head parent="chest_link" />
+  <!-- left handle bar -->
+  <joint name="left_handle_bar" type="fixed">
+    <parent link="pelvis_link"/>
+    <child link="left_handle_bar_link"/>
+    <origin xyz="0.0 0 0.0" rpy="0 0 ${pi}"/>
+  </joint>
+  <!-- left handle bar link -->
+  <link name="left_handle_bar_link">
+    <collision>
+      <origin xyz="0.0375 0.135 0.325" rpy="0 0 0"/>
+      <geometry>
+        <box size="0.285 0.025 0.14" />
+      </geometry>
+      <material name="grey"/>
+    </collision>
+    <visual>
+      <origin xyz="0.0375 0.135 0.325" rpy="0 0 0"/>
+      <geometry>
+        <box size="0.285 0.025 0.14" />
+      </geometry>
+      <material name="grey"/>
+    </visual>
+  </link>
+  <!-- right handle bar -->
+  <joint name="right_handle_bar" type="fixed">
+    <parent link="pelvis_link"/>
+    <child link="right_handle_bar_link"/>
+    <origin xyz="0.0 0 0.0" rpy="0 0 ${pi}"/>
+    <material name="grey"/>
+  </joint>
+  <!-- right handle bar link -->
+  <link name="right_handle_bar_link">
+    <collision>
+      <origin xyz="0.0375 -0.135 0.325" rpy="0 0 0"/>
+      <geometry>
+        <box size="0.285 0.025 0.14" />
+      </geometry>
+      <material name="grey"/>
+    </collision>
+    <visual>
+      <origin xyz="0.0375 -0.135 0.325" rpy="0 0 0"/>
+      <geometry>
+        <box size="0.285 0.025 0.14" />
+      </geometry>
+      <material name="grey"/>
+    </visual>
+  </link>
 </robot>

Commit message: TEMPORARY: adjust torso joint limits

File: thormang3_description/urdf/thormang3.structure.torso.xacro (robot description, xacro)
@@ -52,5 +52,5 @@
     <origin xyz="0 0 0.1705" rpy="0 0 0"/>
     <axis xyz="0 0 1"/>
-    <limit velocity="6.5" effort="1000" lower="${-pi*0.6}" upper="${pi*0.6}" />
+    <limit velocity="6.5" effort="1000" lower="${-pi*0.25}" upper="${pi*0.25}" />
     <dynamics damping="0.1" friction="0.0" />
   </joint>

Commit message: fix handle bars parent link

File: thormang3_description/urdf/thormang3.structure.torso.xacro (robot description, xacro)
@@ -123,5 +123,5 @@
   <!-- left handle bar -->
   <joint name="left_handle_bar" type="fixed">
-    <parent link="pelvis_link"/>
+    <parent link="chest_link"/>
     <child link="left_handle_bar_link"/>
     <origin xyz="0.0 0 0.0" rpy="0 0 ${pi}"/>
@@ -130,5 +130,5 @@
   <link name="left_handle_bar_link">
     <collision>
-      <origin xyz="0.0375 0.135 0.325" rpy="0 0 0"/>
+      <origin xyz="0.0375 0.135 0.155" rpy="0 0 0"/>
       <geometry>
         <box size="0.285 0.025 0.14" />
@@ -137,5 +137,5 @@
     </collision>
     <visual>
-      <origin xyz="0.0375 0.135 0.325" rpy="0 0 0"/>
+      <origin xyz="0.0375 0.135 0.155" rpy="0 0 0"/>
       <geometry>
         <box size="0.285 0.025 0.14" />
@@ -146,5 +146,5 @@
   <!-- right handle bar -->
   <joint name="right_handle_bar" type="fixed">
-    <parent link="pelvis_link"/>
+    <parent link="chest_link"/>
     <child link="right_handle_bar_link"/>
     <origin xyz="0.0 0 0.0" rpy="0 0 ${pi}"/>
@@ -154,5 +154,5 @@
   <link name="right_handle_bar_link">
     <collision>
-      <origin xyz="0.0375 -0.135 0.325" rpy="0 0 0"/>
+      <origin xyz="0.0375 -0.135 0.155" rpy="0 0 0"/>
       <geometry>
         <box size="0.285 0.025 0.14" />
@@ -161,5 +161,5 @@
     </collision>
     <visual>
-      <origin xyz="0.0375 -0.135 0.325" rpy="0 0 0"/>
+      <origin xyz="0.0375 -0.135 0.155" rpy="0 0 0"/>
       <geometry>
         <box size="0.285 0.025 0.14" />

Commit message: handle bars are now part of the chest link

File: thormang3_description/urdf/thormang3.structure.torso.xacro (robot description, xacro)
@@ -94,8 +94,40 @@
       </geometry>
     </collision>
+    <!-- left handle bar -->
+    <collision>
+      <origin xyz="-0.0375 0.135 0.155" rpy="0 0 0"/>
+      <geometry>
+        <box size="0.285 0.025 0.14" />
+      </geometry>
+      <material name="grey"/>
+    </collision>
+    <!-- right handle bar -->
+    <collision>
+      <origin xyz="-0.0375 -0.135 0.155" rpy="0 0 0"/>
+      <geometry>
+        <box size="0.285 0.025 0.14" />
+      </geometry>
+      <material name="grey"/>
+    </collision>
     <visual>
       <origin xyz="0 0 0" rpy="0 0 0"/>
       <geometry>
         <mesh filename="package://thormang3_description/meshes/robotis_chest_link.stl" scale="0.001 0.001 0.001"/>
+      </geometry>
+      <material name="grey"/>
+    </visual>
+    <!-- left handle bar -->
+    <visual>
+      <origin xyz="-0.0375 0.135 0.155" rpy="0 0 0"/>
+      <geometry>
+        <box size="0.285 0.025 0.14" />
+      </geometry>
+      <material name="grey"/>
+    </visual>
+    <!-- right handle bar -->
+    <visual>
+      <origin xyz="-0.0375 -0.135 0.155" rpy="0 0 0"/>
+      <geometry>
+        <box size="0.285 0.025 0.14" />
       </geometry>
       <material name="grey"/>
@@ -121,50 +153,3 @@
   <xacro:thormang3_leg parent="pelvis_link" prefix="r" reflect="-1" />
   <xacro:thormang3_head parent="chest_link" />
-  <!-- left handle bar -->
-  <joint name="left_handle_bar" type="fixed">
-    <parent link="chest_link"/>
-    <child link="left_handle_bar_link"/>
-    <origin xyz="0.0 0 0.0" rpy="0 0 ${pi}"/>
-  </joint>
-  <!-- left handle bar link -->
-  <link name="left_handle_bar_link">
-    <collision>
-      <origin xyz="0.0375 0.135 0.155" rpy="0 0 0"/>
-      <geometry>
-        <box size="0.285 0.025 0.14" />
-      </geometry>
-      <material name="grey"/>
-    </collision>
-    <visual>
-      <origin xyz="0.0375 0.135 0.155" rpy="0 0 0"/>
-      <geometry>
-        <box size="0.285 0.025 0.14" />
-      </geometry>
-      <material name="grey"/>
-    </visual>
-  </link>
-  <!-- right handle bar -->
-  <joint name="right_handle_bar" type="fixed">
-    <parent link="chest_link"/>
-    <child link="right_handle_bar_link"/>
-    <origin xyz="0.0 0 0.0" rpy="0 0 ${pi}"/>
-    <material name="grey"/>
-  </joint>
-  <!-- right handle bar link -->
-  <link name="right_handle_bar_link">
-    <collision>
-      <origin xyz="0.0375 -0.135 0.155" rpy="0 0 0"/>
-      <geometry>
-        <box size="0.285 0.025 0.14" />
-      </geometry>
-      <material name="grey"/>
-    </collision>
-    <visual>
-      <origin xyz="0.0375 -0.135 0.155" rpy="0 0 0"/>
-      <geometry>
-        <box size="0.285 0.025 0.14" />
-      </geometry>
-      <material name="grey"/>
-    </visual>
-  </link>
 </robot>

Commit message: added visual for handle bars

File: thormang3_description/urdf/thormang3.structure.torso.xacro (robot description, xacro)
@@ -119,7 +119,28 @@
     <!-- left handle bar -->
     <visual>
-      <origin xyz="-0.0375 0.135 0.155" rpy="0 0 0"/>
+      <origin xyz="0.095 0.135 0.155" rpy="0 0 0"/>
       <geometry>
-        <box size="0.285 0.025 0.14" />
+        <box size="0.02 0.025 0.14" />
+      </geometry>
+      <material name="grey"/>
+    </visual>
+    <visual>
+      <origin xyz="-0.17 0.135 0.155" rpy="0 0 0"/>
+      <geometry>
+        <box size="0.02 0.025 0.14" />
+      </geometry>
+      <material name="grey"/>
+    </visual>
+    <visual>
+      <origin xyz="-0.0375 0.135 0.215" rpy="0 ${0.5*pi} 0"/>
+      <geometry>
+        <cylinder radius="0.01" length="0.275" />
+      </geometry>
+      <material name="grey"/>
+    </visual>
+    <visual>
+      <origin xyz="-0.0375 0.135 0.095" rpy="0 ${0.5*pi} 0"/>
+      <geometry>
+        <cylinder radius="0.01" length="0.275" />
       </geometry>
       <material name="grey"/>
@@ -127,7 +148,28 @@
     <!-- right handle bar -->
     <visual>
-      <origin xyz="-0.0375 -0.135 0.155" rpy="0 0 0"/>
+      <origin xyz="0.095 -0.135 0.155" rpy="0 0 0"/>
       <geometry>
-        <box size="0.285 0.025 0.14" />
+        <box size="0.02 0.025 0.14" />
+      </geometry>
+      <material name="grey"/>
+    </visual>
+    <visual>
+      <origin xyz="-0.17 -0.135 0.155" rpy="0 0 0"/>
+      <geometry>
+        <box size="0.02 0.025 0.14" />
+      </geometry>
+      <material name="grey"/>
+    </visual>
+    <visual>
+      <origin xyz="-0.0375 -0.135 0.215" rpy="0 ${0.5*pi} 0"/>
+      <geometry>
+        <cylinder radius="0.01" length="0.275" />
+      </geometry>
+      <material name="grey"/>
+    </visual>
+    <visual>
+      <origin xyz="-0.0375 -0.135 0.095" rpy="0 ${0.5*pi} 0"/>
+      <geometry>
+        <cylinder radius="0.01" length="0.275" />
       </geometry>
       <material name="grey"/>

Commit message: new imu orientation

File: thormang3_description/urdf/thormang3.structure.torso.xacro (robot description, xacro)
@@ -186,5 +186,5 @@
     <parent link="pelvis_link"/>
     <child link="imu_link"/>
-    <origin xyz="0.03 0 0.0" rpy="0 0 ${pi}"/>
+    <origin xyz="0.03 0 0.0" rpy="${pi} 0 ${-0.5*pi}"/>
   </joint>
   <link name="imu_link">

Commit message: fixed imu frame and simulated imu is reporting correct linear accelerations and gyro

File: thormang3_description/urdf/thormang3.structure.torso.xacro (robot description, xacro)
@@ -185,5 +185,5 @@
     <parent link="pelvis_link"/>
     <child link="imu_link"/>
-    <origin xyz="0.03 0 0.0" rpy="0 0 ${pi}"/>
+    <origin xyz="0.03 0.0 0.0" rpy="${pi} 0.0 ${pi}"/>
   </joint>
   <link name="imu_link">

Commit message: rotated back imu

File: thormang3_description/urdf/thormang3.structure.torso.xacro (robot description, xacro)
@@ -185,5 +185,5 @@
     <parent link="pelvis_link"/>
     <child link="imu_link"/>
-    <origin xyz="0.03 0.0 0.0" rpy="${pi} 0.0 ${pi}"/>
+    <origin xyz="0.03 0.0 0.0" rpy="0.0 0.0 ${pi}"/>
   </joint>
   <link name="imu_link">

Commit message: added housings without masses (todo) in urdf

File: thormang3_description/urdf/thormang3.structure.torso.xacro (robot description, xacro)
@@ -189,4 +189,76 @@
   <link name="imu_link">
   </link>
+  <!-- backpack housing -->
+  <link name="backpack_link">
+    <visual>
+      <origin xyz="0 0 0" rpy="0 0 0"/>
+      <geometry>
+        <mesh filename="package://thormang3_description/meshes/housing_backpack.stl" scale="0.001 0.001 0.001"/>
+      </geometry>
+      <material name="grey"/>
+    </visual>
+    <collision>
+      <origin xyz="-0.065 0.123 -0.030" rpy="0 0 0"/>
+      <geometry>
+        <box size="0.130 0.260 0.200" />
+      </geometry>
+    </collision>
+    <inertial>
+      <!--TODO measure mass and check center of mass (currently set about in the middle)-->
+      <!--When done, set joint to fixed again (see commented lines below) -->
+      <origin xyz="-0.050 0.123 -0.020" rpy="0 0 0"/>
+      <mass value="4"/>
+      <inertia ixx="1.0" ixy="0.0" ixz="0.0" iyy="1.0" iyz="0.0" izz="1.0" />
+    </inertial>
+  </link>
+  <!--<joint name="backpack_fixed" type="fixed">
+    <parent link="chest_link"/>
+    <child link="backpack_link"/>
+    <origin xyz="-0.030 -0.123 0.130" rpy="0.0 0.0 0.0"/>
+  </joint>-->
+  <joint name="backpack_test_joint" type="revolute">
+    <parent link="chest_link"/>
+    <child link="backpack_link"/>
+    <origin xyz="-0.030 -0.123 0.130" rpy="0 0 0"/>
+    <axis xyz="1 0 0"/>
+    <limit velocity="6.5" effort="1000" lower="0.0" upper="0.0" />
+    <dynamics damping="0.1" friction="0.0" />
+  </joint>
+  <!-- power module housing -->
+  <link name="power_module_link">
+    <visual>
+      <origin xyz="0 0 0" rpy="0 0 0"/>
+      <geometry>
+        <mesh filename="package://thormang3_description/meshes/housing_power_module.stl" scale="0.001 0.001 0.001"/>
+      </geometry>
+      <material name="grey"/>
+    </visual>
+    <collision>
+      <origin xyz="-0.030 0.068 -0.046" rpy="0 0 0"/>
+      <geometry>
+        <box size="0.075 0.150 0.150" />
+      </geometry>
+    </collision>
+    <inertial>
+      <!--TODO measure mass and check center of mass (currently set in the middle)-->
+      <!--When done, set joint to fixed again (see commented lines below) -->
+      <origin xyz="-0.030 0.068 -0.046" rpy="0 0 0"/>
+      <mass value="2"/>
+      <inertia ixx="1.0" ixy="0.0" ixz="0.0" iyy="1.0" iyz="0.0" izz="1.0" />
+    </inertial>
+  </link>
+  <!--<joint name="power_module_fixed" type="fixed">
+    <parent link="pelvis_link"/>
+    <child link="power_module_link"/>
+    <origin xyz="-0.060 -0.068 0.116" rpy="0.0 0.0 0.0"/>
+  </joint>-->
+  <joint name="power_module_test_joint" type="revolute">
+    <parent link="pelvis_link"/>
+    <child link="power_module_link"/>
+    <origin xyz="-0.060 -0.068 0.116" rpy="0 0 0"/>
+    <axis xyz="1 0 0"/>
+    <limit velocity="6.5" effort="1000" lower="0.0" upper="0.0" />
+    <dynamics damping="0.1" friction="0.0" />
+  </joint>
   <xacro:thormang3_arm parent="chest_link" prefix="l" reflect="1" />
   <xacro:thormang3_arm parent="chest_link" prefix="r" reflect="-1" />

Commit message: fixed batteries and power housing positions, removed printing aid from backpack housing

File: thormang3_description/urdf/thormang3.structure.torso.xacro (robot description, xacro)
@@ -26,5 +26,6 @@
   <link name="pelvis_link">
     <collision>
-      <origin xyz="-0.01 0 0.07" rpy="0 0 0"/>
+      <!--<origin xyz="-0.01 0 0.07" rpy="0 0 0"/>-->
+      <origin xyz="0.01 0 0.07" rpy="0 0 0"/>
       <geometry>
         <box size="0.2 0.25 0.17" />
@@ -39,5 +40,6 @@
     </visual>
     <inertial>
-      <origin xyz="-0.011 0.000 0.058" rpy="0 0 0"/>
+      <!--<origin xyz="-0.011 0.000 0.058" rpy="0 0 0"/>-->
+      <origin xyz="0.011 0.000 0.058" rpy="0 0 0"/>
       <mass value="6.869"/>
       <inertia ixx="1.0" ixy="0.0" ixz="0.0" iyy="1.0" iyz="0.0" izz="1.0" />
@@ -50,5 +52,5 @@
     <child link="chest_link"/>
     <!--<origin xyz="0 0 0.1705" rpy="0 0 0"/>-->
-    <origin xyz="0 0 0.1775" rpy="0 0 0"/><!--torso 7mm higher because of pelvis upgrade (cf. new .stl)-->
+    <origin xyz="0 0 0.1755" rpy="0 0 0"/><!--torso 5mm higher because of pelvis upgrade (cf. new .stl)-->
     <axis xyz="0 0 1"/>
     <limit velocity="6.5" effort="1000" lower="${-pi*0.25}" upper="${pi*0.25}" />
@@ -229,5 +231,5 @@
   <link name="power_module_link">
     <visual>
-      <origin xyz="0 0 0" rpy="0 0 0"/>
+      <origin xyz="-0.010 0 0" rpy="0 0 0"/>
       <geometry>
         <mesh filename="package://thormang3_description/meshes/housing_power_module.stl" scale="0.001 0.001 0.001"/>
@@ -236,5 +238,5 @@
     </visual>
     <collision>
-      <origin xyz="-0.030 0.068 -0.046" rpy="0 0 0"/>
+      <origin xyz="-0.040 0.068 -0.046" rpy="0 0 0"/>
       <geometry>
         <box size="0.075 0.150 0.150" />
@@ -244,5 +246,5 @@
       <!--TODO measure mass and check center of mass (currently set in the middle)-->
       <!--When done, set joint to fixed again (see commented lines below) -->
-      <origin xyz="-0.030 0.068 -0.046" rpy="0 0 0"/>
+      <origin xyz="-0.040 0.068 -0.046" rpy="0 0 0"/>
       <mass value="2"/>
       <inertia ixx="1.0" ixy="0.0" ixz="0.0" iyy="1.0" iyz="0.0" izz="1.0" />

Commit message: updated torso in urdf (from 5 to 9 mm spacer)

File: thormang3_description/urdf/thormang3.structure.torso.xacro (robot description, xacro)
@@ -27,7 +27,8 @@
     <collision>
       <!--<origin xyz="-0.01 0 0.07" rpy="0 0 0"/>-->
-      <origin xyz="0.01 0 0.07" rpy="0 0 0"/>
-      <geometry>
-        <box size="0.2 0.25 0.17" />
+      <origin xyz="0.01 0 0.072" rpy="0 0 0"/>
+      <geometry>
+        <!--<box size="0.2 0.25 0.17" />-->
+	<box size="0.2 0.25 0.174" />
       </geometry>
     </collision>
@@ -41,5 +42,5 @@
     <inertial>
       <!--<origin xyz="-0.011 0.000 0.058" rpy="0 0 0"/>-->
-      <origin xyz="0.011 0.000 0.058" rpy="0 0 0"/>
+      <origin xyz="0.011 0.000 0.060" rpy="0 0 0"/>
       <mass value="6.869"/>
       <inertia ixx="1.0" ixy="0.0" ixz="0.0" iyy="1.0" iyz="0.0" izz="1.0" />
@@ -52,5 +53,5 @@
     <child link="chest_link"/>
     <!--<origin xyz="0 0 0.1705" rpy="0 0 0"/>-->
-    <origin xyz="0 0 0.1755" rpy="0 0 0"/><!--torso 5mm higher because of pelvis upgrade (cf. new .stl)-->
+    <origin xyz="0 0 0.1795" rpy="0 0 0"/><!--torso 9mm higher because of pelvis upgrade (cf. new .stl)-->
     <axis xyz="0 0 1"/>
     <limit velocity="6.5" effort="1000" lower="${-pi*0.25}" upper="${pi*0.25}" />

Commit message: updated torso urdf (from 5 to 9mm spacer)

File: thormang3_description/urdf/thormang3.structure.torso.xacro (robot description, xacro)
@@ -26,7 +26,9 @@
   <link name="pelvis_link">
     <collision>
-      <origin xyz="-0.01 0 0.07" rpy="0 0 0"/>
-      <geometry>
-        <box size="0.2 0.25 0.17" />
+      <!--<origin xyz="-0.01 0 0.07" rpy="0 0 0"/>-->
+      <origin xyz="0.01 0 0.072" rpy="0 0 0"/>
+      <geometry>
+        <!--<box size="0.2 0.25 0.17" />-->
+        <box size="0.2 0.25 0.174" />
       </geometry>
     </collision>
@@ -40,11 +42,9 @@
     </visual>
     <inertial>
-      <origin xyz="-0.011 0.000 0.058" rpy="0 0 0"/>
-      <!--<origin xyz="-0.006 0.0 0.061" rpy="0 0 0"/>-->
+      <!--<origin xyz="-0.011 0.000 0.058" rpy="0 0 0"/>-->
+      <origin xyz="0.011 0.000 0.060" rpy="0 0 0"/>
       <mass value="6.869"/>
-      <!--<mass value="6.767"/>-->
       <!--<inertia ixx="1.0" ixy="0.0" ixz="0.0" iyy="1.0" iyz="0.0" izz="1.0" />-->
       <inertia ixx="0.03603" ixy="0.0" ixz="0.00016" iyy="0.02210" iyz="0.0" izz="0.03830" />
-      <!--<inertia ixx="0.059" ixy="0.0" ixz="-0.002" iyy="0.048" iyz="0.0" izz="0.034" />-->
     </inertial>
   </link>
@@ -54,5 +54,5 @@
     <child link="chest_link"/>
     <!--<origin xyz="0 0 0.1705" rpy="0 0 0"/>-->
-    <origin xyz="0 0 0.1775" rpy="0 0 0"/> <!--torso 7mm higher because of pelvis upgrade (cf. new .stl)-->
+    <origin xyz="0 0 0.1795" rpy="0 0 0"/> <!--torso 9mm higher because of pelvis upgrade (cf. new .stl)-->
     <axis xyz="0 0 1"/>
     <limit velocity="6.5" effort="1000" lower="${-pi*0.25}" upper="${pi*0.25}" />

Commit message: updated housings masses and centers of mass

File: thormang3_description/urdf/thormang3.structure.torso.xacro (robot description, xacro)
@@ -182,5 +182,5 @@
       <mass value="5.383"/>
       <inertia ixx="1.0" ixy="0.0" ixz="0.0" iyy="1.0" iyz="0.0" izz="1.0" />
-      <inertia ixx="0.04710" ixy="0.0" ixz="0.04710" iyy="0.02554" iyz="0.0" izz="0.03094" />
+      <!--<inertia ixx="0.04710" ixy="0.0" ixz="0.04710" iyy="0.02554" iyz="0.0" izz="0.03094" />-->
     </inertial>
   </link>
@@ -209,17 +209,16 @@
     </collision>
     <inertial>
-      <!--TODO measure mass and check center of mass (currently set about in the middle)-->
-      <!--When done, set joint to fixed again (see commented lines below) -->
-      <origin xyz="-0.050 0.123 -0.020" rpy="0 0 0"/>
-      <mass value="4"/>
-      <inertia ixx="1.0" ixy="0.0" ixz="0.0" iyy="1.0" iyz="0.0" izz="1.0" />
-    </inertial>
-  </link>
-  <!--<joint name="backpack_fixed" type="fixed">
+      <origin xyz="-0.070 0.118 -0.020" rpy="0 0 0"/> <!-- guessed values -->
+      <mass value="1.280"/> <!--RouterBox with Raspberry Pi = 0.780 kg (measured) + BackPack = about 0.500 kg (guessed)-->
+      <inertia ixx="1.0" ixy="0.0" ixz="0.0" iyy="1.0" iyz="0.0" izz="1.0" />
+    </inertial>
+  </link>
+  <!--Comment/uncomment the following lines to check center of mass of bacpack housing-->
+  <joint name="backpack_fixed" type="fixed">
     <parent link="chest_link"/>
     <child link="backpack_link"/>
     <origin xyz="-0.030 -0.123 0.130" rpy="0.0 0.0 0.0"/>
-  </joint>-->
-  <joint name="backpack_test_joint" type="revolute">
+  </joint>
+  <!--<joint name="backpack_test_joint" type="revolute">
     <parent link="chest_link"/>
     <child link="backpack_link"/>
@@ -228,5 +227,5 @@
     <limit velocity="6.5" effort="1000" lower="0.0" upper="0.0" />
     <dynamics damping="0.1" friction="0.0" />
-  </joint>
+  </joint>-->
   <!-- power module housing -->
   <link name="power_module_link">
@@ -245,17 +244,16 @@
     </collision>
     <inertial>
-      <!--TODO measure mass and check center of mass (currently set in the middle)-->
-      <!--When done, set joint to fixed again (see commented lines below) -->
-      <origin xyz="-0.040 0.068 -0.046" rpy="0 0 0"/>
-      <mass value="2"/>
-      <inertia ixx="1.0" ixy="0.0" ixz="0.0" iyy="1.0" iyz="0.0" izz="1.0" />
-    </inertial>
-  </link>
-  <!--<joint name="power_module_fixed" type="fixed">
+      <origin xyz="-0.035 0.068 -0.046" rpy="0 0 0"/> <!-- guessed values -->
+      <mass value="0.595"/> <!-- measured value -->
+      <inertia ixx="1.0" ixy="0.0" ixz="0.0" iyy="1.0" iyz="0.0" izz="1.0" />
+    </inertial>
+  </link>
+  <!--Comment/uncomment the following lines to check center of mass of power module housing-->
+  <joint name="power_module_fixed" type="fixed">
     <parent link="pelvis_link"/>
     <child link="power_module_link"/>
     <origin xyz="-0.060 -0.068 0.116" rpy="0.0 0.0 0.0"/>
-  </joint>-->
-  <joint name="power_module_test_joint" type="revolute">
+  </joint>
+  <!--<joint name="power_module_test_joint" type="revolute">
     <parent link="pelvis_link"/>
     <child link="power_module_link"/>
@@ -264,5 +262,5 @@
     <limit velocity="6.5" effort="1000" lower="0.0" upper="0.0" />
     <dynamics damping="0.1" friction="0.0" />
-  </joint>
+  </joint>-->
   <xacro:thormang3_arm parent="chest_link" prefix="l" reflect="1" />
   <xacro:thormang3_arm parent="chest_link" prefix="r" reflect="-1" />
