Commit message: added proper base_link in order to meet ROS conventions and get rid of warnings from moveit/KDL

File: thormang3_description/urdf/thormang3.structure.torso.xacro (robot description, xacro)
@@ -13,14 +13,15 @@
       <origin xyz="0 0 0" rpy="0 0 0"/>
       <parent link="world"/>
-      <child link="base"/>
-    </joint>
-    <link name="base">
-    </link>
-    <joint name="base_fixed" type="fixed">
-      <origin xyz="0 0 0.723" rpy="0 0 0"/>
-      <parent link="base"/>
-      <child link="pelvis_link"/>
+      <child link="base_link"/>
     </joint>
   </xacro:if>
+  <!-- fake link without mass -->
+  <link name="base_link">
+  </link>
+  <joint name="base_fixed" type="fixed">
+    <origin xyz="0 0 0" rpy="0 0 0"/>
+    <parent link="base_link"/>
+    <child link="pelvis_link"/>
+  </joint>
   <!-- pelvis_link -->
   <link name="pelvis_link">
@@ -28,5 +29,5 @@
       <origin xyz="0.01 0 0.072" rpy="0 0 0"/>
       <geometry>
-	<box size="0.2 0.25 0.174" />
+        <box size="0.2 0.25 0.174" />
       </geometry>
     </collision>
@@ -182,4 +183,6 @@
   </link>
   <!-- imu joint -->
+  <link name="imu_link">
+  </link>
   <joint name="imu_fixed" type="fixed">
     <parent link="pelvis_link"/>
@@ -187,6 +190,4 @@
     <origin xyz="0.03 0.0 0.0" rpy="0.0 0.0 ${pi}"/>
   </joint>
-  <link name="imu_link">
-  </link>
   <!-- backpack housing -->
   <link name="backpack_link">

Commit message: added collision for sound box

File: thormang3_description/urdf/thormang3.structure.torso.xacro (robot description, xacro)
@@ -94,4 +94,12 @@
       </geometry>
     </collision>
+    <!-- sound box -->
+    <visual>
+      <origin xyz="0.0575 0.0 0.19" rpy="0 0 0"/>
+      <geometry>
+        <box size="0.06 0.27 0.05" />
+      </geometry>
+      <material name="grey"/>
+    </visual>
     <!-- left handle bar -->
     <collision>
