Commit message: adjusted frames because we used different servos in the shoulders

File: thormang3_description/urdf/thormang3.structure.arm.xacro (robot description, xacro)
@@ -7,5 +7,5 @@
         <joint name="l_arm_sh_p1" type="revolute">
           <axis xyz="0 1 0" />
-          <origin xyz="0.0 ${0.152-offset} 0.16" rpy="0 0 0"/>
+          <origin xyz="0.0 ${0.177-offset} 0.16" rpy="0 0 0"/>
           <parent link="${parent}"/>
           <child link="l_arm_sh_p1_link"/>
@@ -306,5 +306,5 @@
         <joint name="r_arm_sh_p1" type="revolute">
           <axis xyz="0 -1 0" />
-          <origin xyz="0.0 ${-0.152+offset} 0.16" rpy="0 0 0"/>
+          <origin xyz="0.0 ${-0.177+offset} 0.16" rpy="0 0 0"/>
           <parent link="${parent}"/>
           <child link="r_arm_sh_p1_link"/>

Commit message: Changed collision geometries of arms to be same as visual

File: thormang3_description/urdf/thormang3.structure.arm.xacro (robot description, xacro)
@@ -17,7 +17,7 @@
         <link name="l_arm_sh_p1_link">
     	  <collision>
-      	    <origin xyz="0 0.03 -0.01" rpy="0 0 0"/>
-      	    <geometry>
-              <box size="0.15 0.1 0.09" />
+      	    <origin xyz="0 0 0" rpy="0 0 0"/>
+      	    <geometry>
+              <mesh filename="package://thormang3_description/meshes/robotis_l_arm_sh_p1_link.stl" scale="0.001 0.001 0.001"/>
       	    </geometry>
     	  </collision>
@@ -49,7 +49,7 @@
         <link name="l_arm_sh_r_link">
     	  <collision>
-      	    <origin xyz="-0.057 0 0" rpy="0 0 0"/>
-      	    <geometry>
-              <box size="0.14 0.09 0.09" />
+      	     <origin xyz="0 0 0" rpy="0 0 0"/>
+      	    <geometry>
+              <mesh filename="package://thormang3_description/meshes/robotis_l_arm_sh_r_link.stl" scale="0.001 0.001 0.001"/>
       	    </geometry>
     	  </collision>
@@ -81,7 +81,7 @@
         <link name="l_arm_sh_p2_link">
     	  <collision>
-      	    <origin xyz="0.01 0.11 0" rpy="0 0 0"/>
-      	    <geometry>
-              <box size="0.1 0.24 0.13" />
+      	    <origin xyz="0 0 0" rpy="0 0 0"/>
+      	    <geometry>
+              <mesh filename="package://thormang3_description/meshes/robotis_l_arm_sh_p2_link.stl" scale="0.001 0.001 0.001"/>
       	    </geometry>
     	  </collision>
@@ -113,7 +113,7 @@
         <link name="l_arm_el_y_link">
     	  <collision>
-      	    <origin xyz="0.08 0.01 -0.057" rpy="0 0 0"/>
-      	    <geometry>
-              <box size="0.17 0.1 0.08" />
+      	    <origin xyz="0 0 0" rpy="0 0 0"/>
+      	    <geometry>
+              <mesh filename="package://thormang3_description/meshes/robotis_l_arm_el_y_link.stl" scale="0.001 0.001 0.001"/>
       	    </geometry>
     	  </collision>
@@ -145,7 +145,7 @@
         <link name="l_arm_wr_r_link">
     	  <collision>
-      	    <origin xyz="0.02 0 0" rpy="0 0 0"/>
-      	    <geometry>
-              <box size="0.05 0.05 0.11" />
+      	    <origin xyz="0 0 0" rpy="0 0 0"/>
+      	    <geometry>
+              <mesh filename="package://thormang3_description/meshes/robotis_l_arm_wr_r_link.stl" scale="0.001 0.001 0.001"/>
       	    </geometry>
     	  </collision>
@@ -177,7 +177,7 @@
         <link name="l_arm_wr_y_link">
     	  <collision>
-      	    <origin xyz="0.03 0 -0.045" rpy="0 0 0"/>
-      	    <geometry>
-              <box size="0.09 0.1 0.09" />
+      	    <origin xyz="0 0 0" rpy="0 0 0"/>
+      	    <geometry>
+              <mesh filename="package://thormang3_description/meshes/robotis_l_arm_wr_y_link.stl" scale="0.001 0.001 0.001"/>
       	    </geometry>
     	  </collision>
@@ -209,7 +209,7 @@
         <link name="l_arm_wr_p_link">
     	  <collision>
-      	    <origin xyz="0.07 0.045 0" rpy="0 0 0"/>
-      	    <geometry>
-              <box size="0.07 0.1 0.06" />
+      	    <origin xyz="0 0 0" rpy="0 0 0"/>
+      	    <geometry>
+              <mesh filename="package://thormang3_description/meshes/robotis_l_arm_wr_p_link.stl" scale="0.001 0.001 0.001"/>
       	    </geometry>
     	  </collision>
@@ -316,7 +316,7 @@
         <link name="r_arm_sh_p1_link">
     	  <collision>
-      	    <origin xyz="0 -0.03 -0.01" rpy="0 0 0"/>
-      	    <geometry>
-              <box size="0.15 0.1 0.09" />
+      	    <origin xyz="0 0 0" rpy="0 0 0"/>
+      	    <geometry>
+              <mesh filename="package://thormang3_description/meshes/robotis_r_arm_sh_p1_link.stl" scale="0.001 0.001 0.001"/>
       	    </geometry>
     	  </collision>
@@ -348,7 +348,7 @@
         <link name="r_arm_sh_r_link">
     	  <collision>
-      	    <origin xyz="-0.057 0 0" rpy="0 0 0"/>
-      	    <geometry>
-              <box size="0.14 0.09 0.09" />
+      	    <origin xyz="0 0 0" rpy="0 0 0"/>
+      	    <geometry>
+              <mesh filename="package://thormang3_description/meshes/robotis_r_arm_sh_r_link.stl" scale="0.001 0.001 0.001"/>
       	    </geometry>
     	  </collision>
@@ -380,7 +380,7 @@
         <link name="r_arm_sh_p2_link">
     	  <collision>
-      	    <origin xyz="0.01 -0.11 0" rpy="0 0 0"/>
-      	    <geometry>
-              <box size="0.1 0.24 0.13" />
+      	    <origin xyz="0 0 0" rpy="0 0 0"/>
+      	    <geometry>
+              <mesh filename="package://thormang3_description/meshes/robotis_r_arm_sh_p2_link.stl" scale="0.001 0.001 0.001"/>
       	    </geometry>
     	  </collision>
@@ -412,7 +412,7 @@
         <link name="r_arm_el_y_link">
     	  <collision>
-      	    <origin xyz="0.08 -0.01 -0.057" rpy="0 0 0"/>
-      	    <geometry>
-              <box size="0.17 0.1 0.08" />
+      	    <origin xyz="0 0 0" rpy="0 0 0"/>
+      	    <geometry>
+              <mesh filename="package://thormang3_description/meshes/robotis_r_arm_el_y_link.stl" scale="0.001 0.001 0.001"/>
       	    </geometry>
     	  </collision>
@@ -444,7 +444,7 @@
         <link name="r_arm_wr_r_link">
     	  <collision>
-      	    <origin xyz="0.02 0 0" rpy="0 0 0"/>
-      	    <geometry>
-              <box size="0.05 0.05 0.11" />
+      	    <origin xyz="0 0 0" rpy="0 0 0"/>
+      	    <geometry>
+              <mesh filename="package://thormang3_description/meshes/robotis_r_arm_wr_r_link.stl" scale="0.001 0.001 0.001"/>
       	    </geometry>
     	  </collision>
@@ -476,7 +476,7 @@
         <link name="r_arm_wr_y_link">
     	  <collision>
-      	    <origin xyz="0.03 0 -0.045" rpy="0 0 0"/>
-      	    <geometry>
-              <box size="0.09 0.1 0.09" />
+      	    <origin xyz="0 0 0" rpy="0 0 0"/>
+      	    <geometry>
+              <mesh filename="package://thormang3_description/meshes/robotis_r_arm_wr_y_link.stl" scale="0.001 0.001 0.001"/>
       	    </geometry>
     	  </collision>
@@ -508,7 +508,7 @@
         <link name="r_arm_wr_p_link">
     	  <collision>
-      	    <origin xyz="0.07 -0.045 0" rpy="0 0 0"/>
-      	    <geometry>
-              <box size="0.07 0.1 0.06" />
+      	    <origin xyz="0 0 0" rpy="0 0 0"/>
+      	    <geometry>
+              <mesh filename="package://thormang3_description/meshes/robotis_r_arm_wr_p_link.stl" scale="0.001 0.001 0.001"/>
       	    </geometry>
     	  </collision>

Commit message: added limits for left arm

File: thormang3_description/urdf/thormang3.structure.arm.xacro (robot description, xacro)
@@ -10,5 +10,5 @@
           <parent link="${parent}"/>
           <child link="l_arm_sh_p1_link"/>
-          <limit velocity="6.5" effort="1000" lower="${-pi*0.5}" upper="${pi*0.5}" />
+          <limit velocity="6.5" effort="1000" lower="-3.6111951066" upper="2.81847847561" />
           <dynamics damping="0.1" friction="0.0" />
         </joint>
@@ -42,5 +42,5 @@
           <parent link="l_arm_sh_p1_link"/>
           <child link="l_arm_sh_r_link"/>
-          <limit velocity="6.5" effort="1000" lower="${-pi*0.5}" upper="${pi*0.5}" />
+          <limit velocity="6.5" effort="1000" lower="-3.09079995355" upper="0.89038382649" />
           <dynamics damping="0.1" friction="0.0" />
         </joint>
@@ -74,5 +74,5 @@
           <parent link="l_arm_sh_r_link"/>
           <child link="l_arm_sh_p2_link"/>
-          <limit velocity="6.5" effort="1000" lower="${-pi*0.5}" upper="${pi*0.5}" />
+          <limit velocity="6.5" effort="1000" lower="-3.108976417" upper="2.26478484267" />
           <dynamics damping="0.1" friction="0.0" />
         </joint>
@@ -106,5 +106,5 @@
           <parent link="l_arm_sh_p2_link"/>
           <child link="l_arm_el_y_link"/>
-          <limit velocity="6.5" effort="1000" lower="${-pi*0.4}" upper="${pi*0.4}" />
+          <limit velocity="6.5" effort="1000" lower="-3.09583228021" upper="0.39169527649" />
           <dynamics damping="0.1" friction="0.0" />
         </joint>
@@ -138,5 +138,5 @@
           <parent link="l_arm_el_y_link"/>
           <child link="l_arm_wr_r_link"/>
-          <limit velocity="6.5" effort="1000" lower="${-pi*0.9}" upper="${pi*0.9}" />
+          <limit velocity="6.5" effort="1000" lower="-4.92581042699" upper="5.78071665106" />
           <dynamics damping="0.1" friction="0.0" />
         </joint>
@@ -170,5 +170,5 @@
           <parent link="l_arm_wr_r_link"/>
           <child link="l_arm_wr_y_link"/>
-          <limit velocity="6.5" effort="1000" lower="${-pi*0.45}" upper="${pi*0.45}" />
+          <limit velocity="6.5" effort="1000" lower="-1.45668540746" upper="1.28462438562" />
           <dynamics damping="0.1" friction="0.0" />
         </joint>
@@ -202,5 +202,5 @@
           <parent link="l_arm_wr_y_link"/>
           <child link="l_arm_wr_p_link"/>
-          <limit velocity="6.5" effort="1000" lower="${-pi*0.45}" upper="${pi*0.45}" />
+          <limit velocity="6.5" effort="1000" lower="-1.34684601987" upper="1.36840018971" />
           <dynamics damping="0.1" friction="0.0" />
         </joint>

Commit message: Revert "added limits for left arm"
This reverts commit d8ea1873f2dd576439aa2b49026324bdb5eab7b3.

File: thormang3_description/urdf/thormang3.structure.arm.xacro (robot description, xacro)
@@ -10,5 +10,5 @@
           <parent link="${parent}"/>
           <child link="l_arm_sh_p1_link"/>
-          <limit velocity="6.5" effort="1000" lower="-3.6111951066" upper="2.81847847561" />
+          <limit velocity="6.5" effort="1000" lower="${-pi*0.5}" upper="${pi*0.5}" />
           <dynamics damping="0.1" friction="0.0" />
         </joint>
@@ -42,5 +42,5 @@
           <parent link="l_arm_sh_p1_link"/>
           <child link="l_arm_sh_r_link"/>
-          <limit velocity="6.5" effort="1000" lower="-3.09079995355" upper="0.89038382649" />
+          <limit velocity="6.5" effort="1000" lower="${-pi*0.5}" upper="${pi*0.5}" />
           <dynamics damping="0.1" friction="0.0" />
         </joint>
@@ -74,5 +74,5 @@
           <parent link="l_arm_sh_r_link"/>
           <child link="l_arm_sh_p2_link"/>
-          <limit velocity="6.5" effort="1000" lower="-3.108976417" upper="2.26478484267" />
+          <limit velocity="6.5" effort="1000" lower="${-pi*0.5}" upper="${pi*0.5}" />
           <dynamics damping="0.1" friction="0.0" />
         </joint>
@@ -106,5 +106,5 @@
           <parent link="l_arm_sh_p2_link"/>
           <child link="l_arm_el_y_link"/>
-          <limit velocity="6.5" effort="1000" lower="-3.09583228021" upper="0.39169527649" />
+          <limit velocity="6.5" effort="1000" lower="${-pi*0.4}" upper="${pi*0.4}" />
           <dynamics damping="0.1" friction="0.0" />
         </joint>
@@ -138,5 +138,5 @@
           <parent link="l_arm_el_y_link"/>
           <child link="l_arm_wr_r_link"/>
-          <limit velocity="6.5" effort="1000" lower="-4.92581042699" upper="5.78071665106" />
+          <limit velocity="6.5" effort="1000" lower="${-pi*0.9}" upper="${pi*0.9}" />
           <dynamics damping="0.1" friction="0.0" />
         </joint>
@@ -170,5 +170,5 @@
           <parent link="l_arm_wr_r_link"/>
           <child link="l_arm_wr_y_link"/>
-          <limit velocity="6.5" effort="1000" lower="-1.45668540746" upper="1.28462438562" />
+          <limit velocity="6.5" effort="1000" lower="${-pi*0.45}" upper="${pi*0.45}" />
           <dynamics damping="0.1" friction="0.0" />
         </joint>
@@ -202,5 +202,5 @@
           <parent link="l_arm_wr_y_link"/>
           <child link="l_arm_wr_p_link"/>
-          <limit velocity="6.5" effort="1000" lower="-1.34684601987" upper="1.36840018971" />
+          <limit velocity="6.5" effort="1000" lower="${-pi*0.45}" upper="${pi*0.45}" />
           <dynamics damping="0.1" friction="0.0" />
         </joint>
