Commit message: Decided to keep things simple and going to add VT hands hard coded. Added xacrodisplay files.

File: thormang3_description/urdf/thormang3.structure.arm.xacro (robot description, xacro)
@@ -3,8 +3,15 @@
     <xacro:property name="pi" value="3.141592654" />
     <xacro:property name="offset" value="0.0" />
-    <!-- Hand 0 description
-    <xacro:include filename="$(find $(arg hand_type_0)_description)/urdf/$(arg hand_type_0).xacro" />-->
-    <!-- Hand 1 description
-    <xacro:include filename="$(find $(arg hand_type_1)_description)/urdf/$(arg hand_type_1).xacro" />-->
+    <xacro:arg name="use_hands" default="true"/>
+    <!-- VT hands description -->
+    <xacro:include filename="$(find thor_vt_hand_description)/urdf/vt_hand_tud.urdf.xacro.xml" />
+    <xacro:macro name="vt_hands_tud_macro">
+    <vt_hand_tud_macro parent="l_arm_wr_p_link" prefix="l" reflect="-1" >
+        <origin xyz="0 0 0" rpy="0 0 0"/>
+    </vt_hand_tud_macro>
+    <vt_hand_tud_macro parent="r_arm_wr_p_link" prefix="r" reflect="1" >
+        <origin xyz="0 0 0" rpy="0 0 0"/>
+    </vt_hand_tud_macro>
+    </xacro:macro>
     <xacro:macro name="thormang3_l_arm" params="parent">
 	<!-- left shoulder pitch 1 joint -->
@@ -213,94 +220,21 @@
         <link name="l_arm_wr_p_link">
     	  <collision>
-      	    <origin xyz="0 0 0" rpy="0 0 0"/>
-      	    <geometry>
-              <mesh filename="package://thormang3_description/meshes/robotis_l_arm_wr_p_link.stl" scale="0.001 0.001 0.001"/>
-      	    </geometry>
-    	  </collision>
-   	  <visual>
-      	    <origin xyz="0 0 0" rpy="0 0 0"/>
-      	    <geometry>
-              <mesh filename="package://thormang3_description/meshes/robotis_l_arm_wr_p_link.stl" scale="0.001 0.001 0.001"/>
-      	    </geometry>
-      	    <material name="grey"/>
-    	  </visual>
-          <inertial>
-      	    <origin xyz="0.065 0.045 0.000" rpy="0 0 0"/>
-      	    <mass value="0.565"/>
+      	    <origin xyz="0.039 0.045 0.000" rpy="${pi/2} ${pi} 0"/>
+      	    <geometry>
+              <mesh filename="package://thormang3_description/meshes/robotis_l_arm_wr_r_link.stl" scale="0.001 0.001 0.001"/>
+      	    </geometry>
+    	  </collision>
+   	  <visual>
+      	    <origin xyz="0.039 0.045 0.000" rpy="${pi/2} ${pi} 0"/>
+      	    <geometry>
+              <mesh filename="package://thormang3_description/meshes/robotis_l_arm_wr_r_link.stl" scale="0.001 0.001 0.001"/>
+      	    </geometry>
+      	    <material name="grey"/>
+    	  </visual>
+          <inertial>
+      	    <origin xyz="0.049 0.045 0.002" rpy="0 0 0"/>
+      	    <mass value="0.087"/>
       	    <inertia ixx="1.0" ixy="0.0" ixz="0.0" iyy="1.0" iyz="0.0" izz="1.0" />
             <!--<inertia ixx="0.00047" ixy="-0.00001" ixz="0.0" iyy="0.00042" iyz="0.0" izz="0.00058" />-->
-    	  </inertial>
-        </link>
-	<!-- left arm gripper joint -->
-        <joint name="l_arm_grip" type="revolute">
-          <axis xyz="0 0 -1" />
-          <origin xyz="0.0877 0.0583 0.0" rpy="0 0 ${4.0*pi/18.0}"/>
-          <parent link="l_arm_wr_p_link"/>
-          <child link="l_arm_grip_link"/>
-          <limit velocity="6.5" effort="1000" lower="0.0" upper="${65.0*pi/180.0}" />
-          <dynamics damping="0.1" friction="0.0" />
-        </joint>
-        <xacro:insert_transmission name="l_arm_grip" />
-	<!-- left arm gripper link -->
-        <link name="l_arm_grip_link">
-   	  <visual>
-      	    <origin xyz="0 0 0" rpy="0 0 0"/>
-      	    <geometry>
-              <mesh filename="package://thormang3_description/meshes/robotis_l_arm_grip_link.stl" scale="0.001 0.001 0.001"/>
-      	    </geometry>
-      	    <material name="grey"/>
-    	  </visual>
-          <inertial>
-      	    <origin xyz="0.031 0.014 0.000" rpy="0 0 0"/>
-      	    <mass value="0.013"/>
-      	    <inertia ixx="1.0" ixy="0.0" ixz="0.0" iyy="1.0" iyz="0.0" izz="1.0" />
-            <!--<inertia ixx="0.0" ixy="0.0" ixz="0.0" iyy="0.00001" iyz="0.0" izz="0.00001" />-->
-    	  </inertial>
-        </link>
-	<!-- left arm gripper 1 joint -->
-        <joint name="l_arm_grip_1" type="revolute">
-          <axis xyz="0 0 1" />
-          <origin xyz="0.0877 0.0317 0.0" rpy="0 0 ${-4.0*pi/18.0}"/>
-          <parent link="l_arm_wr_p_link"/>
-          <child link="l_arm_grip_1_link"/>
-          <limit velocity="6.5" effort="1000" lower="0.0" upper="${65.0*pi/180.0}" />
-          <dynamics damping="0.1" friction="0.0" />
-        </joint>
-        <xacro:insert_transmission name="l_arm_grip_1" />
-	<!-- left arm gripper 1 link -->
-        <link name="l_arm_grip_1_link">
-   	  <visual>
-      	    <origin xyz="0 0 0" rpy="0 0 0"/>
-      	    <geometry>
-              <mesh filename="package://thormang3_description/meshes/robotis_l_arm_grip_1_link.stl" scale="0.001 0.001 0.001"/>
-      	    </geometry>
-      	    <material name="grey"/>
-    	  </visual>
-          <inertial>
-      	    <origin xyz="0.031 -0.014 0.000" rpy="0 0 0"/>
-      	    <mass value="0.013"/>
-      	    <inertia ixx="1.0" ixy="0.0" ixz="0.0" iyy="1.0" iyz="0.0" izz="1.0" />
-            <!--<inertia ixx="0.0" ixy="0.0" ixz="0.0" iyy="0.00001" iyz="0.0" izz="0.00001" />-->
-    	  </inertial>
-        </link>
-	<!-- left end effector -->
-        <joint name="l_arm_end" type="fixed">
-          <origin xyz="0.145 0.045 0" rpy="0 0 0"/>
-          <parent link="l_arm_wr_p_link"/>
-          <child link="l_arm_end_link"/>
-        </joint>
-	<!-- left end effector link -->
-        <link name="l_arm_end_link">
-   	  <visual>
-      	    <origin xyz="0 0 0" rpy="0 0 0"/>
-      	    <geometry>
-              <box size="0.01 0.01 0.01" />
-      	    </geometry>
-      	    <material name="red"/>
-    	  </visual>
-          <inertial>
-      	    <origin xyz="0.0 0.0 0.0" rpy="0 0 0"/>
-      	    <mass value="0.001"/>
-      	    <inertia ixx="1.0" ixy="0.0" ixz="0.0" iyy="1.0" iyz="0.0" izz="1.0" />
     	  </inertial>
         </link>
@@ -512,94 +446,21 @@
         <link name="r_arm_wr_p_link">
     	  <collision>
-      	    <origin xyz="0 0 0" rpy="0 0 0"/>
-      	    <geometry>
-              <mesh filename="package://thormang3_description/meshes/robotis_r_arm_wr_p_link.stl" scale="0.001 0.001 0.001"/>
-      	    </geometry>
-    	  </collision>
-   	  <visual>
-      	    <origin xyz="0 0 0" rpy="0 0 0"/>
-      	    <geometry>
-              <mesh filename="package://thormang3_description/meshes/robotis_r_arm_wr_p_link.stl" scale="0.001 0.001 0.001"/>
-      	    </geometry>
-      	    <material name="grey"/>
-    	  </visual>
-          <inertial>
-      	    <origin xyz="0.065 -0.045 0.000" rpy="0 0 0"/>
-      	    <mass value="0.565"/>
+      	    <origin xyz="0.039 -0.045 0.000" rpy="${-pi/2} ${pi} 0"/>
+      	    <geometry>
+              <mesh filename="package://thormang3_description/meshes/robotis_r_arm_wr_r_link.stl" scale="0.001 0.001 0.001"/>
+      	    </geometry>
+    	  </collision>
+   	  <visual>
+      	    <origin xyz="0.039 -0.045 0.000" rpy="${-pi/2} ${pi} 0"/>
+      	    <geometry>
+              <mesh filename="package://thormang3_description/meshes/robotis_r_arm_wr_r_link.stl" scale="0.001 0.001 0.001"/>
+      	    </geometry>
+      	    <material name="grey"/>
+    	  </visual>
+          <inertial>
+      	    <origin xyz="0.049 -0.045 -0.002" rpy="0 0 0"/>
+      	    <mass value="0.087"/>
       	    <inertia ixx="1.0" ixy="0.0" ixz="0.0" iyy="1.0" iyz="0.0" izz="1.0" />
             <!--<inertia ixx="0.00047" ixy="0.00001" ixz="0.0" iyy="0.00042" iyz="0.0" izz="0.00058" />-->
-    	  </inertial>
-        </link>
-	<!-- right arm gripper joint -->
-        <joint name="r_arm_grip" type="revolute">
-          <axis xyz="0 0 1" />
-          <origin xyz="0.0877 -0.0583 0.0" rpy="0 0 ${-4.0*pi/18.0}"/>
-          <parent link="r_arm_wr_p_link"/>
-          <child link="r_arm_grip_link"/>
-          <limit velocity="6.5" effort="1000" lower="0.0" upper="${65.0*pi/180.0}" />
-          <dynamics damping="0.1" friction="0.0" />
-        </joint>
-        <xacro:insert_transmission name="r_arm_grip" />
-	<!-- right arm gripper link -->
-        <link name="r_arm_grip_link">
-   	  <visual>
-      	    <origin xyz="0 0 0" rpy="0 0 0"/>
-      	    <geometry>
-              <mesh filename="package://thormang3_description/meshes/robotis_r_arm_grip_1_link.stl" scale="0.001 0.001 0.001"/>
-      	    </geometry>
-      	    <material name="grey"/>
-    	  </visual>
-          <inertial>
-      	    <origin xyz="0.031 -0.014 0.000" rpy="0 0 0"/>
-      	    <mass value="0.013"/>
-      	    <inertia ixx="1.0" ixy="0.0" ixz="0.0" iyy="1.0" iyz="0.0" izz="1.0" />
-            <!--<inertia ixx="0.0" ixy="0.0" ixz="0.0" iyy="0.00001" iyz="0.0" izz="0.00001" />-->
-    	  </inertial>
-        </link>
-	<!-- right arm gripper 1 joint -->
-        <joint name="r_arm_grip_1" type="revolute">
-          <axis xyz="0 0 -1" />
-          <origin xyz="0.0877 -0.0317 0.0" rpy="0 0 ${4.0*pi/18.0}"/>
-          <parent link="r_arm_wr_p_link"/>
-          <child link="r_arm_grip_1_link"/>
-          <limit velocity="6.5" effort="1000" lower="0.0" upper="${65.0*pi/180.0}" />
-          <dynamics damping="0.1" friction="0.0" />
-        </joint>
-        <xacro:insert_transmission name="r_arm_grip_1" />
-	<!-- right arm gripper link -->
-        <link name="r_arm_grip_1_link">
-   	  <visual>
-      	    <origin xyz="0 0 0" rpy="0 0 0"/>
-      	    <geometry>
-              <mesh filename="package://thormang3_description/meshes/robotis_r_arm_grip_link.stl" scale="0.001 0.001 0.001"/>
-      	    </geometry>
-      	    <material name="grey"/>
-    	  </visual>
-          <inertial>
-      	    <origin xyz="0.031 0.014 0.000" rpy="0 0 0"/>
-      	    <mass value="0.013"/>
-      	    <inertia ixx="1.0" ixy="0.0" ixz="0.0" iyy="1.0" iyz="0.0" izz="1.0" />
-            <!--<inertia ixx="0.0" ixy="0.0" ixz="0.0" iyy="0.00001" iyz="0.0" izz="0.00001" />-->
-    	  </inertial>
-        </link>
-	<!-- right end effector -->
-        <joint name="r_arm_end" type="fixed">
-          <origin xyz="0.145 -0.045 0" rpy="0 0 0"/>
-          <parent link="r_arm_wr_p_link"/>
-          <child link="r_arm_end_link"/>
-        </joint>
-	<!-- right end effector link -->
-        <link name="r_arm_end_link">
-   	  <visual>
-      	    <origin xyz="0 0 0" rpy="0 0 0"/>
-      	    <geometry>
-              <box size="0.01 0.01 0.01" />
-      	    </geometry>
-      	    <material name="red"/>
-    	  </visual>
-          <inertial>
-      	    <origin xyz="0.0 0.0 0.0" rpy="0 0 0"/>
-      	    <mass value="0.001"/>
-      	    <inertia ixx="1.0" ixy="0.0" ixz="0.0" iyy="1.0" iyz="0.0" izz="1.0" />
     	  </inertial>
         </link>

File: thormang3_description/urdf/thormang3.structure.torso.xacro (robot description, xacro)
@@ -1,5 +1,4 @@
 <?xml version="1.0"?>
-<!-- Revolute-Revolute Manipulator -->
-<robot name="thormang3" xmlns:xacro="http://www.ros.org/wiki/xacro">
+<robot xmlns:xacro="http://www.ros.org/wiki/xacro">
   <!-- some parameters -->
   <xacro:property name="pi" value="3.141592654" />
@@ -87,6 +86,4 @@
   <link name="imu_link">
   </link>
-  <xacro:arg name="hand_type_0" default="no_hand"/>
-  <xacro:arg name="hand_type_0" default="no_hand"/>
   <xacro:thormang3_l_arm parent="chest_link" />
   <xacro:thormang3_r_arm parent="chest_link" />

File: thormang3_description/urdf/thormang3.xacro (robot description, xacro)
@@ -1,6 +1,5 @@
 <?xml version="1.0"?>
-<robot name="thormang3" xmlns:xacro="http://www.ros.org/wiki/xacro">
-  <xacro:arg name="robot_name" default="thormang3"/>
-  <!-- Import all Gazebo-customization elements, including Gazebo colors-->
+<robot name="$(arg robot_name)" xmlns:xacro="http://www.ros.org/wiki/xacro">
+  <!-- Import all Gazebo-customization elements, including Gazebo colors -->
   <xacro:include filename="$(find thor_mang_gazebo)/urdf/thormang3.gazebo" />
   <!-- Import Rviz colors -->

Commit message: Fixed call for vt hand macros

File: thormang3_description/urdf/thormang3.structure.arm.xacro (robot description, xacro)
@@ -6,5 +6,4 @@
     <!-- VT hands description -->
     <xacro:include filename="$(find thor_vt_hand_description)/urdf/vt_hand_tud.urdf.xacro.xml" />
-    <xacro:macro name="vt_hands_tud_macro">
     <vt_hand_tud_macro parent="l_arm_wr_p_link" prefix="l" reflect="-1" >
         <origin xyz="0 0 0" rpy="0 0 0"/>
@@ -13,5 +12,4 @@
         <origin xyz="0 0 0" rpy="0 0 0"/>
     </vt_hand_tud_macro>
-    </xacro:macro>
     <xacro:macro name="thormang3_l_arm" params="parent">
 	<!-- left shoulder pitch 1 joint -->

Commit message: Fixed vt hand pose

File: thormang3_description/urdf/thormang3.structure.arm.xacro (robot description, xacro)
@@ -7,8 +7,8 @@
     <xacro:include filename="$(find thor_vt_hand_description)/urdf/vt_hand_tud.urdf.xacro.xml" />
     <vt_hand_tud_macro parent="l_arm_wr_p_link" prefix="l" reflect="-1" >
-        <origin xyz="0 0 0" rpy="0 0 0"/>
+        <origin xyz="0.05 0.05 0" rpy="0 -1.57 3.14159"/>
     </vt_hand_tud_macro>
     <vt_hand_tud_macro parent="r_arm_wr_p_link" prefix="r" reflect="1" >
-        <origin xyz="0 0 0" rpy="0 0 0"/>
+        <origin xyz="0.05 -0.05 0" rpy="0 1.57 0"/>
     </vt_hand_tud_macro>
     <xacro:macro name="thormang3_l_arm" params="parent">

Commit message: Tuned hand pose

File: thormang3_description/urdf/thormang3.structure.arm.xacro (robot description, xacro)
@@ -7,8 +7,8 @@
     <xacro:include filename="$(find thor_vt_hand_description)/urdf/vt_hand_tud.urdf.xacro.xml" />
     <vt_hand_tud_macro parent="l_arm_wr_p_link" prefix="l" reflect="-1" >
-        <origin xyz="0.05 0.05 0" rpy="0 -1.57 3.14159"/>
+        <origin xyz="0.048 0.068 0" rpy="0 -1.57 3.14159"/>
     </vt_hand_tud_macro>
     <vt_hand_tud_macro parent="r_arm_wr_p_link" prefix="r" reflect="1" >
-        <origin xyz="0.05 -0.05 0" rpy="0 1.57 0"/>
+        <origin xyz="0.048 -0.068 0" rpy="0 1.57 0"/>
     </vt_hand_tud_macro>
     <xacro:macro name="thormang3_l_arm" params="parent">

Commit message: Fixed hand pose

File: thormang3_description/urdf/thormang3.structure.arm.xacro (robot description, xacro)
@@ -7,8 +7,8 @@
     <xacro:include filename="$(find thor_vt_hand_description)/urdf/vt_hand_tud.urdf.xacro.xml" />
     <vt_hand_tud_macro parent="l_arm_wr_p_link" prefix="l" reflect="-1" >
-        <origin xyz="0.048 0.068 0" rpy="0 -1.57 3.14159"/>
+        <origin xyz="0.068 0.045 0" rpy="0 -1.57 3.14159"/>
     </vt_hand_tud_macro>
     <vt_hand_tud_macro parent="r_arm_wr_p_link" prefix="r" reflect="1" >
-        <origin xyz="0.048 -0.068 0" rpy="0 1.57 0"/>
+        <origin xyz="0.068 -0.045 0" rpy="0 1.57 0"/>
     </vt_hand_tud_macro>
     <xacro:macro name="thormang3_l_arm" params="parent">

Commit message: Hands are now optional and auto detected by system

File: thormang3_description/urdf/thormang3.structure.arm.xacro (robot description, xacro)
@@ -3,13 +3,15 @@
     <xacro:property name="pi" value="3.141592654" />
     <xacro:property name="offset" value="0.0" />
-    <xacro:arg name="use_hands" default="true"/>
+    <xacro:arg name="use_hands" default="false"/>
     <!-- VT hands description -->
-    <xacro:include filename="$(find thor_vt_hand_description)/urdf/vt_hand_tud.urdf.xacro.xml" />
-    <vt_hand_tud_macro parent="l_arm_wr_p_link" prefix="l" reflect="-1" >
-        <origin xyz="0.068 0.045 0" rpy="0 -1.57 3.14159"/>
-    </vt_hand_tud_macro>
-    <vt_hand_tud_macro parent="r_arm_wr_p_link" prefix="r" reflect="1" >
-        <origin xyz="0.068 -0.045 0" rpy="0 1.57 0"/>
-    </vt_hand_tud_macro>
+    <xacro:if value="$(arg use_hands)">
+        <xacro:include filename="$(find thor_vt_hand_description)/urdf/vt_hand_tud.urdf.xacro.xml" />
+        <vt_hand_tud_macro parent="l_arm_wr_p_link" prefix="l" reflect="-1" >
+            <origin xyz="0.068 0.045 0" rpy="0 -1.57 3.14159"/>
+        </vt_hand_tud_macro>
+        <vt_hand_tud_macro parent="r_arm_wr_p_link" prefix="r" reflect="1" >
+            <origin xyz="0.068 -0.045 0" rpy="0 1.57 0"/>
+        </vt_hand_tud_macro>
+    </xacro:if>
     <xacro:macro name="thormang3_l_arm" params="parent">
 	<!-- left shoulder pitch 1 joint -->

Commit message: Test with left shoulder link

File: thormang3_description/urdf/thormang3.structure.arm.xacro (robot description, xacro)
@@ -28,7 +28,7 @@
         <link name="l_arm_sh_p1_link">
     	  <collision>
-      	    <origin xyz="0 0 0" rpy="0 0 0"/>
-      	    <geometry>
-              <mesh filename="package://thormang3_description/meshes/robotis_l_arm_sh_p1_link.stl" scale="0.001 0.001 0.001"/>
+      	    <origin xyz="-0.005 0.04 -0.015" rpy="0 0 0"/>
+      	    <geometry>
+              <box size="0.13 0.085 0.09" />
       	    </geometry>
     	  </collision>

Commit message: fixed simple collision geometry

File: thormang3_description/urdf/thormang3.structure.arm.xacro (robot description, xacro)
@@ -28,7 +28,19 @@
         <link name="l_arm_sh_p1_link">
     	  <collision>
-      	    <origin xyz="-0.005 0.04 -0.015" rpy="0 0 0"/>
-      	    <geometry>
-              <box size="0.13 0.085 0.09" />
+      	    <origin xyz="-0.005 0.015 0" rpy="0 0 0"/>
+      	    <geometry>
+              <box size="0.14 0.03 0.06" />
+      	    </geometry>
+    	  </collision>
+          <collision>
+      	    <origin xyz="0.06 0.04 -0.02" rpy="-0.8 0 0"/>
+      	    <geometry>
+              <box size="0.02 0.1 0.05" />
+      	    </geometry>
+    	  </collision>
+          <collision>
+      	    <origin xyz="-0.06 0.04 -0.02" rpy="-0.8 0 0"/>
+      	    <geometry>
+              <box size="0.02 0.1 0.05" />
       	    </geometry>
     	  </collision>
@@ -60,7 +72,7 @@
         <link name="l_arm_sh_r_link">
     	  <collision>
-      	     <origin xyz="0 0 0" rpy="0 0 0"/>
-      	    <geometry>
-              <mesh filename="package://thormang3_description/meshes/robotis_l_arm_sh_r_link.stl" scale="0.001 0.001 0.001"/>
+      	     <origin xyz="-0.055 0.0 0.0" rpy="0 0 0"/>
+      	    <geometry>
+              <box size="0.11 0.06 0.06" />
       	    </geometry>
     	  </collision>
@@ -92,7 +104,7 @@
         <link name="l_arm_sh_p2_link">
     	  <collision>
-      	    <origin xyz="0 0 0" rpy="0 0 0"/>
-      	    <geometry>
-              <mesh filename="package://thormang3_description/meshes/robotis_l_arm_sh_p2_link.stl" scale="0.001 0.001 0.001"/>
+      	    <origin xyz="0.0 0.055 0.0" rpy="0 0 0"/>
+      	    <geometry>
+              <box size="0.06 0.11 0.06" />
       	    </geometry>
     	  </collision>

File: thormang3_description/urdf/thormang3.structure.torso.xacro (robot description, xacro)
@@ -59,5 +59,5 @@
   <link name="chest_link">
     <collision>
-      <origin xyz="-0.01 0 0.11" rpy="0 0 0"/>
+      <origin xyz="-0.04 0 0.1" rpy="0 0 0"/>
       <geometry>
         <box size="0.2 0.25 0.23" />
