Commit message: use reflectance for arm urdf

File: thormang3_description/urdf/thormang3.structure.arm.xacro (robot description, xacro)
@@ -14,19 +14,19 @@
         </vt_hand_tud_macro>
     </xacro:if>
-    <xacro:macro name="thormang3_l_arm" params="parent">
+     <xacro:macro name="thormang3_arm" params="parent prefix reflect">
 	<!-- left shoulder pitch 1 joint -->
-        <joint name="l_arm_sh_p1" type="revolute">
+        <joint name="${prefix}_arm_sh_p1" type="revolute">
           <axis xyz="0 1 0" />
-          <origin xyz="0.0 ${0.177-offset} 0.16" rpy="0 0 0"/>
+          <origin xyz="0.0 ${reflect * 0.177-offset} 0.16" rpy="0 0 0"/>
           <parent link="${parent}"/>
-          <child link="l_arm_sh_p1_link"/>
+          <child link="${prefix}_arm_sh_p1_link"/>
           <limit velocity="6.5" effort="1000" lower="${-pi*0.5}" upper="${pi*0.5}" />
           <dynamics damping="0.1" friction="0.0" />
         </joint>
-        <xacro:insert_transmission name="l_arm_sh_p1" />
+        <xacro:insert_transmission name="${prefix}_arm_sh_p1" />
 	<!-- left shoulder pitch 1 link -->
-        <link name="l_arm_sh_p1_link">
-    	  <collision>
-      	    <origin xyz="-0.005 0.015 0" rpy="0 0 0"/>
+        <link name="${prefix}_arm_sh_p1_link">
+    	  <collision>
+      	    <origin xyz="${reflect * -0.005} ${reflect * 0.015} 0" rpy="0 0 0"/>
       	    <geometry>
               <box size="0.14 0.03 0.06" />
@@ -34,5 +34,5 @@
     	  </collision>
           <collision>
-      	    <origin xyz="0.06 0.04 -0.02" rpy="-0.8 0 0"/>
+      	    <origin xyz="${reflect * 0.06} ${reflect * 0.04} -0.02" rpy="${reflect * -0.8} 0 0"/>
       	    <geometry>
               <box size="0.02 0.1 0.05" />
@@ -40,5 +40,5 @@
     	  </collision>
           <collision>
-      	    <origin xyz="-0.06 0.04 -0.02" rpy="-0.8 0 0"/>
+      	    <origin xyz="${reflect * -0.06} ${reflect * 0.04} -0.02" rpy="${reflect * -0.8} 0 0"/>
       	    <geometry>
               <box size="0.02 0.1 0.05" />
@@ -48,5 +48,5 @@
       	    <origin xyz="0 0 0" rpy="0 0 0"/>
       	    <geometry>
-              <mesh filename="package://thormang3_description/meshes/robotis_l_arm_sh_p1_link.stl" scale="0.001 0.001 0.001"/>
+              <mesh filename="package://thormang3_description/meshes/robotis_${prefix}_arm_sh_p1_link.stl" scale="0.001 0.001 0.001"/>
       	    </geometry>
       	    <material name="grey"/>
@@ -60,17 +60,17 @@
         </link>
 	<!-- left shoulder roll joint -->
-        <joint name="l_arm_sh_r" type="revolute">
+        <joint name="${prefix}_arm_sh_r" type="revolute">
           <axis xyz="-1 0 0" />
-          <origin xyz="0.057 0.060 -0.039" rpy="0 0 0"/>
-          <parent link="l_arm_sh_p1_link"/>
-          <child link="l_arm_sh_r_link"/>
+          <origin xyz="${reflect * 0.057} ${reflect * 0.060} -0.039" rpy="0 0 0"/>
+          <parent link="${prefix}_arm_sh_p1_link"/>
+          <child link="${prefix}_arm_sh_r_link"/>
           <limit velocity="6.5" effort="1000" lower="${-pi*0.5}" upper="${pi*0.5}" />
           <dynamics damping="0.1" friction="0.0" />
         </joint>
-        <xacro:insert_transmission name="l_arm_sh_r" />
+        <xacro:insert_transmission name="${prefix}_arm_sh_r" />
 	<!-- left shoulder roll link -->
-        <link name="l_arm_sh_r_link">
-    	  <collision>
-      	     <origin xyz="-0.055 0.0 0.0" rpy="0 0 0"/>
+        <link name="${prefix}_arm_sh_r_link">
+    	  <collision>
+      	     <origin xyz="${reflect * -0.055} 0.0 0.0" rpy="0 0 0"/>
       	    <geometry>
               <box size="0.11 0.06 0.06" />
@@ -80,5 +80,5 @@
       	    <origin xyz="0 0 0" rpy="0 0 0"/>
       	    <geometry>
-              <mesh filename="package://thormang3_description/meshes/robotis_l_arm_sh_r_link.stl" scale="0.001 0.001 0.001"/>
+              <mesh filename="package://thormang3_description/meshes/robotis_${prefix}_arm_sh_r_link.stl" scale="0.001 0.001 0.001"/>
       	    </geometry>
       	    <material name="grey"/>
@@ -92,25 +92,25 @@
         </link>
 	<!-- left shoulder pitch 2 joint -->
-        <joint name="l_arm_sh_p2" type="revolute">
+        <joint name="${prefix}_arm_sh_p2" type="revolute">
           <axis xyz="0 1 0" />
-          <origin xyz="-0.057 0.033 0.0" rpy="0 0 0"/>
-          <parent link="l_arm_sh_r_link"/>
-          <child link="l_arm_sh_p2_link"/>
+          <origin xyz="${reflect * -0.057} ${reflect * 0.033} 0.0" rpy="0 0 0"/>
+          <parent link="${prefix}_arm_sh_r_link"/>
+          <child link="${prefix}_arm_sh_p2_link"/>
           <limit velocity="6.5" effort="1000" lower="${-pi*0.5}" upper="${pi*0.5}" />
           <dynamics damping="0.1" friction="0.0" />
         </joint>
-        <xacro:insert_transmission name="l_arm_sh_p2" />
+        <xacro:insert_transmission name="${prefix}_arm_sh_p2" />
 	<!-- left shoulder pitch2 link -->
-        <link name="l_arm_sh_p2_link">
-    	  <collision>
-      	    <origin xyz="0.0 0.055 0.0" rpy="0 0 0"/>
-      	    <geometry>
-              <box size="0.06 0.11 0.06" />
-      	    </geometry>
-    	  </collision>
-   	  <visual>
-      	    <origin xyz="0 0 0" rpy="0 0 0"/>
-      	    <geometry>
-              <mesh filename="package://thormang3_description/meshes/robotis_l_arm_sh_p2_link.stl" scale="0.001 0.001 0.001"/>
+        <link name="${prefix}_arm_sh_p2_link">
+    	  <collision>
+      	    <origin xyz="0.0 ${reflect * 0.055} 0.0" rpy="0 0 0"/>
+      	    <geometry>
+              <box size="0.06 0.14 0.06" />
+      	    </geometry>
+    	  </collision>
+   	  <visual>
+      	    <origin xyz="0 0 0" rpy="0 0 0"/>
+      	    <geometry>
+              <mesh filename="package://thormang3_description/meshes/robotis_${prefix}_arm_sh_p2_link.stl" scale="0.001 0.001 0.001"/>
       	    </geometry>
       	    <material name="grey"/>
@@ -124,25 +124,25 @@
         </link>
 	<!-- left elbow yaw joint -->
-        <joint name="l_arm_el_y" type="revolute">
+        <joint name="${prefix}_arm_el_y" type="revolute">
           <axis xyz="0 0 -1" />
-          <origin xyz="0.030 0.187 0.057" rpy="0 0 0"/>
-          <parent link="l_arm_sh_p2_link"/>
-          <child link="l_arm_el_y_link"/>
+          <origin xyz="${reflect * 0.030} ${reflect * 0.187} 0.057" rpy="0 0 0"/>
+          <parent link="${prefix}_arm_sh_p2_link"/>
+          <child link="${prefix}_arm_el_y_link"/>
           <limit velocity="6.5" effort="1000" lower="${-pi*0.4}" upper="${pi*0.4}" />
           <dynamics damping="0.1" friction="0.0" />
         </joint>
-        <xacro:insert_transmission name="l_arm_el_y" />
+        <xacro:insert_transmission name="${prefix}_arm_el_y" />
 	<!-- left elbow yaw link -->
-        <link name="l_arm_el_y_link">
-    	  <collision>
-      	    <origin xyz="0 0 0" rpy="0 0 0"/>
-      	    <geometry>
-              <mesh filename="package://thormang3_description/meshes/robotis_l_arm_el_y_link.stl" scale="0.001 0.001 0.001"/>
-      	    </geometry>
-    	  </collision>
-   	  <visual>
-      	    <origin xyz="0 0 0" rpy="0 0 0"/>
-      	    <geometry>
-              <mesh filename="package://thormang3_description/meshes/robotis_l_arm_el_y_link.stl" scale="0.001 0.001 0.001"/>
+        <link name="${prefix}_arm_el_y_link">
+    	  <collision>
+      	    <origin xyz="0 0 0" rpy="0 0 0"/>
+      	    <geometry>
+              <mesh filename="package://thormang3_description/meshes/robotis_${prefix}_arm_el_y_link.stl" scale="0.001 0.001 0.001"/>
+      	    </geometry>
+    	  </collision>
+   	  <visual>
+      	    <origin xyz="0 0 0" rpy="0 0 0"/>
+      	    <geometry>
+              <mesh filename="package://thormang3_description/meshes/robotis_${prefix}_arm_el_y_link.stl" scale="0.001 0.001 0.001"/>
       	    </geometry>
       	    <material name="grey"/>
@@ -156,25 +156,25 @@
         </link>
 	<!-- left wrist roll joint -->
-        <joint name="l_arm_wr_r" type="revolute">
+        <joint name="${prefix}_arm_wr_r" type="revolute">
           <axis xyz="1 0 0" />
-          <origin xyz="0.171 0.030 -0.057" rpy="0 0 0"/>
-          <parent link="l_arm_el_y_link"/>
-          <child link="l_arm_wr_r_link"/>
+          <origin xyz="0.171 ${reflect * 0.030} -0.057" rpy="0 0 0"/>
+          <parent link="${prefix}_arm_el_y_link"/>
+          <child link="${prefix}_arm_wr_r_link"/>
           <limit velocity="6.5" effort="1000" lower="${-pi*0.9}" upper="${pi*0.9}" />
           <dynamics damping="0.1" friction="0.0" />
         </joint>
-        <xacro:insert_transmission name="l_arm_wr_r" />
+        <xacro:insert_transmission name="${prefix}_arm_wr_r" />
 	<!-- left wrist roll link -->
-        <link name="l_arm_wr_r_link">
-    	  <collision>
-      	    <origin xyz="0 0 0" rpy="0 0 0"/>
-      	    <geometry>
-              <mesh filename="package://thormang3_description/meshes/robotis_l_arm_wr_r_link.stl" scale="0.001 0.001 0.001"/>
-      	    </geometry>
-    	  </collision>
-   	  <visual>
-      	    <origin xyz="0 0 0" rpy="0 0 0"/>
-      	    <geometry>
-              <mesh filename="package://thormang3_description/meshes/robotis_l_arm_wr_r_link.stl" scale="0.001 0.001 0.001"/>
+        <link name="${prefix}_arm_wr_r_link">
+    	  <collision>
+      	    <origin xyz="0 0 0" rpy="0 0 0"/>
+      	    <geometry>
+              <mesh filename="package://thormang3_description/meshes/robotis_${prefix}_arm_wr_r_link.stl" scale="0.001 0.001 0.001"/>
+      	    </geometry>
+    	  </collision>
+   	  <visual>
+      	    <origin xyz="0 0 0" rpy="0 0 0"/>
+      	    <geometry>
+              <mesh filename="package://thormang3_description/meshes/robotis_${prefix}_arm_wr_r_link.stl" scale="0.001 0.001 0.001"/>
       	    </geometry>
       	    <material name="grey"/>
@@ -188,25 +188,25 @@
         </link>
 	<!-- left wrist yaw joint -->
-        <joint name="l_arm_wr_y" type="revolute">
+        <joint name="${prefix}_arm_wr_y" type="revolute">
           <axis xyz="0 0 -1" />
           <origin xyz="0.039 0.0 0.045" rpy="0 0 0"/>
-          <parent link="l_arm_wr_r_link"/>
-          <child link="l_arm_wr_y_link"/>
+          <parent link="${prefix}_arm_wr_r_link"/>
+          <child link="${prefix}_arm_wr_y_link"/>
           <limit velocity="6.5" effort="1000" lower="${-pi*0.45}" upper="${pi*0.45}" />
           <dynamics damping="0.1" friction="0.0" />
         </joint>
-        <xacro:insert_transmission name="l_arm_wr_y" />
+        <xacro:insert_transmission name="${prefix}_arm_wr_y" />
 	<!-- left wrist yaw link -->
-        <link name="l_arm_wr_y_link">
-    	  <collision>
-      	    <origin xyz="0 0 0" rpy="0 0 0"/>
-      	    <geometry>
-              <mesh filename="package://thormang3_description/meshes/robotis_l_arm_wr_y_link.stl" scale="0.001 0.001 0.001"/>
-      	    </geometry>
-    	  </collision>
-   	  <visual>
-      	    <origin xyz="0 0 0" rpy="0 0 0"/>
-      	    <geometry>
-              <mesh filename="package://thormang3_description/meshes/robotis_l_arm_wr_y_link.stl" scale="0.001 0.001 0.001"/>
+        <link name="${prefix}_arm_wr_y_link">
+    	  <collision>
+      	    <origin xyz="0 0 0" rpy="0 0 0"/>
+      	    <geometry>
+              <mesh filename="package://thormang3_description/meshes/robotis_${prefix}_arm_wr_y_link.stl" scale="0.001 0.001 0.001"/>
+      	    </geometry>
+    	  </collision>
+   	  <visual>
+      	    <origin xyz="0 0 0" rpy="0 0 0"/>
+      	    <geometry>
+              <mesh filename="package://thormang3_description/meshes/robotis_${prefix}_arm_wr_y_link.stl" scale="0.001 0.001 0.001"/>
       	    </geometry>
       	    <material name="grey"/>
@@ -220,25 +220,25 @@
         </link>
 	<!-- left wrist pitch joint -->
-        <joint name="l_arm_wr_p" type="revolute">
+        <joint name="${prefix}_arm_wr_p" type="revolute">
           <axis xyz="0 -1 0" />
-          <origin xyz="0.045 -0.045 -0.045" rpy="0 0 0"/>
-          <parent link="l_arm_wr_y_link"/>
-          <child link="l_arm_wr_p_link"/>
+          <origin xyz="0.045 ${reflect * -0.045} -0.045" rpy="0 0 0"/>
+          <parent link="${prefix}_arm_wr_y_link"/>
+          <child link="${prefix}_arm_wr_p_link"/>
           <limit velocity="6.5" effort="1000" lower="${-pi*0.45}" upper="${pi*0.45}" />
           <dynamics damping="0.1" friction="0.0" />
         </joint>
-        <xacro:insert_transmission name="l_arm_wr_p" />
+        <xacro:insert_transmission name="${prefix}_arm_wr_p" />
 	<!-- left wrist pitch link -->
-        <link name="l_arm_wr_p_link">
-    	  <collision>
-      	    <origin xyz="0.039 0.045 0.000" rpy="${pi/2} ${pi} 0"/>
-      	    <geometry>
-              <mesh filename="package://thormang3_description/meshes/robotis_l_arm_wr_r_link.stl" scale="0.001 0.001 0.001"/>
-      	    </geometry>
-    	  </collision>
-   	  <visual>
-      	    <origin xyz="0.039 0.045 0.000" rpy="${pi/2} ${pi} 0"/>
-      	    <geometry>
-              <mesh filename="package://thormang3_description/meshes/robotis_l_arm_wr_r_link.stl" scale="0.001 0.001 0.001"/>
+        <link name="${prefix}_arm_wr_p_link">
+    	  <collision>
+      	    <origin xyz="0.039 ${reflect * 0.045} 0.000" rpy="${pi/2} ${pi} 0"/>
+      	    <geometry>
+              <mesh filename="package://thormang3_description/meshes/robotis_${prefix}_arm_wr_r_link.stl" scale="0.001 0.001 0.001"/>
+      	    </geometry>
+    	  </collision>
+   	  <visual>
+      	    <origin xyz="0.039 ${reflect * 0.045} 0.000" rpy="${pi/2} ${pi} 0"/>
+      	    <geometry>
+              <mesh filename="package://thormang3_description/meshes/robotis_${prefix}_arm_wr_r_link.stl" scale="0.001 0.001 0.001"/>
       	    </geometry>
       	    <material name="grey"/>
@@ -252,229 +252,3 @@
         </link>
     </xacro:macro>
-    <xacro:macro name="thormang3_r_arm" params="parent">
-	<!-- right shoulder pitch 1 joint -->
-        <joint name="r_arm_sh_p1" type="revolute">
-          <axis xyz="0 -1 0" />
-          <origin xyz="0.0 ${-0.177+offset} 0.16" rpy="0 0 0"/>
-          <parent link="${parent}"/>
-          <child link="r_arm_sh_p1_link"/>
-          <limit velocity="6.5" effort="1000" lower="${-pi*0.5}" upper="${pi*0.5}" />
-          <dynamics damping="0.1" friction="0.0" />
-        </joint>
-        <xacro:insert_transmission name="r_arm_sh_p1" />
-	<!-- right shoulder pitch 1 link -->
-        <link name="r_arm_sh_p1_link">
-    	  <collision>
-      	    <origin xyz="0 0 0" rpy="0 0 0"/>
-      	    <geometry>
-              <mesh filename="package://thormang3_description/meshes/robotis_r_arm_sh_p1_link.stl" scale="0.001 0.001 0.001"/>
-      	    </geometry>
-    	  </collision>
-   	  <visual>
-      	    <origin xyz="0 0 0" rpy="0 0 0"/>
-      	    <geometry>
-              <mesh filename="package://thormang3_description/meshes/robotis_r_arm_sh_p1_link.stl" scale="0.001 0.001 0.001"/>
-      	    </geometry>
-      	    <material name="grey"/>
-    	  </visual>
-          <inertial>
-      	    <origin xyz="-0.003 -0.020 -0.005" rpy="0 0 0"/>
-      	    <mass value="0.194"/>
-      	    <inertia ixx="1.0" ixy="0.0" ixz="0.0" iyy="1.0" iyz="0.0" izz="1.0" />
-            <!--<inertia ixx="0.00018" ixy="0.0" ixz="0.0" iyy="0.00058" iyz="-0.00004" izz="0.00057" />-->
-    	  </inertial>
-        </link>
-	<!-- right shoulder roll joint -->
-        <joint name="r_arm_sh_r" type="revolute">
-          <axis xyz="-1 0 0" />
-          <origin xyz="0.057 -0.060 -0.039" rpy="0 0 0"/>
-          <parent link="r_arm_sh_p1_link"/>
-          <child link="r_arm_sh_r_link"/>
-          <limit velocity="6.5" effort="1000" lower="${-pi*0.5}" upper="${pi*0.5}" />
-          <dynamics damping="0.1" friction="0.0" />
-        </joint>
-        <xacro:insert_transmission name="r_arm_sh_r" />
-	<!-- right shoulder roll link -->
-        <link name="r_arm_sh_r_link">
-    	  <collision>
-      	    <origin xyz="0 0 0" rpy="0 0 0"/>
-      	    <geometry>
-              <mesh filename="package://thormang3_description/meshes/robotis_r_arm_sh_r_link.stl" scale="0.001 0.001 0.001"/>
-      	    </geometry>
-    	  </collision>
-   	  <visual>
-      	    <origin xyz="0 0 0" rpy="0 0 0"/>
-      	    <geometry>
-              <mesh filename="package://thormang3_description/meshes/robotis_r_arm_sh_r_link.stl" scale="0.001 0.001 0.001"/>
-      	    </geometry>
-      	    <material name="grey"/>
-    	  </visual>
-          <inertial>
-      	    <origin xyz="-0.060 -0.002 0.000" rpy="0 0 0"/>
-      	    <mass value="0.875"/>
-      	    <inertia ixx="1.0" ixy="0.0" ixz="0.0" iyy="1.0" iyz="0.0" izz="1.0" />
-            <!--<inertia ixx="0.00043" ixy="0.0" ixz="0.0" iyy="0.00112" iyz="0.0" izz="0.00113" />-->
-    	  </inertial>
-        </link>
-	<!-- right shoulder pitch 2 joint -->
-        <joint name="r_arm_sh_p2" type="revolute">
-          <axis xyz="0 -1 0" />
-          <origin xyz="-0.057 -0.033 0.0" rpy="0 0 0"/>
-          <parent link="r_arm_sh_r_link"/>
-          <child link="r_arm_sh_p2_link"/>
-          <limit velocity="6.5" effort="1000" lower="${-pi*0.5}" upper="${pi*0.5}" />
-          <dynamics damping="0.1" friction="0.0" />
-        </joint>
-        <xacro:insert_transmission name="r_arm_sh_p2" />
-	<!-- right shoulder pitch2 link -->
-        <link name="r_arm_sh_p2_link">
-    	  <collision>
-      	    <origin xyz="0 0 0" rpy="0 0 0"/>
-      	    <geometry>
-              <mesh filename="package://thormang3_description/meshes/robotis_r_arm_sh_p2_link.stl" scale="0.001 0.001 0.001"/>
-      	    </geometry>
-    	  </collision>
-   	  <visual>
-      	    <origin xyz="0 0 0" rpy="0 0 0"/>
-      	    <geometry>
-              <mesh filename="package://thormang3_description/meshes/robotis_r_arm_sh_p2_link.stl" scale="0.001 0.001 0.001"/>
-      	    </geometry>
-      	    <material name="grey"/>
-    	  </visual>
-          <inertial>
-      	    <origin xyz="0.000 -0.073 0.000" rpy="0 0 0"/>
-      	    <mass value="1.122"/>
-      	    <inertia ixx="1.0" ixy="0.0" ixz="0.0" iyy="1.0" iyz="0.0" izz="1.0" />
-            <!--<inertia ixx="0.00277" ixy="0.00002" ixz="-0.00001" iyy="0.00090" iyz="0.00004" izz="0.00255" />-->
-    	  </inertial>
-        </link>
-	<!-- right elbow yaw joint -->
-        <joint name="r_arm_el_y" type="revolute">
-          <axis xyz="0 0 -1" />
-          <origin xyz="0.030 -0.187 0.057" rpy="0 0 0"/>
-          <parent link="r_arm_sh_p2_link"/>
-          <child link="r_arm_el_y_link"/>
-          <limit velocity="6.5" effort="1000" lower="${-pi*0.4}" upper="${pi*0.4}" />
-          <dynamics damping="0.1" friction="0.0" />
-        </joint>
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
File: thormang3_description/urdf/thormang3.structure.torso.xacro (robot description, xacro)
@@ -116,6 +116,6 @@
   <link name="imu_link">
   </link>
-  <xacro:thormang3_l_arm parent="chest_link" />
-  <xacro:thormang3_r_arm parent="chest_link" />
+  <xacro:thormang3_arm parent="chest_link" prefix="l" reflect="1" />
+  <xacro:thormang3_arm parent="chest_link" prefix="r" reflect="-1" />
   <xacro:thormang3_l_leg parent="pelvis_link" />
   <xacro:thormang3_r_leg parent="pelvis_link" />
