Commit message: use simple collision model for arms

File: thormang3_description/urdf/thormang3.structure.arm.xacro (robot description, xacro)
@@ -15,5 +15,5 @@
     </xacro:if>
      <xacro:macro name="thormang3_arm" params="parent prefix reflect">
-	<!-- left shoulder pitch 1 joint -->
+	<!-- shoulder pitch 1 joint -->
         <joint name="${prefix}_arm_sh_p1" type="revolute">
           <axis xyz="0 1 0" />
@@ -25,5 +25,5 @@
         </joint>
         <xacro:insert_transmission name="${prefix}_arm_sh_p1" />
-	<!-- left shoulder pitch 1 link -->
+	<!-- shoulder pitch 1 link -->
         <link name="${prefix}_arm_sh_p1_link">
     	  <collision>
@@ -59,8 +59,8 @@
     	  </inertial>
         </link>
-	<!-- left shoulder roll joint -->
+	<!-- shoulder roll joint -->
         <joint name="${prefix}_arm_sh_r" type="revolute">
           <axis xyz="-1 0 0" />
-          <origin xyz="${reflect * 0.057} ${reflect * 0.060} -0.039" rpy="0 0 0"/>
+          <origin xyz="0.057 ${reflect * 0.060} -0.039" rpy="0 0 0"/>
           <parent link="${prefix}_arm_sh_p1_link"/>
           <child link="${prefix}_arm_sh_r_link"/>
@@ -69,8 +69,8 @@
         </joint>
         <xacro:insert_transmission name="${prefix}_arm_sh_r" />
-	<!-- left shoulder roll link -->
+	<!-- shoulder roll link -->
         <link name="${prefix}_arm_sh_r_link">
     	  <collision>
-      	     <origin xyz="${reflect * -0.055} 0.0 0.0" rpy="0 0 0"/>
+      	     <origin xyz="-0.055 0.0 0.0" rpy="0 0 0"/>
       	    <geometry>
               <box size="0.11 0.06 0.06" />
@@ -91,8 +91,8 @@
     	  </inertial>
         </link>
-	<!-- left shoulder pitch 2 joint -->
+	<!-- shoulder pitch 2 joint -->
         <joint name="${prefix}_arm_sh_p2" type="revolute">
           <axis xyz="0 1 0" />
-          <origin xyz="${reflect * -0.057} ${reflect * 0.033} 0.0" rpy="0 0 0"/>
+          <origin xyz="-0.057 ${reflect * 0.033} 0.0" rpy="0 0 0"/>
           <parent link="${prefix}_arm_sh_r_link"/>
           <child link="${prefix}_arm_sh_p2_link"/>
@@ -101,10 +101,28 @@
         </joint>
         <xacro:insert_transmission name="${prefix}_arm_sh_p2" />
-	<!-- left shoulder pitch2 link -->
+	<!-- shoulder pitch2 link -->
         <link name="${prefix}_arm_sh_p2_link">
     	  <collision>
-      	    <origin xyz="0.0 ${reflect * 0.055} 0.0" rpy="0 0 0"/>
-      	    <geometry>
-              <box size="0.06 0.14 0.06" />
+      	    <origin xyz="0.0 ${reflect * 0.06} 0.0" rpy="0 0 0"/>
+      	    <geometry>
+              <box size="0.06 0.14 0.11" />
+      	    </geometry>
+    	  </collision>
+	  <collision>
+      	    <origin xyz="0 ${reflect * 0.145} 0" rpy="0 ${-pi*0.5}  0"/>
+      	    <geometry>
+              <box size="0.14 0.03 0.06" />
+      	    </geometry>
+    	  </collision>
+	  <collision>
+      	    <origin xyz="0.015 ${reflect * 0.175} -0.06" rpy="${reflect * -0.8} ${-pi*0.5} 0"/>
+      	    <geometry>
+              <box size="0.02 0.1 0.05" />
+      	    </geometry>
+    	  </collision>
+          <collision>
+      	    <origin xyz="0.015 ${reflect * 0.175} 0.06" rpy="${reflect * -0.8} ${-pi*0.5} 0"/>
+      	    <geometry>
+              <box size="0.02 0.1 0.05" />
       	    </geometry>
     	  </collision>
@@ -123,8 +141,8 @@
     	  </inertial>
         </link>
-	<!-- left elbow yaw joint -->
+	<!-- elbow yaw joint -->
         <joint name="${prefix}_arm_el_y" type="revolute">
           <axis xyz="0 0 -1" />
-          <origin xyz="${reflect * 0.030} ${reflect * 0.187} 0.057" rpy="0 0 0"/>
+          <origin xyz="0.030 ${reflect * 0.187} 0.057" rpy="0 0 0"/>
           <parent link="${prefix}_arm_sh_p2_link"/>
           <child link="${prefix}_arm_el_y_link"/>
@@ -133,10 +151,16 @@
         </joint>
         <xacro:insert_transmission name="${prefix}_arm_el_y" />
-	<!-- left elbow yaw link -->
+	<!-- elbow yaw link -->
         <link name="${prefix}_arm_el_y_link">
-    	  <collision>
-      	    <origin xyz="0 0 0" rpy="0 0 0"/>
-      	    <geometry>
-              <mesh filename="package://thormang3_description/meshes/robotis_${prefix}_arm_el_y_link.stl" scale="0.001 0.001 0.001"/>
+	  <collision>
+      	    <origin xyz="0.0 0.0 -0.06" rpy="${pi*0.5} 0 ${pi*0.25}"/>
+      	    <geometry>
+              <box size="0.06 0.12 0.06" />
+      	    </geometry>
+    	  </collision>
+	  <collision>
+      	    <origin xyz="0.08 ${reflect * 0.03} -0.0575" rpy="0 0 0"/>
+      	    <geometry>
+              <box size="0.18 0.06 0.06" />
       	    </geometry>
     	  </collision>
@@ -155,5 +179,5 @@
     	  </inertial>
         </link>
-	<!-- left wrist roll joint -->
+	<!-- wrist roll joint -->
         <joint name="${prefix}_arm_wr_r" type="revolute">
           <axis xyz="1 0 0" />
@@ -165,5 +189,5 @@
         </joint>
         <xacro:insert_transmission name="${prefix}_arm_wr_r" />
-	<!-- left wrist roll link -->
+	<!-- wrist roll link -->
         <link name="${prefix}_arm_wr_r_link">
     	  <collision>
@@ -171,4 +195,22 @@
       	    <geometry>
               <mesh filename="package://thormang3_description/meshes/robotis_${prefix}_arm_wr_r_link.stl" scale="0.001 0.001 0.001"/>
+      	    </geometry>
+    	  </collision>
+	  <collision>
+      	    <origin xyz="0.01 0.0 0.0" rpy="${-pi*0.5} 0 0 "/>
+      	    <geometry>
+              <box size="0.02 0.1 0.05" />
+      	    </geometry>
+    	  </collision>
+	  <collision>
+      	    <origin xyz="0.0325 0.0 0.05" rpy="0 0 0 "/>
+      	    <geometry>
+              <box size="0.065 0.05 0.01" />
+      	    </geometry>
+    	  </collision>
+	  <collision>
+      	    <origin xyz="0.0325 0.0 -0.05" rpy="0 0 0 "/>
+      	    <geometry>
+              <box size="0.065 0.05 0.01" />
       	    </geometry>
     	  </collision>
@@ -187,5 +229,5 @@
     	  </inertial>
         </link>
-	<!-- left wrist yaw joint -->
+	<!-- wrist yaw joint -->
         <joint name="${prefix}_arm_wr_y" type="revolute">
           <axis xyz="0 0 -1" />
@@ -197,10 +239,16 @@
         </joint>
         <xacro:insert_transmission name="${prefix}_arm_wr_y" />
-	<!-- left wrist yaw link -->
+	<!-- wrist yaw link -->
         <link name="${prefix}_arm_wr_y_link">
-    	  <collision>
-      	    <origin xyz="0 0 0" rpy="0 0 0"/>
-      	    <geometry>
-              <mesh filename="package://thormang3_description/meshes/robotis_${prefix}_arm_wr_y_link.stl" scale="0.001 0.001 0.001"/>
+	  <collision>
+      	    <origin xyz="0.0 0.0 -0.045" rpy="${pi*0.5} 0 0"/>
+      	    <geometry>
+              <box size="0.045 0.09 0.045" />
+      	    </geometry>
+    	  </collision>
+	  <collision>
+      	    <origin xyz="0.045 0.0 -0.045" rpy="0 0 0"/>
+      	    <geometry>
+              <box size="0.045 0.09 0.045" />
       	    </geometry>
     	  </collision>
@@ -219,5 +267,5 @@
     	  </inertial>
         </link>
-	<!-- left wrist pitch joint -->
+	<!-- wrist pitch joint -->
         <joint name="${prefix}_arm_wr_p" type="revolute">
           <axis xyz="0 -1 0" />
@@ -229,10 +277,22 @@
         </joint>
         <xacro:insert_transmission name="${prefix}_arm_wr_p" />
-	<!-- left wrist pitch link -->
+	<!-- wrist pitch link -->
         <link name="${prefix}_arm_wr_p_link">
-    	  <collision>
-      	    <origin xyz="0.039 ${reflect * 0.045} 0.000" rpy="${pi/2} ${pi} 0"/>
-      	    <geometry>
-              <mesh filename="package://thormang3_description/meshes/robotis_${prefix}_arm_wr_r_link.stl" scale="0.001 0.001 0.001"/>
+	  <collision>
+      	    <origin xyz="0.0055 ${reflect *0.09} 0.0" rpy="${pi*0.5} ${pi*0.5} 0"/>
+      	    <geometry>
+              <box size="0.05 0.065 0.01" />
+      	    </geometry>
+    	  </collision>
+	  <collision>
+      	    <origin xyz="0.0055 ${reflect *-0.005} 0.0" rpy="${pi*0.5} ${pi*0.5} 0"/>
+      	    <geometry>
+              <box size="0.05 ${reflect *0.065} 0.01" />
+      	    </geometry>
+    	  </collision>
+	  <collision>
+      	    <origin xyz="0.04 ${reflect * 0.043} 0.0" rpy="0 0 0 "/>
+      	    <geometry>
+              <box size="0.02 0.105 0.05" />
       	    </geometry>
     	  </collision>

Commit message: change rotation axis depending on reflectance parameter

File: thormang3_description/urdf/thormang3.structure.arm.xacro (robot description, xacro)
@@ -17,5 +17,5 @@
 	<!-- shoulder pitch 1 joint -->
         <joint name="${prefix}_arm_sh_p1" type="revolute">
-          <axis xyz="0 1 0" />
+          <axis xyz="0 ${reflect} 0" />
           <origin xyz="0.0 ${reflect * 0.177-offset} 0.16" rpy="0 0 0"/>
           <parent link="${parent}"/>

Commit message: rotate another rotation axis

File: thormang3_description/urdf/thormang3.structure.arm.xacro (robot description, xacro)
@@ -93,5 +93,5 @@
 	<!-- shoulder pitch 2 joint -->
         <joint name="${prefix}_arm_sh_p2" type="revolute">
-          <axis xyz="0 1 0" />
+          <axis xyz="0 ${reflect} 0" />
           <origin xyz="-0.057 ${reflect * 0.033} 0.0" rpy="0 0 0"/>
           <parent link="${prefix}_arm_sh_r_link"/>

Commit message: set joint limits

File: thormang3_description/urdf/thormang3.structure.arm.xacro (robot description, xacro)
@@ -21,5 +21,16 @@
           <parent link="${parent}"/>
           <child link="${prefix}_arm_sh_p1_link"/>
-          <limit velocity="6.5" effort="1000" lower="${-pi*0.5}" upper="${pi*0.5}" />
+	  <!--<xacro:if value="${reflect - 1}">
+	    <limit velocity="6.5" effort="1000" lower="${-pi}" upper="${pi*0.5}" />
+	  </xacro:if>
+	  <xacro:unless value="${reflect - 1}">
+	    <limit velocity="6.5" effort="1000" lower="${-0.5*pi}" upper="${pi}" />
+	  </xacro:unless>-->
+	  <xacro:if value="${reflect - 1}">
+	    <limit velocity="6.5" effort="1000" lower="${-0.5*pi}" upper="${pi*0.5}" />
+	  </xacro:if>
+	  <xacro:unless value="${reflect - 1}">
+	    <limit velocity="6.5" effort="1000" lower="${-0.5*pi}" upper="${0.5*pi}" />
+	  </xacro:unless>
           <dynamics damping="0.1" friction="0.0" />
         </joint>
@@ -65,5 +76,5 @@
           <parent link="${prefix}_arm_sh_p1_link"/>
           <child link="${prefix}_arm_sh_r_link"/>
-          <limit velocity="6.5" effort="1000" lower="${-pi*0.5}" upper="${pi*0.5}" />
+          <limit velocity="6.5" effort="1000" lower="-1.16" upper="${pi*0.75}" />
           <dynamics damping="0.1" friction="0.0" />
         </joint>
@@ -97,5 +108,5 @@
           <parent link="${prefix}_arm_sh_r_link"/>
           <child link="${prefix}_arm_sh_p2_link"/>
-          <limit velocity="6.5" effort="1000" lower="${-pi*0.5}" upper="${pi*0.5}" />
+          <limit velocity="6.5" effort="1000" lower="${-pi}" upper="${pi}" />
           <dynamics damping="0.1" friction="0.0" />
         </joint>
@@ -273,5 +284,5 @@
           <parent link="${prefix}_arm_wr_y_link"/>
           <child link="${prefix}_arm_wr_p_link"/>
-          <limit velocity="6.5" effort="1000" lower="${-pi*0.45}" upper="${pi*0.45}" />
+          <limit velocity="6.5" effort="1000" lower="${-pi*0.4}" upper="${pi*0.4}" />
           <dynamics damping="0.1" friction="0.0" />
         </joint>

File: thormang3_description/urdf/thormang3.structure.head.xacro (robot description, xacro)
@@ -41,5 +41,5 @@
           <parent link="head_y_link"/>
           <child link="head_p_link"/>
-          <limit velocity="6.5" effort="1000" lower="${-pi*0.5}" upper="${pi*0.5}" />
+          <limit velocity="6.5" effort="1000" lower="-0.745" upper="1.301" />
           <dynamics damping="0.1" friction="0.0" />
         </joint>

Commit message: use only 1 and a  smaller pi value to prevent bugs with joint limits

File: thormang3_description/urdf/thormang3.structure.arm.xacro (robot description, xacro)
@@ -1,5 +1,4 @@
 <?xml version="1.0"?>
 <robot xmlns:xacro="http://ros.org/wiki/xacro">
-    <xacro:property name="pi" value="3.141592654" />
     <xacro:property name="offset" value="0.0" />
     <xacro:arg name="use_hands" default="false"/>
@@ -22,4 +21,10 @@
           <child link="${prefix}_arm_sh_p1_link"/>
           <limit velocity="6.5" effort="1000" lower="${-pi*0.5}" upper="${pi*0.5}" />
+	  <xacro:if value="${reflect - 1}">
+           <limit velocity="6.5" effort="1000" lower="${-pi}" upper="${pi*0.5}" />
+	  </xacro:if>
+	  <xacro:unless value="${reflect - 1}">
+	    <limit velocity="6.5" effort="1000" lower="${-0.5*pi}" upper="${pi}" />
+	  </xacro:unless>
           <dynamics damping="0.1" friction="0.0" />
         </joint>
@@ -65,5 +70,5 @@
           <parent link="${prefix}_arm_sh_p1_link"/>
           <child link="${prefix}_arm_sh_r_link"/>
-          <limit velocity="6.5" effort="1000" lower="${-pi*0.5}" upper="${pi*0.5}" />
+          <limit velocity="6.5" effort="1000" lower="${-1.16}" upper="${pi*0.75}" />
           <dynamics damping="0.1" friction="0.0" />
         </joint>
@@ -97,5 +102,5 @@
           <parent link="${prefix}_arm_sh_r_link"/>
           <child link="${prefix}_arm_sh_p2_link"/>
-          <limit velocity="6.5" effort="1000" lower="${-pi*0.5}" upper="${pi*0.5}" />
+	  <limit velocity="6.5" effort="1000" lower="${-pi}" upper="${pi}" />
           <dynamics damping="0.1" friction="0.0" />
         </joint>
@@ -273,5 +278,5 @@
           <parent link="${prefix}_arm_wr_y_link"/>
           <child link="${prefix}_arm_wr_p_link"/>
-          <limit velocity="6.5" effort="1000" lower="${-pi*0.45}" upper="${pi*0.45}" />
+          <limit velocity="6.5" effort="1000" lower="${-pi*0.4}" upper="${pi*0.4}" />
           <dynamics damping="0.1" friction="0.0" />
         </joint>

File: thormang3_description/urdf/thormang3.structure.head.xacro (robot description, xacro)
@@ -1,5 +1,4 @@
 <?xml version="1.0"?>
 <robot xmlns:xacro="http://ros.org/wiki/xacro">
-    <xacro:property name="pi" value="3.141592654" />
     <xacro:include filename="$(find hector_components_description)/urdf/hector_multisensor_head.urdf.xacro" />
     <xacro:macro name="thormang3_head" params="parent">

File: thormang3_description/urdf/thormang3.structure.leg.xacro (robot description, xacro)
@@ -1,5 +1,4 @@
 <?xml version="1.0"?>
 <robot xmlns:xacro="http://ros.org/wiki/xacro">
-    <xacro:property name="pi" value="3.141592654" />
     <xacro:macro name="thormang3_l_leg" params="parent">
 	<!-- left hip yaw joint -->

File: thormang3_description/urdf/thormang3.structure.torso.xacro (robot description, xacro)
@@ -2,5 +2,5 @@
 <robot xmlns:xacro="http://www.ros.org/wiki/xacro">
   <!-- some parameters -->
-  <xacro:property name="pi" value="3.141592654" />
+  <xacro:property name="pi" value="3.141592" />
   <xacro:include filename="$(find thormang3_description)/urdf/thormang3.structure.arm.xacro" />
   <xacro:include filename="$(find thormang3_description)/urdf/thormang3.structure.leg.xacro" />

Commit message: fixed 2 missing reflections

File: thormang3_description/urdf/thormang3.structure.arm.xacro (robot description, xacro)
@@ -274,5 +274,5 @@
 	<!-- wrist pitch joint -->
         <joint name="${prefix}_arm_wr_p" type="revolute">
-          <axis xyz="0 -1 0" />
+          <axis xyz="0 ${-reflect} 0" />
           <origin xyz="0.045 ${reflect * -0.045} -0.045" rpy="0 0 0"/>
           <parent link="${prefix}_arm_wr_y_link"/>
@@ -303,5 +303,5 @@
     	  </collision>
    	  <visual>
-      	    <origin xyz="0.039 ${reflect * 0.045} 0.000" rpy="${pi/2} ${pi} 0"/>
+      	    <origin xyz="0.039 ${reflect * 0.045} 0.000" rpy="${reflect * pi/2} ${pi} 0"/>
       	    <geometry>
               <mesh filename="package://thormang3_description/meshes/robotis_${prefix}_arm_wr_r_link.stl" scale="0.001 0.001 0.001"/>

Commit message: forgot to mirror a joint limit

File: thormang3_description/urdf/thormang3.structure.arm.xacro (robot description, xacro)
@@ -20,5 +20,4 @@
           <parent link="${parent}"/>
           <child link="${prefix}_arm_sh_p1_link"/>
-          <limit velocity="6.5" effort="1000" lower="${-pi*0.5}" upper="${pi*0.5}" />
 	  <xacro:if value="${reflect - 1}">
            <limit velocity="6.5" effort="1000" lower="${-pi}" upper="${pi*0.5}" />
@@ -70,5 +69,10 @@
           <parent link="${prefix}_arm_sh_p1_link"/>
           <child link="${prefix}_arm_sh_r_link"/>
-          <limit velocity="6.5" effort="1000" lower="${-1.16}" upper="${pi*0.75}" />
+	  <xacro:if value="${reflect - 1}">
+           <limit velocity="6.5" effort="1000" lower="-1.16" upper="${pi*0.75}" />
+	  </xacro:if>
+	  <xacro:unless value="${reflect - 1}">
+	    <limit velocity="6.5" effort="1000" lower="${-pi*0.75}" upper="1.16" />
+	  </xacro:unless>
           <dynamics damping="0.1" friction="0.0" />
         </joint>

Commit message: use correct inertial origins

File: thormang3_description/urdf/thormang3.structure.arm.xacro (robot description, xacro)
@@ -57,5 +57,5 @@
     	  </visual>
           <inertial>
-      	    <origin xyz="-0.003 0.020 -0.005" rpy="0 0 0"/>
+      	    <origin xyz="-0.003 ${reflect * 0.020} -0.005" rpy="0 0 0"/>
       	    <mass value="0.194"/>
       	    <inertia ixx="1.0" ixy="0.0" ixz="0.0" iyy="1.0" iyz="0.0" izz="1.0" />
@@ -94,5 +94,5 @@
     	  </visual>
           <inertial>
-      	    <origin xyz="-0.060 0.002 0.000" rpy="0 0 0"/>
+      	    <origin xyz="-0.060 ${reflect * 0.002} 0.000" rpy="0 0 0"/>
       	    <mass value="0.875"/>
             <inertia ixx="1.0" ixy="0.0" ixz="0.0" iyy="1.0" iyz="0.0" izz="1.0" />
@@ -182,5 +182,5 @@
     	  </visual>
           <inertial>
-      	    <origin xyz="0.042 0.012 -0.058" rpy="0 0 0"/>
+      	    <origin xyz="0.042 ${reflect * 0.012} -0.058" rpy="0 0 0"/>
       	    <mass value="1.357"/>
 	    <inertia ixx="1.0" ixy="0.0" ixz="0.0" iyy="1.0" iyz="0.0" izz="1.0" />
@@ -232,5 +232,5 @@
     	  </visual>
           <inertial>
-      	    <origin xyz="0.010 0.000 0.002" rpy="0 0 0"/>
+      	    <origin xyz="0.010 0.000 ${reflect * 0.002}" rpy="0 0 0"/>
       	    <mass value="0.087"/>
             <inertia ixx="1.0" ixy="0.0" ixz="0.0" iyy="1.0" iyz="0.0" izz="1.0" />
@@ -270,5 +270,5 @@
     	  </visual>
           <inertial>
-      	    <origin xyz="0.023 0.001 -0.046" rpy="0 0 0"/>
+      	    <origin xyz="0.023 ${reflect * 0.001} -0.046" rpy="0 0 0"/>
       	    <mass value="0.768"/>
       	    <inertia ixx="1.0" ixy="0.0" ixz="0.0" iyy="1.0" iyz="0.0" izz="1.0" />
@@ -314,5 +314,5 @@
     	  </visual>
           <inertial>
-      	    <origin xyz="0.049 0.045 0.002" rpy="0 0 0"/>
+      	    <origin xyz="0.049 ${reflect * 0.045} ${reflect * 0.002}" rpy="0 0 0"/>
       	    <mass value="0.087"/>
       	    <inertia ixx="1.0" ixy="0.0" ixz="0.0" iyy="1.0" iyz="0.0" izz="1.0" />

Commit message: adjust collision model to prevent self collision

File: thormang3_description/urdf/thormang3.structure.arm.xacro (robot description, xacro)
@@ -113,5 +113,5 @@
         <link name="${prefix}_arm_sh_p2_link">
     	  <collision>
-      	    <origin xyz="0.0 ${reflect * 0.06} 0.0" rpy="0 0 0"/>
+      	    <origin xyz="0.0 ${reflect * 0.075} 0.0" rpy="0 0 0"/>
       	    <geometry>
               <box size="0.06 0.14 0.11" />
@@ -171,5 +171,5 @@
       	    <origin xyz="0.08 ${reflect * 0.03} -0.0575" rpy="0 0 0"/>
       	    <geometry>
-              <box size="0.18 0.06 0.06" />
+              <box size="0.17 0.06 0.06" />
       	    </geometry>
     	  </collision>

Commit message: Fixed sh pitch joint limitt

File: thormang3_description/urdf/thormang3.structure.arm.xacro (robot description, xacro)
@@ -21,8 +21,8 @@
           <child link="${prefix}_arm_sh_p1_link"/>
 	  <xacro:if value="${reflect - 1}">
-           <limit velocity="6.5" effort="1000" lower="${-pi}" upper="${pi*0.5}" />
+           <limit velocity="6.5" effort="1000" lower="${-pi*0.5}" upper="${pi}" />
 	  </xacro:if>
 	  <xacro:unless value="${reflect - 1}">
-	    <limit velocity="6.5" effort="1000" lower="${-0.5*pi}" upper="${pi}" />
+	    <limit velocity="6.5" effort="1000" lower="${-pi}" upper="${pi*0.5}" />
 	  </xacro:unless>
           <dynamics damping="0.1" friction="0.0" />

Commit message: Fixed shoulder roll joint limits

File: thormang3_description/urdf/thormang3.structure.arm.xacro (robot description, xacro)
@@ -70,8 +70,8 @@
           <child link="${prefix}_arm_sh_r_link"/>
 	  <xacro:if value="${reflect - 1}">
-           <limit velocity="6.5" effort="1000" lower="-1.16" upper="${pi*0.75}" />
+           <limit velocity="6.5" effort="1000"  lower="${-pi*0.75}" upper="1.16" />
 	  </xacro:if>
 	  <xacro:unless value="${reflect - 1}">
-	    <limit velocity="6.5" effort="1000" lower="${-pi*0.75}" upper="1.16" />
+	    <limit velocity="6.5" effort="1000" lower="-1.16" upper="${pi*0.75}" />
 	  </xacro:unless>
           <dynamics damping="0.1" friction="0.0" />

Commit message: added new ft links in wrists for accurate ft sensor simulation

File: thormang3_description/urdf/thormang3.structure.arm.xacro (robot description, xacro)
@@ -7,9 +7,9 @@
     <xacro:if value="$(arg use_hands)">
         <xacro:include filename="$(find thor_vt_hand_description)/urdf/vt_hand_tud.urdf.xacro.xml" />
-        <vt_hand_tud_macro parent="l_arm_wr_p_link" prefix="l" reflect="-1" >
-            <origin xyz="0.068 0.045 0" rpy="0 -1.57 3.14159"/>
+        <vt_hand_tud_macro parent="l_wrist_ft_link" prefix="l" reflect="-1" >
+            <origin xyz="0.013 0 0" rpy="0 -1.57 3.14159"/>
         </vt_hand_tud_macro>
-        <vt_hand_tud_macro parent="r_arm_wr_p_link" prefix="r" reflect="1" >
-            <origin xyz="0.068 -0.045 0" rpy="0 1.57 0"/>
+        <vt_hand_tud_macro parent="r_wrist_ft_link" prefix="r" reflect="1" >
+            <origin xyz="0.013 0 0" rpy="0 1.57 0"/>
         </vt_hand_tud_macro>
     </xacro:if>
@@ -239,4 +239,15 @@
     	  </inertial>
         </link>
+    <!-- left ft joint -->
+    <!--use "fixed" revolute joint for FT sensor simulation-->
+        <joint name="l_arm_ft" type="revolute">
+          <origin xyz="0.055 0.045 0" rpy="0 0 0"/>
+          <parent link="l_arm_wr_p_link"/>
+          <child link="l_wrist_ft_link"/>
+          <limit velocity="6.5" effort="1000" lower="0" upper="0" />
+        </joint>
+    <!-- right wrist ft link -->
+        <link name="l_wrist_ft_link">
+        </link>
     </xacro:macro>
     <xacro:macro name="thormang3_r_arm" params="parent">
@@ -463,5 +474,16 @@
       	    <inertia ixx="1.0" ixy="0.0" ixz="0.0" iyy="1.0" iyz="0.0" izz="1.0" />
             <!--<inertia ixx="0.00047" ixy="0.00001" ixz="0.0" iyy="0.00042" iyz="0.0" izz="0.00058" />-->
-    	  </inertial>
+    	    </inertial>
+        </link>
+    <!-- right ft joint -->
+    <!--use "fixed" revolute joint for FT sensor simulation-->
+        <joint name="r_arm_ft" type="revolute">
+          <origin xyz="0.055 -0.045 0" rpy="0 0 0"/>
+          <parent link="r_arm_wr_p_link"/>
+          <child link="r_wrist_ft_link"/>
+          <limit velocity="6.5" effort="1000" lower="0" upper="0" />
+        </joint>
+    <!-- right wrist ft link -->
+        <link name="r_wrist_ft_link">
         </link>
     </xacro:macro>
