Commit message: rotated imus to better match real orientation

File: thormang3_description/urdf/thormang3.structure.arm.xacro (robot description, xacro)
@@ -7,8 +7,8 @@
         <xacro:include filename="$(find thor_vt_hand_description)/urdf/vt_hand_tud.urdf.xacro.xml" />
         <vt_hand_tud_macro parent="l_wrist_ft_link" prefix="l" reflect="-1" >
-            <origin xyz="0.013 0 0" rpy="0 -1.57 3.14159"/>
+            <origin xyz="0.013 0 0" rpy="0 ${pi} ${0.5 * pi}"/>
         </vt_hand_tud_macro>
         <vt_hand_tud_macro parent="r_wrist_ft_link" prefix="r" reflect="1" >
-            <origin xyz="0.013 0 0" rpy="0 1.57 0"/>
+            <origin xyz="0.013 0 0" rpy="0 ${pi} -${0.5 * pi}"/>
         </vt_hand_tud_macro>
     </xacro:if>
@@ -323,5 +323,5 @@
     <!--use "fixed" revolute joint for FT sensor simulation-->
         <joint name="${prefix}_arm_ft" type="revolute">
-          <origin xyz="0.055 ${reflect * 0.045} 0" rpy="0 0 0"/>
+          <origin xyz="0.055 ${reflect * 0.045} 0" rpy="-${0.5 * pi} 0 ${0.5 * pi}"/>
           <parent link="${prefix}_arm_wr_p_link"/>
           <child link="${prefix}_wrist_ft_link"/>

Commit message: fixed ft link orientation

File: thormang3_description/urdf/thormang3.structure.arm.xacro (robot description, xacro)
@@ -7,8 +7,8 @@
         <xacro:include filename="$(find thor_vt_hand_description)/urdf/vt_hand_tud.urdf.xacro.xml" />
         <vt_hand_tud_macro parent="l_wrist_ft_link" prefix="l" reflect="-1" >
-            <origin xyz="0.013 0 0" rpy="0 ${pi} ${0.5 * pi}"/>
+            <origin xyz="0.013 0 0" rpy="0 0 -${0.5 * pi}"/>
         </vt_hand_tud_macro>
         <vt_hand_tud_macro parent="r_wrist_ft_link" prefix="r" reflect="1" >
-            <origin xyz="0.013 0 0" rpy="0 ${pi} -${0.5 * pi}"/>
+            <origin xyz="0.013 0 0" rpy="0 0 ${0.5 * pi}"/>
         </vt_hand_tud_macro>
     </xacro:if>
@@ -323,5 +323,5 @@
     <!--use "fixed" revolute joint for FT sensor simulation-->
         <joint name="${prefix}_arm_ft" type="revolute">
-          <origin xyz="0.055 ${reflect * 0.045} 0" rpy="-${0.5 * pi} 0 ${0.5 * pi}"/>
+          <origin xyz="0.055 ${reflect * 0.045} 0" rpy="-${0.5 * pi} 0 -${0.5 * pi}"/>
           <parent link="${prefix}_arm_wr_p_link"/>
           <child link="${prefix}_wrist_ft_link"/>

File: thormang3_description/urdf/thormang3.structure.leg.xacro (robot description, xacro)
@@ -211,5 +211,5 @@
         <!--use "fixed" revolute joint for FT sensor simulation-->
         <joint name="${prefix}_leg_ft" type="revolute">
-            <origin xyz="-0.057 0.0 -0.087" rpy="0 0 0"/>
+            <origin xyz="-0.057 0.0 -0.087" rpy="${pi} 0 0"/>
             <parent link="${prefix}_leg_an_r_link"/>
             <child link="${prefix}_foot_ft_link"/>
@@ -221,5 +221,5 @@
         <!-- ft fixed joint -->
         <joint name="${prefix}_leg_ft_fixed" type="fixed">
-            <origin xyz="0 0.0 -0.0275" rpy="0 0 0"/>
+            <origin xyz="0 0.0 0.0275" rpy="${pi} 0 0"/>
             <parent link="${prefix}_foot_ft_link"/>
             <child link="${prefix}_leg_foot_link"/>

Commit message: rotated ft sensors again

File: thormang3_description/urdf/thormang3.structure.arm.xacro (robot description, xacro)
@@ -7,8 +7,8 @@
         <xacro:include filename="$(find thor_vt_hand_description)/urdf/vt_hand_tud.urdf.xacro.xml" />
         <vt_hand_tud_macro parent="l_wrist_ft_link" prefix="l" reflect="-1" >
-            <origin xyz="0.013 0 0" rpy="0 0 -${0.5 * pi}"/>
+            <origin xyz="0.013 0 0" rpy="0 0 ${0.5 * pi}"/>
         </vt_hand_tud_macro>
         <vt_hand_tud_macro parent="r_wrist_ft_link" prefix="r" reflect="1" >
-            <origin xyz="0.013 0 0" rpy="0 0 ${0.5 * pi}"/>
+            <origin xyz="0.013 0 0" rpy="0 0 -${0.5 * pi}"/>
         </vt_hand_tud_macro>
     </xacro:if>
@@ -323,5 +323,5 @@
     <!--use "fixed" revolute joint for FT sensor simulation-->
         <joint name="${prefix}_arm_ft" type="revolute">
-          <origin xyz="0.055 ${reflect * 0.045} 0" rpy="-${0.5 * pi} 0 -${0.5 * pi}"/>
+          <origin xyz="0.055 ${reflect * 0.045} 0" rpy="${0.5 * pi} 0 ${0.5 * pi}"/>
           <parent link="${prefix}_arm_wr_p_link"/>
           <child link="${prefix}_wrist_ft_link"/>

File: thormang3_description/urdf/thormang3.structure.leg.xacro (robot description, xacro)
@@ -211,5 +211,5 @@
         <!--use "fixed" revolute joint for FT sensor simulation-->
         <joint name="${prefix}_leg_ft" type="revolute">
-            <origin xyz="-0.057 0.0 -0.087" rpy="${pi} 0 0"/>
+            <origin xyz="-0.057 0.0 -0.087" rpy="${pi} 0 ${pi}"/>
             <parent link="${prefix}_leg_an_r_link"/>
             <child link="${prefix}_foot_ft_link"/>
@@ -221,5 +221,5 @@
         <!-- ft fixed joint -->
         <joint name="${prefix}_leg_ft_fixed" type="fixed">
-            <origin xyz="0 0.0 0.0275" rpy="${pi} 0 0"/>
+            <origin xyz="0 0.0 0.0275" rpy="${pi} 0 ${pi}"/>
             <parent link="${prefix}_foot_ft_link"/>
             <child link="${prefix}_leg_foot_link"/>

Commit message: fixed ft orientation of left wrist and fixed distance of hand from sensor

File: thormang3_description/urdf/thormang3.structure.arm.xacro (robot description, xacro)
@@ -7,8 +7,8 @@
         <xacro:include filename="$(find thor_vt_hand_description)/urdf/vt_hand_tud.urdf.xacro.xml" />
         <vt_hand_tud_macro parent="l_wrist_ft_link" prefix="l" reflect="-1" >
-            <origin xyz="0.013 0 0" rpy="0 0 ${0.5 * pi}"/>
+            <origin xyz="0 0 0.013" rpy="0 0 -${0.5 * pi}"/>
         </vt_hand_tud_macro>
         <vt_hand_tud_macro parent="r_wrist_ft_link" prefix="r" reflect="1" >
-            <origin xyz="0.013 0 0" rpy="0 0 -${0.5 * pi}"/>
+            <origin xyz="0 0 0.013" rpy="0 0 -${0.5 * pi}"/>
         </vt_hand_tud_macro>
     </xacro:if>
@@ -323,5 +323,5 @@
     <!--use "fixed" revolute joint for FT sensor simulation-->
         <joint name="${prefix}_arm_ft" type="revolute">
-          <origin xyz="0.055 ${reflect * 0.045} 0" rpy="${0.5 * pi} 0 ${0.5 * pi}"/>
+          <origin xyz="0.055 ${reflect * 0.045} 0" rpy="${-reflect * 0.5 * pi} 0 ${-reflect * 0.5 * pi}"/>
           <parent link="${prefix}_arm_wr_p_link"/>
           <child link="${prefix}_wrist_ft_link"/>

Commit message: cleanup

File: thormang3_description/urdf/thormang3.structure.arm.xacro (robot description, xacro)
@@ -86,5 +86,5 @@
             </geometry>
         </collision>
-      <visual>
+        <visual>
             <origin xyz="0 0 0" rpy="0 0 0"/>
             <geometry>
@@ -93,5 +93,5 @@
             <material name="grey"/>
         </visual>
-          <inertial>
+        <inertial>
             <origin xyz="-0.060 ${reflect * 0.002} 0.000" rpy="0 0 0"/>
             <mass value="0.875"/>
@@ -106,5 +106,5 @@
           <parent link="${prefix}_arm_sh_r_link"/>
           <child link="${prefix}_arm_sh_p2_link"/>
-    <limit velocity="6.5" effort="1000" lower="${-pi}" upper="${pi}" />
+          <limit velocity="6.5" effort="1000" lower="${-pi}" upper="${pi}" />
           <dynamics damping="0.1" friction="0.0" />
         </joint>
@@ -118,5 +118,5 @@
             </geometry>
         </collision>
-    <collision>
+        <collision>
             <origin xyz="0 ${reflect * 0.145} 0" rpy="0 ${-pi*0.5}  0"/>
             <geometry>
@@ -124,5 +124,5 @@
             </geometry>
         </collision>
-    <collision>
+        <collision>
             <origin xyz="0.015 ${reflect * 0.175} -0.06" rpy="${reflect * -0.8} ${-pi*0.5} 0"/>
             <geometry>
@@ -130,5 +130,5 @@
             </geometry>
         </collision>
-          <collision>
+        <collision>
             <origin xyz="0.015 ${reflect * 0.175} 0.06" rpy="${reflect * -0.8} ${-pi*0.5} 0"/>
             <geometry>
@@ -136,5 +136,5 @@
             </geometry>
         </collision>
-       <visual>
+        <visual>
             <origin xyz="0 0 0" rpy="0 0 0"/>
             <geometry>
@@ -143,5 +143,5 @@
             <material name="grey"/>
         </visual>
-          <inertial>
+        <inertial>
             <origin xyz="0.000 0.073 0.000" rpy="0 0 0"/>
             <mass value="1.122"/>

Commit message: fixed limits leading to undesired behavior in simulation

File: thormang3_description/urdf/thormang3.structure.arm.xacro (robot description, xacro)
@@ -106,5 +106,5 @@
           <parent link="${prefix}_arm_sh_r_link"/>
           <child link="${prefix}_arm_sh_p2_link"/>
-          <limit velocity="6.5" effort="1000" lower="${-pi}" upper="${pi}" />
+          <limit velocity="6.5" effort="1000" lower="${-pi+0.001}" upper="${pi-0.001}" />
           <dynamics damping="0.1" friction="0.0" />
         </joint>

Commit message: fixed indents

File: thormang3_description/urdf/thormang3.structure.arm.xacro (robot description, xacro)
@@ -5,11 +5,11 @@
     <!-- VT hands description -->
     <xacro:if value="$(arg use_hands)">
-        <xacro:include filename="$(find thor_vt_hand_description)/urdf/vt_hand_tud.urdf.xacro.xml" />
-        <vt_hand_tud_macro parent="l_wrist_ft_link" prefix="l" reflect="-1" >
-            <origin xyz="0 0 0.013" rpy="0 0 -${0.5 * pi}"/>
-        </vt_hand_tud_macro>
-        <vt_hand_tud_macro parent="r_wrist_ft_link" prefix="r" reflect="1" >
-            <origin xyz="0 0 0.013" rpy="0 0 -${0.5 * pi}"/>
-        </vt_hand_tud_macro>
+      <xacro:include filename="$(find thor_vt_hand_description)/urdf/vt_hand_tud.urdf.xacro.xml" />
+      <vt_hand_tud_macro parent="l_wrist_ft_link" prefix="l" reflect="-1" >
+        <origin xyz="0 0 0.013" rpy="0 0 -${0.5 * pi}"/>
+      </vt_hand_tud_macro>
+      <vt_hand_tud_macro parent="r_wrist_ft_link" prefix="r" reflect="1" >
+        <origin xyz="0 0 0.013" rpy="0 0 -${0.5 * pi}"/>
+      </vt_hand_tud_macro>
     </xacro:if>
     <xacro:macro name="thormang3_arm" params="parent prefix reflect">
@@ -20,10 +20,10 @@
           <parent link="${parent}"/>
           <child link="${prefix}_arm_sh_p1_link"/>
-    <xacro:if value="${reflect - 1}">
-           <limit velocity="6.5" effort="1000" lower="${-pi*0.5}" upper="${pi}" />
-    </xacro:if>
-    <xacro:unless value="${reflect - 1}">
-      <limit velocity="6.5" effort="1000" lower="${-pi}" upper="${pi*0.5}" />
-    </xacro:unless>
+          <xacro:if value="${reflect - 1}">
+            <limit velocity="6.5" effort="1000" lower="${-pi*0.5}" upper="${pi}" />
+          </xacro:if>
+          <xacro:unless value="${reflect - 1}">
+            <limit velocity="6.5" effort="1000" lower="${-pi}" upper="${pi*0.5}" />
+          </xacro:unless>
           <dynamics damping="0.1" friction="0.0" />
         </joint>
@@ -31,10 +31,10 @@
   <!-- shoulder pitch 1 link -->
         <link name="${prefix}_arm_sh_p1_link">
-        <collision>
+          <collision>
             <origin xyz="${reflect * -0.005} ${reflect * 0.015} 0" rpy="0 0 0"/>
             <geometry>
               <box size="0.14 0.03 0.06" />
             </geometry>
-        </collision>
+          </collision>
           <collision>
             <origin xyz="${reflect * 0.06} ${reflect * 0.04} -0.02" rpy="${reflect * -0.8} 0 0"/>
@@ -42,5 +42,5 @@
               <box size="0.02 0.1 0.05" />
             </geometry>
-        </collision>
+          </collision>
           <collision>
             <origin xyz="${reflect * -0.06} ${reflect * 0.04} -0.02" rpy="${reflect * -0.8} 0 0"/>
@@ -48,6 +48,6 @@
               <box size="0.02 0.1 0.05" />
             </geometry>
-        </collision>
-      <visual>
+          </collision>
+          <visual>
             <origin xyz="0 0 0" rpy="0 0 0"/>
             <geometry>
@@ -55,5 +55,5 @@
             </geometry>
             <material name="grey"/>
-        </visual>
+          </visual>
           <inertial>
             <origin xyz="-0.003 ${reflect * 0.020} -0.005" rpy="0 0 0"/>
@@ -61,5 +61,5 @@
             <inertia ixx="1.0" ixy="0.0" ixz="0.0" iyy="1.0" iyz="0.0" izz="1.0" />
             <!--<inertia ixx="0.00018" ixy="0.0" ixz="0.0" iyy="0.00058" iyz="0.00004" izz="0.00057" />-->
-        </inertial>
+          </inertial>
         </link>
   <!-- shoulder roll joint -->
@@ -69,10 +69,10 @@
           <parent link="${prefix}_arm_sh_p1_link"/>
           <child link="${prefix}_arm_sh_r_link"/>
-    <xacro:if value="${reflect - 1}">
-           <limit velocity="6.5" effort="1000"  lower="${-pi*0.75}" upper="1.16" />
-    </xacro:if>
-    <xacro:unless value="${reflect - 1}">
-      <limit velocity="6.5" effort="1000" lower="-1.16" upper="${pi*0.75}" />
-    </xacro:unless>
+          <xacro:if value="${reflect - 1}">
+            <limit velocity="6.5" effort="1000"  lower="${-pi*0.75}" upper="1.16" />
+          </xacro:if>
+          <xacro:unless value="${reflect - 1}">
+            <limit velocity="6.5" effort="1000" lower="-1.16" upper="${pi*0.75}" />
+          </xacro:unless>
           <dynamics damping="0.1" friction="0.0" />
         </joint>
@@ -112,29 +112,29 @@
   <!-- shoulder pitch2 link -->
         <link name="${prefix}_arm_sh_p2_link">
-        <collision>
+          <collision>
             <origin xyz="0.0 ${reflect * 0.075} 0.0" rpy="0 0 0"/>
             <geometry>
               <box size="0.06 0.14 0.11" />
             </geometry>
-        </collision>
-        <collision>
+          </collision>
+          <collision>
             <origin xyz="0 ${reflect * 0.145} 0" rpy="0 ${-pi*0.5}  0"/>
             <geometry>
               <box size="0.14 0.03 0.06" />
             </geometry>
-        </collision>
-        <collision>
+          </collision>
+          <collision>
             <origin xyz="0.015 ${reflect * 0.175} -0.06" rpy="${reflect * -0.8} ${-pi*0.5} 0"/>
             <geometry>
               <box size="0.02 0.1 0.05" />
             </geometry>
-        </collision>
-        <collision>
+          </collision>
+          <collision>
             <origin xyz="0.015 ${reflect * 0.175} 0.06" rpy="${reflect * -0.8} ${-pi*0.5} 0"/>
             <geometry>
               <box size="0.02 0.1 0.05" />
             </geometry>
-        </collision>
-        <visual>
+          </collision>
+          <visual>
             <origin xyz="0 0 0" rpy="0 0 0"/>
             <geometry>
@@ -142,11 +142,11 @@
             </geometry>
             <material name="grey"/>
-        </visual>
-        <inertial>
+          </visual>
+          <inertial>
             <origin xyz="0.000 0.073 0.000" rpy="0 0 0"/>
             <mass value="1.122"/>
             <inertia ixx="1.0" ixy="0.0" ixz="0.0" iyy="1.0" iyz="0.0" izz="1.0" />
             <!--<inertia ixx="0.00277" ixy="-0.00002" ixz="-0.00001" iyy="0.00090" iyz="-0.00004" izz="0.00255" />-->
-        </inertial>
+          </inertial>
         </link>
   <!-- elbow yaw joint -->
@@ -162,17 +162,17 @@
   <!-- elbow yaw link -->
         <link name="${prefix}_arm_el_y_link">
-    <collision>
+          <collision>
             <origin xyz="0.0 0.0 -0.06" rpy="${pi*0.5} 0 ${pi*0.25}"/>
             <geometry>
               <box size="0.06 0.12 0.06" />
             </geometry>
-        </collision>
-    <collision>
+          </collision>
+          <collision>
             <origin xyz="0.08 ${reflect * 0.03} -0.0575" rpy="0 0 0"/>
             <geometry>
               <box size="0.17 0.06 0.06" />
             </geometry>
-        </collision>
-       <visual>
+          </collision>
+          <visual>
             <origin xyz="0 0 0" rpy="0 0 0"/>
             <geometry>
@@ -180,11 +180,11 @@
             </geometry>
             <material name="grey"/>
-        </visual>
+          </visual>
           <inertial>
             <origin xyz="0.042 ${reflect * 0.012} -0.058" rpy="0 0 0"/>
             <mass value="1.357"/>
-      <inertia ixx="1.0" ixy="0.0" ixz="0.0" iyy="1.0" iyz="0.0" izz="1.0" />
+            <inertia ixx="1.0" ixy="0.0" ixz="0.0" iyy="1.0" iyz="0.0" izz="1.0" />
             <!--<inertia ixx="0.00152" ixy="-0.00100" ixz="-0.00006" iyy="0.00560" iyz="-0.00002" izz="0.00528" />-->
-        </inertial>
+          </inertial>
         </link>
   <!-- wrist roll joint -->
@@ -200,29 +200,29 @@
   <!-- wrist roll link -->
         <link name="${prefix}_arm_wr_r_link">
-        <collision>
+          <collision>
             <origin xyz="0 0 0" rpy="0 0 0"/>
             <geometry>
               <mesh filename="package://thormang3_description/meshes/robotis_${prefix}_arm_wr_r_link.stl" scale="0.001 0.001 0.001"/>
             </geometry>
-        </collision>
-    <collision>
+          </collision>
+          <collision>
             <origin xyz="0.01 0.0 0.0" rpy="${-pi*0.5} 0 0 "/>
             <geometry>
               <box size="0.02 0.1 0.05" />
             </geometry>
-        </collision>
-    <collision>
+          </collision>
+          <collision>
             <origin xyz="0.0325 0.0 0.05" rpy="0 0 0 "/>
             <geometry>
               <box size="0.065 0.05 0.01" />
             </geometry>
-        </collision>
-    <collision>
+          </collision>
+          <collision>
             <origin xyz="0.0325 0.0 -0.05" rpy="0 0 0 "/>
             <geometry>
               <box size="0.065 0.05 0.01" />
             </geometry>
-        </collision>
-       <visual>
+          </collision>
+         <visual>
             <origin xyz="0 0 0" rpy="0 0 0"/>
             <geometry>
@@ -230,5 +230,5 @@
             </geometry>
             <material name="grey"/>
-        </visual>
+          </visual>
           <inertial>
             <origin xyz="0.010 0.000 ${reflect * 0.002}" rpy="0 0 0"/>
@@ -236,5 +236,5 @@
             <inertia ixx="1.0" ixy="0.0" ixz="0.0" iyy="1.0" iyz="0.0" izz="1.0" />
             <!--<inertia ixx="0.00012" ixy="0.0" ixz="0.0" iyy="0.00011" iyz="0.0" izz="0.00003" />-->
-        </inertial>
+          </inertial>
         </link>
   <!-- wrist yaw joint -->
@@ -250,17 +250,17 @@
   <!-- wrist yaw link -->
         <link name="${prefix}_arm_wr_y_link">
-    <collision>
+          <collision>
             <origin xyz="0.0 0.0 -0.045" rpy="${pi*0.5} 0 0"/>
             <geometry>
               <box size="0.045 0.09 0.045" />
             </geometry>
-        </collision>
-    <collision>
+          </collision>
+          <collision>
             <origin xyz="0.045 0.0 -0.045" rpy="0 0 0"/>
             <geometry>
               <box size="0.045 0.09 0.045" />
             </geometry>
-        </collision>
-       <visual>
+          </collision>
+          <visual>
             <origin xyz="0 0 0" rpy="0 0 0"/>
             <geometry>
@@ -268,5 +268,5 @@
             </geometry>
             <material name="grey"/>
-        </visual>
+          </visual>
           <inertial>
             <origin xyz="0.023 ${reflect * 0.001} -0.046" rpy="0 0 0"/>
@@ -274,5 +274,5 @@
             <inertia ixx="1.0" ixy="0.0" ixz="0.0" iyy="1.0" iyz="0.0" izz="1.0" />
             <!--<inertia ixx="0.00059" ixy="-0.00002" ixz="-0.00002" iyy="0.00078" iyz="0.0" izz="0.00078" />-->
-        </inertial>
+          </inertial>
         </link>
   <!-- wrist pitch joint -->
@@ -288,23 +288,23 @@
   <!-- wrist pitch link -->
         <link name="${prefix}_arm_wr_p_link">
-        <collision>
+          <collision>
             <origin xyz="0.0055 ${reflect *0.09} 0.0" rpy="${pi*0.5} ${pi*0.5} 0"/>
             <geometry>
               <box size="0.05 0.065 0.01" />
             </geometry>
-        </collision>
-        <collision>
+          </collision>
+          <collision>
             <origin xyz="0.0055 ${reflect *-0.005} 0.0" rpy="${pi*0.5} ${pi*0.5} 0"/>
             <geometry>
               <box size="0.05 ${reflect *0.065} 0.01" />
             </geometry>
-        </collision>
-    <collision>
+          </collision>
+          <collision>
             <origin xyz="0.04 ${reflect * 0.043} 0.0" rpy="0 0 0 "/>
             <geometry>
               <box size="0.02 0.105 0.05" />
             </geometry>
-        </collision>
-       <visual>
+          </collision>
+          <visual>
             <origin xyz="0.039 ${reflect * 0.045} 0.000" rpy="${reflect * pi/2} ${pi} 0"/>
             <geometry>
@@ -312,5 +312,5 @@
             </geometry>
             <material name="grey"/>
-        </visual>
+          </visual>
           <inertial>
             <origin xyz="0.049 ${reflect * 0.045} ${reflect * 0.002}" rpy="0 0 0"/>
