Commit message: added new pelvis, set real inertias except fingers, begun to tune the gains without hands

File: thormang3_description/urdf/thormang3.structure.arm.xacro (robot description, xacro)
@@ -78,6 +78,6 @@
         <origin xyz="-0.003 ${reflect * 0.020} -0.005" rpy="0 0 0" />
         <mass value="0.194" />
-        <inertia ixx="1.0" ixy="0.0" ixz="0.0" iyy="1.0" iyz="0.0" izz="1.0" />
-        <!--<inertia ixx="0.00018" ixy="0.0" ixz="0.0" iyy="0.00058" iyz="0.00004" izz="0.00057" />-->
+        <!--<inertia ixx="1.0" ixy="0.0" ixz="0.0" iyy="1.0" iyz="0.0" izz="1.0" />-->
+        <inertia ixx="0.00018" ixy="0.0" ixz="0.0" iyy="0.00058" iyz="${reflect * 0.00004}" izz="0.00057" />
       </inertial>
     </link>
@@ -115,6 +115,6 @@
         <origin xyz="-0.060 ${reflect * 0.002} 0.000" rpy="0 0 0" />
         <mass value="0.875" />
-        <inertia ixx="1.0" ixy="0.0" ixz="0.0" iyy="1.0" iyz="0.0" izz="1.0" />
-        <!--<inertia ixx="0.00043" ixy="0.0" ixz="0.0" iyy="0.00112" iyz="0.0" izz="0.00113" />-->
+        <!--<inertia ixx="1.0" ixy="0.0" ixz="0.0" iyy="1.0" iyz="0.0" izz="1.0" />-->
+        <inertia ixx="0.00043" ixy="0.0" ixz="0.0" iyy="0.00112" iyz="0.0" izz="0.00113" />
     </inertial>
     </link>
@@ -163,8 +163,8 @@
       </visual>
       <inertial>
-        <origin xyz="0.000 0.073 0.000" rpy="0 0 0" />
+        <origin xyz="0.000 ${reflect * 0.073} 0.000" rpy="0 0 0" />
         <mass value="1.122" />
-        <inertia ixx="1.0" ixy="0.0" ixz="0.0" iyy="1.0" iyz="0.0" izz="1.0" />
-        <!--<inertia ixx="0.00277" ixy="-0.00002" ixz="-0.00001" iyy="0.00090" iyz="-0.00004" izz="0.00255" />-->
+        <!--<inertia ixx="1.0" ixy="0.0" ixz="0.0" iyy="1.0" iyz="0.0" izz="1.0" />-->
+        <inertia ixx="0.00277" ixy="${reflect * -0.00002}" ixz="-0.00001" iyy="0.00090" iyz="${reflect * -0.00004}" izz="0.00255" />
       </inertial>
     </link>
@@ -203,6 +203,6 @@
         <origin xyz="0.042 ${reflect * 0.012} -0.058" rpy="0 0 0" />
         <mass value="1.357" />
-        <inertia ixx="1.0" ixy="0.0" ixz="0.0" iyy="1.0" iyz="0.0" izz="1.0" />
-        <!--<inertia ixx="0.00152" ixy="-0.00100" ixz="-0.00006" iyy="0.00560" iyz="-0.00002" izz="0.00528" />-->
+        <!--<inertia ixx="1.0" ixy="0.0" ixz="0.0" iyy="1.0" iyz="0.0" izz="1.0" />-->
+        <inertia ixx="0.00152" ixy="${reflect * -0.00100}" ixz="-0.00006" iyy="0.00560" iyz="${reflect * -0.00002}" izz="0.00528" />
       </inertial>
     </link>
@@ -253,6 +253,6 @@
         <origin xyz="0.010 0.000 ${reflect * 0.002}" rpy="0 0 0" />
         <mass value="0.087" />
-        <inertia ixx="1.0" ixy="0.0" ixz="0.0" iyy="1.0" iyz="0.0" izz="1.0" />
-        <!--<inertia ixx="0.00012" ixy="0.0" ixz="0.0" iyy="0.00011" iyz="0.0" izz="0.00003" />-->
+        <!--<inertia ixx="1.0" ixy="0.0" ixz="0.0" iyy="1.0" iyz="0.0" izz="1.0" />-->
+        <inertia ixx="0.00012" ixy="0.0" ixz="0.0" iyy="0.00011" iyz="0.0" izz="0.00003" />
       </inertial>
     </link>
@@ -291,6 +291,6 @@
         <origin xyz="0.023 ${reflect * 0.001} -0.046" rpy="0 0 0" />
         <mass value="0.768" />
-        <inertia ixx="1.0" ixy="0.0" ixz="0.0" iyy="1.0" iyz="0.0" izz="1.0" />
-        <!--<inertia ixx="0.00059" ixy="-0.00002" ixz="-0.00002" iyy="0.00078" iyz="0.0" izz="0.00078" />-->
+        <!--<inertia ixx="1.0" ixy="0.0" ixz="0.0" iyy="1.0" iyz="0.0" izz="1.0" />-->
+        <inertia ixx="0.00059" ixy="${reflect * -0.00002}" ixz="-0.00002" iyy="0.00078" iyz="0.0" izz="0.00078" />
       </inertial>
     </link>
@@ -333,21 +333,23 @@
       </visual>
       <inertial>
-        <origin xyz="0.049 ${reflect * 0.045} ${reflect * 0.002}" rpy="0 0 0" />
+        <!--<origin xyz="0.049 ${reflect * 0.045} ${reflect * 0.002}" rpy="0 0 0" />-->
+	<origin xyz="0.029 ${reflect * 0.045} 0.0" rpy="0 0 0" />
         <mass value="0.087" />
-        <inertia ixx="1.0" ixy="0.0" ixz="0.0" iyy="1.0" iyz="0.0" izz="1.0" />
-        <!--<inertia ixx="0.00047" ixy="-0.00001" ixz="0.0" iyy="0.00042" iyz="0.0" izz="0.00058" />-->
+        <!--<inertia ixx="1.0" ixy="0.0" ixz="0.0" iyy="1.0" iyz="0.0" izz="1.0" />-->
+        <!--<inertia ixx="0.00047" ixy="${reflect * -0.00001}" ixz="0.0" iyy="0.00042" iyz="0.0" izz="0.00058" />-->
+        <inertia ixx="0.00012" ixy="0.0" ixz="0.0" iyy="0.00003" iyz="0.0" izz="0.00011" />
       </inertial>
     </link>
     <!--ft joint -->
     <!--use "fixed" revolute joint for FT sensor simulation-->
-    <joint name="${prefix}_arm_ft" type="revolute">
+    <!--<joint name="${prefix}_arm_ft" type="revolute">
       <origin xyz="0.055 ${reflect * 0.045} 0" rpy="${-reflect * 0.5 * pi} 0 ${-reflect * 0.5 * pi}" />
       <parent link="${prefix}_arm_wr_p_link" />
       <child link="${prefix}_wrist_ft_link" />
       <limit velocity="6.5" effort="1000" lower="0" upper="0" />
-    </joint>
+    </joint>-->
     <!-- wrist ft link -->
-    <link name="${prefix}_wrist_ft_link">
-    </link>
+    <!--<link name="${prefix}_wrist_ft_link">
+    </link>-->
   </xacro:macro>
 </robot>

File: thormang3_description/urdf/thormang3.structure.head.xacro (robot description, xacro)
@@ -31,5 +31,6 @@
       	    <origin xyz="0.0 -0.002 0.010" rpy="0 0 0"/>
       	    <mass value="0.087"/>
-      	    <inertia ixx="1.0" ixy="0.0" ixz="0.0" iyy="1.0" iyz="0.0" izz="1.0" />
+      	    <!--<inertia ixx="1.0" ixy="0.0" ixz="0.0" iyy="1.0" iyz="0.0" izz="1.0" />-->
+	    <inertia ixx="0.00011" ixy="0.0" ixz="0.0" iyy="0.00003" iyz="0.0" izz="0.00012" />
     	  </inertial>
         </link>
@@ -60,7 +61,10 @@
     	  </visual>
           <inertial>
-      	    <origin xyz="0.009 0.046 0.022" rpy="0 0 0"/>
-      	    <mass value="0.724"/>
-      	    <inertia ixx="1.0" ixy="0.0" ixz="0.0" iyy="1.0" iyz="0.0" izz="1.0" />
+      	    <origin xyz="-0.012 0.044 0.072" rpy="0 0 0"/>
+      	    <!--<mass value="0.724"/>-->
+	    <mass value="1.048"/>
+      	    <!--<inertia ixx="1.0" ixy="0.0" ixz="0.0" iyy="1.0" iyz="0.0" izz="1.0" />  -->
+	    <!--<inertia ixx="0.00113" ixy="0.00001" ixz="-0.00005" iyy="0.00114" iyz="0.00002" izz="0.00084" />-->
+            <inertia ixx="0.00336" ixy="-0.00029" ixz="-0.00042" iyy="0.0032" iyz="-0.00008" izz="0.00126" />
     	  </inertial>
         </link>
@@ -73,5 +77,5 @@
 	<hector_multisensor_head_macro parent="head_y_link" name="head" scaling="0.001">
 	  <origin xyz="0.0 0.0 0.0" rpy="${M_PI*0.5} 0.0 ${M_PI*0.5}"/>
-	  <!-- Calibrated origin of the laser scanner-->
+	  <!-- Calibrated origin of the laser scanner -->
 	   <xacro:include filename="$(find thormang3_description)/calibration/multisensor_head_calibration.urdf.xacro" />
 	</hector_multisensor_head_macro>

File: thormang3_description/urdf/thormang3.structure.leg.xacro (robot description, xacro)
@@ -28,8 +28,8 @@
             </visual>
             <inertial>
-                <origin xyz="0.012 ${reflect * 0.000} -0.025" rpy="0 0 0"/>
+                <origin xyz="-0.012 ${reflect * 0.000} -0.025" rpy="0 0 0"/>
                 <mass value="0.243"/>
-                <inertia ixx="1.0" ixy="0.0" ixz="0.0" iyy="1.0" iyz="0.0" izz="1.0" />
-              <!-- <inertia ixx="0.00024" ixy="0.0" ixz="0.0" iyy="0.00101" iyz="0.0" izz="0.00092" /> -->
+                <!-- <inertia ixx="1.0" ixy="0.0" ixz="0.0" iyy="1.0" iyz="0.0" izz="1.0" /> -->
+                <inertia ixx="0.00024" ixy="0.0" ixz="0.0" iyy="0.00101" iyz="0.0" izz="0.00092" />
             </inertial>
         </link>
@@ -64,6 +64,6 @@
                 <origin xyz="-0.068 ${reflect * 0.000} 0.000" rpy="0 0 0"/>
                 <mass value="1.045"/>
-                <inertia ixx="1.0" ixy="0.0" ixz="0.0" iyy="1.0" iyz="0.0" izz="1.0" />
-                <!-- <inertia ixx="0.00056" ixy="0.0" ixz="0.0" iyy="0.00168" iyz="0.0" izz="0.00171" /> -->
+                <!-- <inertia ixx="1.0" ixy="0.0" ixz="0.0" iyy="1.0" iyz="0.0" izz="1.0" /> -->
+                <inertia ixx="0.00056" ixy="0.0" ixz="0.0" iyy="0.00168" iyz="0.0" izz="0.00171" />
             </inertial>
         </link>
@@ -101,6 +101,6 @@
                 <origin xyz="0.022 ${reflect * -0.007} -0.168" rpy="0 0 0"/>
                 <mass value="3.095"/>
-                <inertia ixx="1.0" ixy="0.0" ixz="0.0" iyy="1.0" iyz="0.0" izz="1.0" />
-                <!-- <inertia ixx="0.04328" ixy="0.00028" ixz="0.00288" iyy="0.04042" iyz="-0.00202" izz="0.00560" /> -->
+                <!-- <inertia ixx="1.0" ixy="0.0" ixz="0.0" iyy="1.0" iyz="0.0" izz="1.0" />  -->
+                <inertia ixx="0.04328" ixy="${reflect * 0.00028}" ixz="0.00287" iyy="0.04042" iyz="${reflect *-0.00202}" izz="0.00560" />
             </inertial>
         </link>
@@ -138,6 +138,6 @@
                 <origin xyz="-0.002 ${reflect * -0.066} -0.183" rpy="0 0 0"/>
                 <mass value="2.401"/>
-                <inertia ixx="1.0" ixy="0.0" ixz="0.0" iyy="1.0" iyz="0.0" izz="1.0" />
-                <!-- <inertia ixx="0.01971" ixy="0.00031" ixz="-0.00294" iyy="0.01687" iyz="0.00140" izz="0.00574" /> -->
+                <!--<inertia ixx="1.0" ixy="0.0" ixz="0.0" iyy="1.0" iyz="0.0" izz="1.0" />-->
+                <inertia ixx="0.01971" ixy="${reflect * 0.00031}" ixz="-0.00294" iyy="0.01687" iyz="${reflect * 0.00140}" izz="0.00574" />
             </inertial>
         </link>
@@ -172,6 +172,6 @@
                 <origin xyz="-0.011 ${reflect * -0.033} 0.000" rpy="0 0 0"/>
                 <mass value="1.045"/>
-                <inertia ixx="1.0" ixy="0.0" ixz="0.0" iyy="1.0" iyz="0.0" izz="1.0" />
-                <!-- <inertia ixx="0.00056" ixy="0.0" ixz="0.0" iyy="0.00168" iyz="0.0" izz="0.00171" /> -->
+                <!-- <inertia ixx="1.0" ixy="0.0" ixz="0.0" iyy="1.0" iyz="0.0" izz="1.0" /> -->
+                <inertia ixx="0.00056" ixy="0.0" ixz="0.0" iyy="0.00168" iyz="0.0" izz="0.00171" />
             </inertial>
         </link>
@@ -204,6 +204,6 @@
                 <origin xyz="-0.070 ${reflect * 0.000} -0.048" rpy="0 0 0"/>
                 <mass value="0.223"/>
-                <inertia ixx="1.0" ixy="0.0" ixz="0.0" iyy="1.0" iyz="0.0" izz="1.0" />
-                <!-- <inertia ixx="0.00022" ixy="0.0" ixz="-0.00001" iyy="0.00099" iyz="0.0" izz="0.00091" /> -->
+                <!-- <inertia ixx="1.0" ixy="0.0" ixz="0.0" iyy="1.0" iyz="0.0" izz="1.0" /> -->
+                <inertia ixx="0.00022" ixy="0.0" ixz="-0.00001" iyy="0.00099" iyz="0.0" izz="0.00091" />
             </inertial>
         </link>
@@ -241,8 +241,9 @@
             </visual>
             <inertial>
-                <origin xyz="0.000 ${reflect * 0.009} -0.013" rpy="0 0 0"/>
+		<!--<origin xyz="0.000 ${reflect * 0.009} -0.013" rpy="0 0 0"/>-->
+                <origin xyz="0.000 ${reflect * 0.009} +0.013" rpy="0 0 0"/>
                 <mass value="1.689"/>
-                <inertia ixx="1.0" ixy="0.0" ixz="0.0" iyy="1.0" iyz="0.0" izz="1.0" />
-                <!-- <inertia ixx="0.00219" ixy="0.0" ixz="0.0" iyy="0.00433" iyz="0.00011" izz="0.00609" /> -->
+                <!-- <inertia ixx="1.0" ixy="0.0" ixz="0.0" iyy="1.0" iyz="0.0" izz="1.0" /> -->
+                <inertia ixx="0.00219" ixy="0.0" ixz="0.0" iyy="0.00433" iyz="${reflect * 0.00011}" izz="0.00609" />
             </inertial>
         </link>

File: thormang3_description/urdf/thormang3.structure.torso.xacro (robot description, xacro)
@@ -34,5 +34,6 @@
       <origin xyz="0 0 0" rpy="0 0 0"/>
       <geometry>
-        <mesh filename="package://thormang3_description/meshes/robotis_pelvis_link.stl" scale="0.001 0.001 0.001"/>
+	<!--<mesh filename="package://thormang3_description/meshes/robotis_pelvis_link.stl" scale="0.001 0.001 0.001"/>-->
+        <mesh filename="package://thormang3_description/meshes/robotis_pelvis_link_upgraded.stl" scale="0.001 0.001 0.001"/>
       </geometry>
       <material name="grey"/>
@@ -40,7 +41,10 @@
     <inertial>
       <origin xyz="-0.011 0.000 0.058" rpy="0 0 0"/>
+      <!--<origin xyz="-0.006 0.0 0.061" rpy="0 0 0"/>-->
       <mass value="6.869"/>
-      <inertia ixx="1.0" ixy="0.0" ixz="0.0" iyy="1.0" iyz="0.0" izz="1.0" />
-      <!--<inertia ixx="0.03603" ixy="0.0" ixz="0.00016" iyy="0.02210" iyz="0.0" izz="0.03830" />-->
+      <!--<mass value="6.767"/>-->
+      <!--<inertia ixx="1.0" ixy="0.0" ixz="0.0" iyy="1.0" iyz="0.0" izz="1.0" />-->
+      <inertia ixx="0.03603" ixy="0.0" ixz="0.00016" iyy="0.02210" iyz="0.0" izz="0.03830" />
+      <!--<inertia ixx="0.059" ixy="0.0" ixz="-0.002" iyy="0.048" iyz="0.0" izz="0.034" />-->
     </inertial>
   </link>
@@ -49,5 +53,6 @@
     <parent link="pelvis_link"/>
     <child link="chest_link"/>
-    <origin xyz="0 0 0.1705" rpy="0 0 0"/>
+    <!--<origin xyz="0 0 0.1705" rpy="0 0 0"/>-->
+    <origin xyz="0 0 0.1775" rpy="0 0 0"/> <!--torso 7mm higher because of pelvis upgrade (cf. new .stl)-->
     <axis xyz="0 0 1"/>
     <limit velocity="6.5" effort="1000" lower="${-pi*0.25}" upper="${pi*0.25}" />
@@ -177,6 +182,6 @@
       <origin xyz="-0.007 0.000 0.109" rpy="0 0 0"/>
       <mass value="5.383"/>
-      <inertia ixx="1.0" ixy="0.0" ixz="0.0" iyy="1.0" iyz="0.0" izz="1.0" />
-      <inertia ixx="0.04710" ixy="0.0" ixz="0.04710" iyy="0.02554" iyz="0.0" izz="0.03094" />
+      <!--<inertia ixx="1.0" ixy="0.0" ixz="0.0" iyy="1.0" iyz="0.0" izz="1.0" />-->
+      <inertia ixx="0.04710" ixy="0.0" ixz="0.00036" iyy="0.02554" iyz="0.0" izz="0.03094" />
     </inertial>
   </link>

Commit message: added torso upgrade and fixed CoMs

File: thormang3_description/urdf/thormang3.structure.arm.xacro (robot description, xacro)
@@ -144,5 +144,5 @@
           </visual>
           <inertial>
-            <origin xyz="0.000 0.073 0.000" rpy="0 0 0" />
+            <origin xyz="0.000 ${reflect * 0.073} 0.000" rpy="0 0 0" />
             <mass value="1.122" />
             <inertia ixx="1.0" ixy="0.0" ixz="0.0" iyy="1.0" iyz="0.0" izz="1.0" />
@@ -314,5 +314,5 @@
           </visual>
           <inertial>
-            <origin xyz="0.049 ${reflect * 0.045} ${reflect * 0.002}" rpy="0 0 0" />
+            <origin xyz="0.029 ${reflect * 0.045} 0.0" rpy="0 0 0" />
             <mass value="0.087" />
             <inertia ixx="1.0" ixy="0.0" ixz="0.0" iyy="1.0" iyz="0.0" izz="1.0" />

File: thormang3_description/urdf/thormang3.structure.head.xacro (robot description, xacro)
@@ -60,6 +60,8 @@
     	  </visual>
           <inertial>
-      	    <origin xyz="0.009 0.046 0.022" rpy="0 0 0"/>
-      	    <mass value="0.724"/>
+      	    <!--<origin xyz="0.009 0.046 0.022" rpy="0 0 0"/>-->
+      	    <origin xyz="-0.012 0.044 0.072" rpy="0 0 0"/>
++      	    <!--<mass value="0.724"/>-->
++	    <mass value="1.048"/>
       	    <inertia ixx="1.0" ixy="0.0" ixz="0.0" iyy="1.0" iyz="0.0" izz="1.0" />
     	  </inertial>

File: thormang3_description/urdf/thormang3.structure.leg.xacro (robot description, xacro)
@@ -28,5 +28,5 @@
             </visual>
             <inertial>
-                <origin xyz="0.012 ${reflect * 0.000} -0.025" rpy="0 0 0"/>
+                <origin xyz="-0.012 ${reflect * 0.000} -0.025" rpy="0 0 0"/>
                 <mass value="0.243"/>
                 <inertia ixx="1.0" ixy="0.0" ixz="0.0" iyy="1.0" iyz="0.0" izz="1.0" />
@@ -241,5 +241,5 @@
             </visual>
             <inertial>
-                <origin xyz="0.000 ${reflect * 0.009} -0.013" rpy="0 0 0"/>
+                <origin xyz="0.000 ${reflect * 0.009} 0.013" rpy="0 0 0"/>
                 <mass value="1.689"/>
                 <inertia ixx="1.0" ixy="0.0" ixz="0.0" iyy="1.0" iyz="0.0" izz="1.0" />

File: thormang3_description/urdf/thormang3.structure.torso.xacro (robot description, xacro)
@@ -34,5 +34,5 @@
       <origin xyz="0 0 0" rpy="0 0 0"/>
       <geometry>
-        <mesh filename="package://thormang3_description/meshes/robotis_pelvis_link.stl" scale="0.001 0.001 0.001"/>
+        <mesh filename="package://thormang3_description/meshes/robotis_pelvis_link_upgraded.stl" scale="0.001 0.001 0.001"/>
       </geometry>
       <material name="grey"/>
@@ -49,5 +49,6 @@
     <parent link="pelvis_link"/>
     <child link="chest_link"/>
-    <origin xyz="0 0 0.1705" rpy="0 0 0"/>
+    <!--<origin xyz="0 0 0.1705" rpy="0 0 0"/>-->
+    <origin xyz="0 0 0.1775" rpy="0 0 0"/><!--torso 7mm higher because of pelvis upgrade (cf. new .stl)-->
     <axis xyz="0 0 1"/>
     <limit velocity="6.5" effort="1000" lower="${-pi*0.25}" upper="${pi*0.25}" />

Commit message: Extended urdf in order to fix issues with MoveIt

File: thormang3_description/urdf/thormang3.structure.arm.xacro (robot description, xacro)
@@ -2,4 +2,11 @@
 <robot xmlns:xacro="http://ros.org/wiki/xacro">
   <xacro:property name="offset" value="0.0" />
+  <xacro:arg name="wrist_ft_sensor" default="true" />
+  <xacro:if value="$(arg wrist_ft_sensor)">
+    <xacro:property name="arm_ft_joint_type" value="revolute" />
+  </xacro:if>
+  <xacro:unless value="$(arg wrist_ft_sensor)">
+    <xacro:property name="arm_ft_joint_type" value="fixed" />
+  </xacro:unless>
   <xacro:arg name="l_hand_type" default="none" />
   <xacro:arg name="r_hand_type" default="none" />
@@ -341,5 +348,5 @@
     <!--ft joint -->
     <!--use "fixed" revolute joint for FT sensor simulation-->
-    <joint name="${prefix}_arm_ft" type="revolute">
+    <joint name="${prefix}_arm_ft" type="${arm_ft_joint_type}">
       <origin xyz="0.055 ${reflect * 0.045} 0" rpy="${-reflect * 0.5 * pi} 0 ${-reflect * 0.5 * pi}" />
       <parent link="${prefix}_arm_wr_p_link" />

File: thormang3_description/urdf/thormang3.structure.torso.xacro (robot description, xacro)
@@ -5,5 +5,5 @@
   <xacro:include filename="$(find thormang3_description)/urdf/thormang3.structure.leg.xacro" />
   <xacro:include filename="$(find thormang3_description)/urdf/thormang3.structure.head.xacro" />
-  <!-- Used for pinning robot -->
+  <!-- used for pinning robot -->
   <xacro:arg name="pinned" default="false"/>
   <xacro:if value="$(arg pinned)">

Commit message: fixed negative box size

File: thormang3_description/urdf/thormang3.structure.arm.xacro (robot description, xacro)
@@ -324,5 +324,5 @@
         <origin xyz="0.0055 ${reflect *-0.005} 0.0" rpy="${pi*0.5} ${pi*0.5} 0" />
         <geometry>
-          <box size="0.05 ${reflect *0.065} 0.01" />
+          <box size="0.05 0.065 0.01" />
         </geometry>
       </collision>
