Commit message: lidar calibratin

File: thormang3_description/calibration/multisensor_head_calibration.urdf.xacro (robot description, xacro)
@@ -1,9 +1,9 @@
 <?xml version="1.0"?>
 <!-- =================================================================================== -->
-<!-- |    This document was autogenerated by lidar_calibration on 1.07.2016, 10:56:42.| -->
+<!-- |    This document was autogenerated by lidar_calibration on 2.07.2016, 19:03:39.| -->
 <!-- |    Insert this transformation between frames head_lidar_mount_link and head_link_hokuyo_laser_frame. | -->
 <!-- |    EDITING THIS FILE BY HAND IS NOT RECOMMENDED                                 | -->
 <!-- =================================================================================== -->
 <robot xmlns:xacro="http://www.ros.org/wiki/xacro" name="calibration">
-  <origin rpy="0 0 0" xyz="0 0 -0"/>
+  <origin rpy="3.14159 3.11752 3.14058" xyz="0 -0.00237062 0.0100379"/>
 </robot>

Commit message: migration for kinetic

File: thormang3_description/calibration/multisensor_head_calibration.urdf.xacro (robot description, xacro)
@@ -5,5 +5,5 @@
 <!-- |    EDITING THIS FILE BY HAND IS NOT RECOMMENDED                                 | -->
 <!-- =================================================================================== -->
-<robot xmlns:xacro="http://www.ros.org/wiki/xacro" name="calibration">
+<robot xmlns:xacro="http://ros.org/wiki/xacro" name="calibration">
   <origin rpy="3.14159 3.11752 3.14058" xyz="0 -0.00237062 0.0100379"/>
 </robot>

File: thormang3_description/urdf/thormang3.structure.head.xacro (robot description, xacro)
@@ -71,5 +71,5 @@
           <child link="head_link"/>
         </joint>
-	<hector_multisensor_head_macro parent="head_y_link"  name="head" scaling="0.001">
+	<hector_multisensor_head_macro parent="head_y_link" name="head" scaling="0.001">
 	  <origin xyz="0.0 0.0 0.0" rpy="${M_PI*0.5} 0.0 ${M_PI*0.5}"/>
 	  <!-- Calibrated origin of the laser scanner-->

File: thormang3_description/urdf/thormang3.structure.torso.xacro (robot description, xacro)
@@ -1,6 +1,5 @@
 <?xml version="1.0"?>
-<robot xmlns:xacro="http://www.ros.org/wiki/xacro">
+<robot xmlns:xacro="http://ros.org/wiki/xacro">
   <!-- some parameters -->
-  <xacro:property name="pi" value="3.141592" />
   <xacro:include filename="$(find thormang3_description)/urdf/thormang3.structure.arm.xacro" />
   <xacro:include filename="$(find thormang3_description)/urdf/thormang3.structure.leg.xacro" />

File: thormang3_description/urdf/thormang3.xacro (robot description, xacro)
@@ -1,4 +1,5 @@
 <?xml version="1.0"?>
-<robot name="$(arg robot_name)" xmlns:xacro="http://www.ros.org/wiki/xacro">
+<robot name="$(arg robot_name)" xmlns:xacro="http://ros.org/wiki/xacro">
+  <xacro:include filename="$(find thormang3_description)/urdf/thormang3.transmissions.xacro" />
   <!-- Import all Gazebo-customization elements, including Gazebo colors -->
   <xacro:include filename="$(find thormang3_description)/urdf/thormang3.gazebo" />
@@ -6,4 +7,3 @@
   <xacro:include filename="$(find thormang3_description)/urdf/materials.xacro" />
   <xacro:include filename="$(find thormang3_description)/urdf/thormang3.structure.torso.xacro" />
-  <xacro:include filename="$(find thormang3_description)/urdf/thormang3.transmissions.xacro" />
 </robot>

Commit message: updated calibration

File: thormang3_description/calibration/multisensor_head_calibration.urdf.xacro (robot description, xacro)
@@ -6,4 +6,4 @@
 <!-- =================================================================================== -->
 <robot xmlns:xacro="http://ros.org/wiki/xacro" name="calibration">
-  <origin rpy="3.14159 3.11752 3.14058" xyz="0 -0.00237062 0.0100379"/>
+  <origin rpy="0 0.0459734 0.00054707" xyz="0 0.000151927 0.00627848"/>
 </robot>
